File: Test Projects/Teensy_test_layout.kicad_pcb (KiCad board)
At the start: 2 copper layers, 304.8 x 177.8 mm, 137 parts, among them P1 CONN_01X02, P10 CONN_01X06, P11 CONN_01X06, P12 CONN_01X06, P13 CONN_01X08, P14 CONN_01X08, P15 CONN_01X08, P16 CONN_01X08, P17 CONN_01X08, P18 CONN_01X08, P19 CONN_01X08, P2 CONN_01X03, P20 CONN_01X08, P21 CONN_01X07, P22 CONN_01X08, P23 CONN_01X08, P24 CONN_01X08, P25 CONN_01X08, P26 CONN_01X08, P27 CONN_01X08, P28 CONN_01X08, P29 CONN_01X08, P3 COLS0, P30 CONN_01X03, P4 COLS1, P5 CONN_01X06, P6 CONN_01X06, P7 CONN_01X06, P8 CONN_01X06, P9 CONN_01X06, U1 LDO-adj-4term, U10 SF-74x125, U11 2N168, U12 SF-LM358, U13 SF-4052, U14 SF-4052, U15 SF-4052, U16 SF-4052, U17 SF-4052, U18 SF-4052, U19 SF-4052, U2 LDO-adj-4term, U20 SF-4052, U21 SF-4052, U22 SF-4052, U23 SF-74HC595, U24 SF-74HC595, U25 SF-74HC595, U26 SF-74HC595, U27 SF-74HC595, U28 SF-74HC595, U29 SF-74HC595, U3 Teensy_3.2, U30 SF-74HC595, U31 SGTL5000, U4 LDO-adj-4term, U5 SGTL5000, U6 SF-MicroSD-12term, U7 SF-74HC595, U8 SF-74HC595, U9 SF-74x125

Commit message: First major routing pass
Parts:
- added C42: C, Capacitors_SMD:C_0603, F.Cu at (72.4, 127.0)
- added JMP8: 2Jumper, SparkFun-Footprints:SF-2way-open, F.Cu at (78.7, 133.3)
- added JMP9: 2Jumper, SparkFun-Footprints:SF-2way-open, F.Cu at (78.7, 135.9)
- added P31: PIN20, SparkFun-Footprints:Single_PTH, F.Cu at (50.8, 99.1)
- added P32: PIN8, SparkFun-Footprints:Single_PTH, F.Cu at (58.4, 121.9)
- added P33: SIO2, SparkFun-Footprints:Single_PTH, F.Cu at (76.2, 133.3)
- added P34: ~HOLD~/SIO3, SparkFun-Footprints:Single_PTH, F.Cu at (76.2, 135.9)
- added P35: PIN37, SparkFun-Footprints:Single_PTH, F.Cu at (71.1, 104.1)
- added P36: PIN29, SparkFun-Footprints:Single_PTH, F.Cu at (64.8, 96.5)
- added P37: PIN31, SparkFun-Footprints:Single_PTH, F.Cu at (59.7, 96.5)
- added REF**: MountingHole_3mm, Mounting_Holes:MountingHole_3mm, F.Cu at (274.3, 110.5)
- added REF**: MountingHole_3mm, Mounting_Holes:MountingHole_3mm, F.Cu at (30.5, 146.1)
- added REF**: MountingHole_3mm, Mounting_Holes:MountingHole_3mm, F.Cu at (30.5, 31.8)
- added REF**: MountingHole_3mm, Mounting_Holes:MountingHole_3mm, F.Cu at (189.2, 109.2)
- added REF**: MountingHole_3mm, Mounting_Holes:MountingHole_3mm, F.Cu at (101.6, 120.7)
- added REF**: MountingHole_3mm, Mounting_Holes:MountingHole_3mm, F.Cu at (88.9, 50.8)
- added REF**: MountingHole_3mm, Mounting_Holes:MountingHole_3mm, F.Cu at (31.8, 95.2)
- added REF**: MountingHole_3mm, Mounting_Holes:MountingHole_3mm, F.Cu at (232.4, 63.5)
- added REF**: MountingHole_3mm, Mounting_Holes:MountingHole_3mm, F.Cu at (151.1, 63.5)
- added REF**: MountingHole_3mm, Mounting_Holes:MountingHole_3mm, F.Cu at (274.3, 31.8)
- added REF**: MountingHole_3mm, Mounting_Holes:MountingHole_3mm, F.Cu at (274.3, 146.1)
- added U32: SPI_MEMORY_SOIC8, SparkFun-Footprints:SF-SOIC-8, F.Cu at (76.2, 127.0)
- moved JMP1 67.8 mm to (30.5, 109.9)
- moved JMP4 33.6 mm to (94.6, 101.0), turned to 180 degrees
- moved P2 31.2 mm to (108.0, 92.7), turned to 0 degrees
- moved C11 26.9 mm to (100.3, 97.4), turned to 90 degrees
- moved JMP3 25.6 mm to (88.5, 97.8)
- moved JMP2 24.7 mm to (88.5, 99.7)
- moved C12 22.5 mm to (104.8, 92.5), turned to 90 degrees
- moved C39 22.2 mm to (87.6, 73.4), turned to 90 degrees
- moved JMP6 21.4 mm to (87.9, 81.3)
- moved JMP7 21.3 mm to (87.9, 79.4)
- moved C13 20.9 mm to (104.8, 97.6)
- moved U5 17.7 mm to (94.0, 94.6), turned to 180 degrees
- moved R7 17.5 mm to (100.3, 101.6), turned to 0 degrees
- moved C10 16.6 mm to (88.9, 90.2)
- moved R8 16.0 mm to (76.2, 94.7), turned to 270 degrees
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Connections:
- net Net-(C8-Pad1) renamed +3V3_REG
- net Net-(JMP1-Pad1) renamed +3V3_TOUT
- net SD_MISO renamed SPI_MISO
- C15 pad 1: Net-(C15-Pad1) -> +3V3
- C15 pad 2: Net-(C15-Pad2) -> GND
- C16 pad 1: Net-(C16-Pad1) -> +3V3
- C16 pad 2: Net-(C16-Pad2) -> GND
- JACK1 pad 1: Net-(JACK1-Pad1) -> (no net)
- JACK1 pad 2: Net-(JACK1-Pad2) -> (no net)
- JACK1 pad 3: Net-(JACK1-Pad3) -> (no net)
- JACK1 pad 6: Net-(JACK1-Pad6) -> (no net)
- JACK1 pad 7: Net-(JACK1-Pad7) -> (no net)
- JACK2 pad 1: Net-(JACK2-Pad1) -> (no net)
- JACK2 pad 2: Net-(JACK2-Pad2) -> (no net)
- JACK2 pad 3: Net-(JACK2-Pad3) -> (no net)
- JACK2 pad 6: Net-(JACK2-Pad6) -> (no net)
- JACK2 pad 7: Net-(JACK2-Pad7) -> (no net)
- JACK3 pad 1: Net-(JACK3-Pad1) -> (no net)
- JACK3 pad 2: Net-(JACK3-Pad2) -> (no net)
- JACK3 pad 3: Net-(JACK3-Pad3) -> (no net)
- JACK3 pad 6: Net-(JACK3-Pad6) -> (no net)
- JACK3 pad 7: Net-(JACK3-Pad7) -> (no net)
- U11 pad 1: Net-(U11-Pad1) -> (no net)
- U11 pad 4: Net-(U11-Pad4) -> (no net)
- U11 pad 7: Net-(U11-Pad7) -> (no net)
- U12 pad 1: Net-(U12-Pad1) -> (no net)
- U12 pad 2: Net-(U12-Pad2) -> (no net)
- U12 pad 3: Net-(U12-Pad3) -> (no net)
- U12 pad 5: Net-(U12-Pad5) -> (no net)
- U12 pad 6: Net-(U12-Pad6) -> (no net)
- U12 pad 7: Net-(U12-Pad7) -> (no net)
- U13 pad 16: Net-(U13-Pad16) -> (no net)
- U13 pad 8: Net-(U13-Pad8) -> (no net)
- U14 pad 16: Net-(U14-Pad16) -> (no net)
- U14 pad 8: Net-(U14-Pad8) -> (no net)
- U15 pad 16: Net-(U15-Pad16) -> (no net)
- U15 pad 8: Net-(U15-Pad8) -> (no net)
- U16 pad 16: Net-(U16-Pad16) -> (no net)
- U16 pad 8: Net-(U16-Pad8) -> (no net)
- U17 pad 16: Net-(U17-Pad16) -> (no net)
- U17 pad 8: Net-(U17-Pad8) -> (no net)
- U18 pad 16: Net-(U18-Pad16) -> (no net)
- U18 pad 8: Net-(U18-Pad8) -> (no net)
- U19 pad 16: Net-(U19-Pad16) -> (no net)
- U19 pad 8: Net-(U19-Pad8) -> (no net)
- U20 pad 16: Net-(U20-Pad16) -> (no net)
- U20 pad 8: Net-(U20-Pad8) -> (no net)
- U21 pad 16: Net-(U21-Pad16) -> (no net)
- U21 pad 8: Net-(U21-Pad8) -> (no net)
- U22 pad 16: Net-(U22-Pad16) -> (no net)
- U22 pad 8: Net-(U22-Pad8) -> (no net)
- U23 pad 10: Net-(U23-Pad10) -> !LED_RST
- U23 pad 11: SD_LED_SCK -> SPI_SCK
- U23 pad 12: LEDLATCH -> LED_LATCH
- U23 pad 13: LEDOE -> LED_OE
- U23 pad 14: SD_LED_MOSI -> SPI_MOSI
- U24 pad 10: Net-(U24-Pad10) -> !LED_RST
- U24 pad 11: SD_LED_SCK -> SPI_SCK
- U24 pad 12: LEDLATCH -> LED_LATCH
- U24 pad 13: LEDOE -> LED_OE
- U25 pad 10: Net-(U25-Pad10) -> !LED_RST
- U25 pad 11: SD_LED_SCK -> SPI_SCK
- U25 pad 12: LEDLATCH -> LED_LATCH
- U25 pad 13: LEDOE -> LED_OE
- U26 pad 10: Net-(U26-Pad10) -> !LED_RST
- U26 pad 11: SD_LED_SCK -> SPI_SCK
- U26 pad 12: LEDLATCH -> LED_LATCH
- U26 pad 13: LEDOE -> LED_OE
- U27 pad 10: Net-(U27-Pad10) -> !LED_RST
- U27 pad 11: SD_LED_SCK -> SPI_SCK
- U27 pad 12: LEDLATCH -> LED_LATCH
- U27 pad 13: LEDOE -> LED_OE
- U28 pad 10: Net-(U28-Pad10) -> !LED_RST
- U28 pad 11: SD_LED_SCK -> SPI_SCK
- U28 pad 12: LEDLATCH -> LED_LATCH
- U28 pad 13: LEDOE -> LED_OE
- U29 pad 10: Net-(U29-Pad10) -> !LED_RST
- U29 pad 11: SD_LED_SCK -> SPI_SCK
- U29 pad 12: LEDLATCH -> LED_LATCH
- U29 pad 13: LEDOE -> LED_OE
- U3 pad 14: LEDLATCH -> SPI_SCK
- U3 pad 26: SD_LED_SCK -> !LED_RST
- U3 pad 31: SD_LED_MOSI -> Net-(P37-Pad1)
- U3 pad 32: Net-(U3-Pad32) -> LED_LATCH
- U3 pad 33: Net-(U3-Pad33) -> LED_OE
- U3 pad 35: Net-(U3-Pad35) -> (no net)
- U3 pad 38: Net-(U3-Pad38) -> (no net)
- U3 pad 41: Net-(U3-Pad41) -> (no net)
- U3 pad 48: Net-(U3-Pad48) -> (no net)
- U3 pad 49: Net-(U3-Pad49) -> (no net)
- U3 pad 6: LEDOE -> RAM_CS
- U3 pad 7: Net-(U3-Pad7) -> SPI_MOSI
- U30 pad 10: Net-(U30-Pad10) -> !LED_RST
- U30 pad 11: SD_LED_SCK -> SPI_SCK
- U30 pad 12: LEDLATCH -> LED_LATCH
- U30 pad 13: LEDOE -> LED_OE
- U30 pad 9: Net-(U30-Pad9) -> (no net)
- U31 pad 11: Net-(U31-Pad11) -> (no net)
- U31 pad 12: Net-(U31-Pad12) -> (no net)
- U31 pad 13: Net-(U31-Pad13) -> (no net)
- U31 pad 14: Net-(U31-Pad14) -> (no net)
- U31 pad 15: Net-(U31-Pad15) -> (no net)
- U31 pad 16: Net-(U31-Pad16) -> (no net)
- U31 pad 18: Net-(U31-Pad18) -> (no net)
- U5 pad 11: Net-(U5-Pad11) -> (no net)
- U5 pad 12: Net-(U5-Pad12) -> (no net)
- U5 pad 13: Net-(U5-Pad13) -> (no net)
- U5 pad 14: Net-(U5-Pad14) -> (no net)
- U5 pad 15: Net-(U5-Pad15) -> (no net)
- U5 pad 16: Net-(U5-Pad16) -> (no net)
- U5 pad 18: Net-(U5-Pad18) -> (no net)
- U6 pad 1: Net-(U6-Pad1) -> (no net)
- U6 pad 10: Net-(U6-Pad10) -> (no net)
- U6 pad 11: Net-(U6-Pad11) -> (no net)
- U6 pad 12: Net-(U6-Pad12) -> (no net)
- U6 pad 3: SD_LED_MOSI -> SPI_MOSI
- U6 pad 5: SD_LED_SCK -> SPI_SCK
- U6 pad 8: Net-(U6-Pad8) -> (no net)
- U6 pad 9: Net-(U6-Pad9) -> (no net)
- U7 pad 10: Net-(U7-Pad10) -> +3V3
- U7 pad 16: Net-(C15-Pad1) -> +3V3
- U7 pad 8: Net-(C15-Pad2) -> GND
- U8 pad 10: Net-(U8-Pad10) -> +3V3
- U8 pad 14: Net-(U8-Pad14) -> Net-(U7-Pad9)
- U8 pad 16: Net-(C16-Pad1) -> +3V3
- U8 pad 8: Net-(C16-Pad2) -> GND
- U8 pad 9: Net-(U8-Pad9) -> (no net)
Routing:
- net LED_LATCH: track 0.00 -> 247.0 mm, vias 0 -> 9
- net SPI_SCK: track 0.00 -> 244.7 mm, vias 0 -> 11
- net LED_OE: track 0.00 -> 236.3 mm, vias 0 -> 9
- net !LED_RST: track 0.00 -> 230.0 mm, vias 0 -> 9
- net +5V: track 0.00 -> 207.6 mm, vias 0 -> 8
- net KA3: track 0.00 -> 87.3 mm
- net KA1: track 0.00 -> 82.0 mm
- net KA0: track 0.00 -> 81.7 mm, vias 0 -> 2
- net SPI_MOSI: track 0.00 -> 81.1 mm, vias 0 -> 5
- net KA2: track 0.00 -> 79.5 mm
- net +3V3: track 0.00 -> 69.3 mm, vias 0 -> 4
- net BCLK: track 0.00 -> 60.7 mm, vias 0 -> 3
- net SD_CS: track 0.00 -> 49.1 mm, vias 0 -> 2
- net BOE: track 0.00 -> 46.0 mm, vias 0 -> 3
- net BLATCH: track 0.00 -> 45.8 mm, vias 0 -> 3
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- added copper zone on B.Cu, net GND
- added copper zone on F.Cu, net GND
Other:
- board size 304.8 x 177.8 mm -> 254 x 127 mm
- net class Jack Interface added: clearance 0.254, trace_width 0.4064, via_dia 0.635, via_drill 0.381

Commit message: Post review with Byron
Parts:
- removed REF** (x11): MountingHole_3mm, Mounting_Holes:MountingHole_3mm
- added P38: CONN_01X05, Pin_Headers:Pin_Header_Straight_1x05, F.Cu at (112.4, 89.5)
- added P39: CONN_01X05, Pin_Headers:Pin_Header_Straight_1x05, F.Cu at (112.4, 71.1)
- C10, C11, C12, C13, C14, C37, C38, C39, C40, C41: footprint Capacitors_SMD:C_1206 -> Capacitors_SMD:C_0603
- moved C27 21.5 mm to (142.2, 114.9), turned to 90 degrees
- moved U21 17.1 mm to (148.6, 116.8), turned to 180 degrees
- moved C21 16.8 mm to (165.7, 111.8), turned to 0 degrees
- moved C22 16.7 mm to (185.9, 111.8), turned to 0 degrees
- moved C19 12.3 mm to (118.7, 111.8), turned to 0 degrees
- moved JMP4 10.9 mm to (85.7, 94.6), turned to 270 degrees
- moved C20 10.3 mm to (134.0, 111.8), turned to 0 degrees
- moved JMP5 10.0 mm to (85.7, 75.6), turned to 270 degrees
- moved R16 8.84 mm to (102.2, 74.9), turned to 270 degrees
- moved R7 8.47 mm to (102.2, 93.3), turned to 270 degrees
- moved P30 7.73 mm to (107.3, 81.3), turned to 270 degrees
- moved U14 7.73 mm to (132.1, 118.1)
- moved P2 7.01 mm to (107.3, 99.7), turned to 270 degrees
- moved C12 6.41 mm to (98.4, 93.3)
- moved C13 6.13 mm to (100.3, 93.3), turned to 90 degrees
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Connections:
- JACK1 pad 1: (no net) -> Net-(JACK1-Pad1)
- JACK1 pad 2: (no net) -> Net-(JACK1-Pad2)
- JACK1 pad 3: (no net) -> Net-(JACK1-Pad3)
- JACK1 pad 6: (no net) -> Net-(JACK1-Pad6)
- JACK1 pad 7: (no net) -> Net-(JACK1-Pad7)
- JACK2 pad 1: (no net) -> Net-(JACK2-Pad1)
- JACK2 pad 2: (no net) -> Net-(JACK2-Pad2)
- JACK2 pad 3: (no net) -> Net-(JACK2-Pad3)
- JACK2 pad 6: (no net) -> Net-(JACK2-Pad6)
- JACK2 pad 7: (no net) -> Net-(JACK2-Pad7)
- JACK3 pad 1: (no net) -> Net-(JACK3-Pad1)
- JACK3 pad 2: (no net) -> Net-(JACK3-Pad2)
- JACK3 pad 3: (no net) -> Net-(JACK3-Pad3)
- JACK3 pad 6: (no net) -> Net-(JACK3-Pad6)
- JACK3 pad 7: (no net) -> Net-(JACK3-Pad7)
- U11 pad 1: (no net) -> Net-(U11-Pad1)
- U11 pad 4: (no net) -> Net-(U11-Pad4)
- U11 pad 7: (no net) -> Net-(U11-Pad7)
- U12 pad 1: (no net) -> Net-(U12-Pad1)
- U12 pad 2: (no net) -> Net-(U12-Pad2)
- U12 pad 3: (no net) -> Net-(U12-Pad3)
- U12 pad 5: (no net) -> Net-(U12-Pad5)
- U12 pad 6: (no net) -> Net-(U12-Pad6)
- U12 pad 7: (no net) -> Net-(U12-Pad7)
- U13 pad 16: (no net) -> VDD
- U13 pad 8: (no net) -> GND
- U14 pad 16: (no net) -> VDD
- U14 pad 8: (no net) -> GND
- U15 pad 16: (no net) -> VDD
- U15 pad 8: (no net) -> GND
- U16 pad 16: (no net) -> VDD
- U16 pad 8: (no net) -> GND
- U17 pad 16: (no net) -> VDD
- U17 pad 8: (no net) -> GND
- U18 pad 16: (no net) -> VDD
- U18 pad 8: (no net) -> GND
- U19 pad 16: (no net) -> VDD
- U19 pad 8: (no net) -> GND
- U20 pad 16: (no net) -> VDD
- U20 pad 8: (no net) -> GND
- U21 pad 16: (no net) -> VDD
- U21 pad 8: (no net) -> GND
- U22 pad 16: (no net) -> VDD
- U22 pad 8: (no net) -> GND
- U3 pad 35: (no net) -> Net-(U3-Pad35)
- U3 pad 38: (no net) -> Net-(U3-Pad38)
- U3 pad 41: (no net) -> Net-(U3-Pad41)
- U3 pad 48: (no net) -> Net-(U3-Pad48)
- U3 pad 49: (no net) -> Net-(U3-Pad49)
- U30 pad 9: (no net) -> Net-(U30-Pad9)
- U31 pad 11: (no net) -> Net-(P39-Pad4)
- U31 pad 12: (no net) -> Net-(P39-Pad5)
- U31 pad 13: (no net) -> Net-(P39-Pad3)
- U31 pad 14: (no net) -> Net-(P39-Pad2)
- U31 pad 15: (no net) -> Net-(U31-Pad15)
- U31 pad 16: (no net) -> Net-(U31-Pad16)
- U31 pad 18: (no net) -> Net-(U31-Pad18)
- U31 pad 33: (no net) -> GND
- U5 pad 11: (no net) -> Net-(P38-Pad4)
- U5 pad 12: (no net) -> Net-(P38-Pad5)
- U5 pad 13: (no net) -> Net-(P38-Pad3)
- U5 pad 14: (no net) -> Net-(P38-Pad2)
- U5 pad 15: (no net) -> Net-(U5-Pad15)
- U5 pad 16: (no net) -> Net-(U5-Pad16)
- U5 pad 18: (no net) -> Net-(U5-Pad18)
- U5 pad 33: (no net) -> GND
- U6 pad 1: (no net) -> Net-(U6-Pad1)
- U6 pad 10: (no net) -> Net-(U6-Pad10)
- U6 pad 11: (no net) -> Net-(U6-Pad11)
- U6 pad 12: (no net) -> Net-(U6-Pad12)
- U6 pad 8: (no net) -> Net-(U6-Pad8)
- U6 pad 9: (no net) -> Net-(U6-Pad9)
- U8 pad 9: (no net) -> Net-(U8-Pad9)
Routing:
- net EN: track 0.00 -> 81.4 mm, vias 0 -> 5
- net VDD: track 0.00 -> 51.4 mm
- net B: track 0.00 -> 36.7 mm, vias 0 -> 3
- net A: track 0.00 -> 36.5 mm, vias 0 -> 3
- net GND: track 0.66 -> 35.2 mm, vias 0 -> 1
- net K12: track 0.00 -> 21.0 mm, vias 0 -> 2
- net K4: track 0.00 -> 19.4 mm, vias 0 -> 2
- net K16: track 0.00 -> 16.5 mm
- net K25: track 0.00 -> 15.5 mm
- net Net-(C8-Pad1): track 15.4 -> 0.00 mm
- net +3V3_REG: track 0.00 -> 15.4 mm
- net K28: track 0.00 -> 15.0 mm, vias 0 -> 2
- net K6: track 0.00 -> 14.9 mm, vias 0 -> 2
- net K17: track 0.00 -> 14.8 mm
- net K20: track 0.00 -> 13.1 mm, vias 0 -> 2
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
Commit message: Added holes, moved layout
Parts:
- added C43: 10u, Capacitors_Tantalum_SMD:TantalC_SizeB_EIA-3528_Reflow, F.Cu at (31.8, 100.3)
- added C44: 10u, Capacitors_Tantalum_SMD:TantalC_SizeB_EIA-3528_Reflow, F.Cu at (49.5, 103.5)
- added C45: 10u, Capacitors_Tantalum_SMD:TantalC_SizeB_EIA-3528_Reflow, F.Cu at (49.5, 98.4)
- added C46: 2.2u, Capacitors_Tantalum_SMD:TantalC_SizeB_EIA-3528_Reflow, F.Cu at (160.0, 86.3)
- added C47: 2.2u, Capacitors_Tantalum_SMD:TantalC_SizeB_EIA-3528_Reflow, F.Cu at (155.6, 86.3)
- added C48: 2.2u, Capacitors_Tantalum_SMD:TantalC_SizeB_EIA-3528_Reflow, F.Cu at (151.8, 86.3)
- added C49: 2.2u, Capacitors_Tantalum_SMD:TantalC_SizeB_EIA-3528_Reflow, F.Cu at (147.3, 86.3)
- added C50: 2.2u, Capacitors_Tantalum_SMD:TantalC_SizeB_EIA-3528_Reflow, F.Cu at (160.0, 66.0)
- added C51: 2.2u, Capacitors_Tantalum_SMD:TantalC_SizeB_EIA-3528_Reflow, F.Cu at (155.6, 66.0)
- added C52: 2.2u, Capacitors_Tantalum_SMD:TantalC_SizeB_EIA-3528_Reflow, F.Cu at (151.8, 66.0)
- added C53: 2.2u, Capacitors_Tantalum_SMD:TantalC_SizeB_EIA-3528_Reflow, F.Cu at (147.3, 66.0)
- added C54: D, Capacitors_Tantalum_SMD:TantalC_SizeB_EIA-3528_Reflow, F.Cu at (78.7, 48.3)
- added H1: Hole, Mounting_Holes:MountingHole_3mm, F.Cu at (38.1, 116.8)
- added H2: Hole, Mounting_Holes:MountingHole_3mm, F.Cu at (43.2, 43.2)
- added H3: Hole, Mounting_Holes:MountingHole_3mm, F.Cu at (66.0, 66.0)
- added H4: Hole, Mounting_Holes:MountingHole_3mm, F.Cu at (114.3, 63.5)
- added H5: Hole, Mounting_Holes:MountingHole_3mm, F.Cu at (116.8, 144.8)
- added H6: Hole, Mounting_Holes:MountingHole_3mm, F.Cu at (193.0, 63.5)
- added H7: Hole, Mounting_Holes:MountingHole_3mm, F.Cu at (276.9, 48.3)
- added H8: Hole, Mounting_Holes:MountingHole_3mm, F.Cu at (271.8, 144.8)
- added JMP10: 2Jumper, SparkFun-Footprints:SF-2way-open, F.Cu at (147.3, 86.3)
- added JMP11: 2Jumper, SparkFun-Footprints:SF-2way-open, F.Cu at (151.8, 86.3)
- added JMP12: 2Jumper, SparkFun-Footprints:SF-2way-open, F.Cu at (155.6, 86.3)
- added JMP13: 2Jumper, SparkFun-Footprints:SF-2way-open, F.Cu at (160.0, 86.3)
- added JMP14: 2Jumper, SparkFun-Footprints:SF-2way-open, F.Cu at (147.3, 66.0)
- added JMP15: 2Jumper, SparkFun-Footprints:SF-2way-open, F.Cu at (161.0, 70.4)
- added JMP16: 2Jumper, SparkFun-Footprints:SF-2way-open, F.Cu at (155.6, 66.0)
- added JMP17: 2Jumper, SparkFun-Footprints:SF-2way-open, F.Cu at (160.0, 66.0)
- added JMP18: THRU, SparkFun-Footprints:SF-2way-open, F.Cu at (77.2, 64.8)
- added JMP19: IN2, SparkFun-Footprints:SF-2way-open, F.Cu at (66.7, 50.6)
- added JMP20: IN2, SparkFun-Footprints:SF-2way-open, F.Cu at (68.6, 49.8)
- added P40: CONN_01X08, Pin_Headers:Pin_Header_Straight_1x08, F.Cu at (274.3, 91.4)
- added P41: CONN_01X08, Pin_Headers:Pin_Header_Straight_1x08, F.Cu at (256.5, 121.9)
- added P42: CONN_01X08, Pin_Headers:Pin_Header_Straight_1x08, F.Cu at (248.9, 91.4)
- added P43: CONN_01X08, Pin_Headers:Pin_Header_Straight_1x08, F.Cu at (231.1, 121.9)
- added P44: CONN_01X08, Pin_Headers:Pin_Header_Straight_1x08, F.Cu at (215.9, 91.4)
- added P45: CONN_01X08, Pin_Headers:Pin_Header_Straight_1x08, F.Cu at (198.1, 121.9)
- added P46: CONN_01X08, Pin_Headers:Pin_Header_Straight_1x08, F.Cu at (190.5, 91.7)
- added P47: CONN_01X08, Pin_Headers:Pin_Header_Straight_1x08, F.Cu at (172.7, 122.2)
- added P48: CONN_01X08, Pin_Headers:Pin_Header_Straight_1x08, F.Cu at (274.3, 96.5)
- added P49: CONN_01X08, Pin_Headers:Pin_Header_Straight_1x08, F.Cu at (256.5, 116.8)
- added P50: CONN_01X08, Pin_Headers:Pin_Header_Straight_1x08, F.Cu at (248.9, 96.5)
- added P51: CONN_01X08, Pin_Headers:Pin_Header_Straight_1x08, F.Cu at (231.1, 116.8)
- added P52: CONN_01X08, Pin_Headers:Pin_Header_Straight_1x08, F.Cu at (215.9, 96.5)
- added P53: CONN_01X08, Pin_Headers:Pin_Header_Straight_1x08, F.Cu at (198.1, 116.8)
- added P54: CONN_01X08, Pin_Headers:Pin_Header_Straight_1x08, F.Cu at (172.7, 117.1)
- added P55: CONN_01X08, Pin_Headers:Pin_Header_Straight_1x08, F.Cu at (190.5, 96.8)
- added P56: CONN_01X01, SparkFun-Footprints:TestHole, F.Cu at (41.3, 108.0)
- added P57: CONN_01X01, SparkFun-Footprints:TestHole, F.Cu at (38.1, 108.0)
- added P58: VUU, Pin_Headers:Pin_Header_Straight_1x01, F.Cu at (44.5, 108.0)
- added P59: CONN_01X01, SparkFun-Footprints:TestHole, F.Cu at (39.4, 92.7)
- added P60: CONN_01X01, SparkFun-Footprints:TestHole, F.Cu at (44.5, 92.7)
- added P61: CONN_01X01, SparkFun-Footprints:TestHole, F.Cu at (41.9, 92.7)
- added P62: UGND, Pin_Headers:Pin_Header_Straight_1x01, F.Cu at (44.5, 95.9)
- added P63: CONN_01X01, Pin_Headers:Pin_Header_Straight_1x01, F.Cu at (31.8, 95.2)
- added P64: DIN1, SparkFun-Footprints:TestHole, F.Cu at (92.7, 92.1)
- added P65: DOUT1, SparkFun-Footprints:TestHole, F.Cu at (97.2, 94.6)
- added P66: SDA0, SparkFun-Footprints:TestHole, F.Cu at (85.1, 94.0)
- added P67: SCL0, SparkFun-Footprints:TestHole, F.Cu at (97.2, 90.8)
- added P68: MCLK, SparkFun-Footprints:TestHole, F.Cu at (86.4, 90.2)
- added P69: BCLK, SparkFun-Footprints:TestHole, F.Cu at (91.4, 91.4)
- added P70: LRCLK, SparkFun-Footprints:TestHole, F.Cu at (93.3, 89.5)
- added P71: DIN0, SparkFun-Footprints:TestHole, F.Cu at (89.5, 85.1)
- added P72: DOUT0, SparkFun-Footprints:TestHole, F.Cu at (89.5, 93.3)
- added P73: IN2TTL, SparkFun-Footprints:TestHole, F.Cu at (94.0, 64.1)
- added R17: 4.7k, Resistors_SMD:R_0603, F.Cu at (109.2, 132.1)
- added R18: 4.7k, Resistors_SMD:R_0603, F.Cu at (97.3, 130.2)
- added R19: 11.3K, Resistors_SMD:R_0603, F.Cu at (43.8, 103.6)
- added R20: 34K, Resistors_SMD:R_0603, F.Cu at (43.8, 99.6)
- added R21: 100k, Resistors_SMD:R_0603, F.Cu at (147.3, 94.8)
- added R22: 100k, Resistors_SMD:R_0603, F.Cu at (151.8, 94.8)
- added R23: 100k, Resistors_SMD:R_0603, F.Cu at (154.9, 94.8)
- added R24: 100k, Resistors_SMD:R_0603, F.Cu at (160.0, 94.8)
- added R25: 100k, Resistors_SMD:R_0603, F.Cu at (147.3, 74.9)
- added R26: 100k, Resistors_SMD:R_0603, F.Cu at (152.4, 74.9)
- added R27: 100k, Resistors_SMD:R_0603, F.Cu at (154.9, 74.9)
- added R28: 100k, Resistors_SMD:R_0603, F.Cu at (160.0, 74.9)
- added R29: 220, Resistors_SMD:R_0603, F.Cu at (88.9, 48.3)
- added R30: 220, Resistors_SMD:R_0603, F.Cu at (88.9, 68.6)
- added U33: LDO-adj-4term, SparkFun-Footprints:SF-SOT-223, F.Cu at (38.1, 101.0)
- added U34: 2N168, SparkFun-Footprints:SF-SMD-8, F.Cu at (78.7, 66.0)
- C17: value C -> D
- P38, P39: value CONN_01X05 -> CONN_01X06; footprint Pin_Headers:Pin_Header_Straight_1x05 -> Pin_Headers:Pin_Header_Straight_1x06
- R10, R11, R12, R13, R14, R15: value R -> 220
- moved U12 94.5 mm to (211.5, 70.5)
- moved C18 94.5 mm to (218.4, 70.0)
- moved P14 69.2 mm to (190.5, 94.3), turned to 270 degrees
- moved P13 63.9 mm to (172.7, 119.7)
- moved U13 57.8 mm to (174.0, 109.5)
- moved U14 57.5 mm to (188.0, 104.4), turned to 270 degrees
- moved P16 56.4 mm to (215.9, 94.0), turned to 270 degrees
- moved C19 52.3 mm to (169.4, 99.1)
- moved P18 50.4 mm to (248.9, 94.0), turned to 270 degrees
- moved P15 48.9 mm to (198.1, 119.4)
- moved C20 47.7 mm to (181.6, 114.6), turned to 90 degrees
- moved P38 47.7 mm to (160.0, 91.4), turned to 270 degrees
- moved P39 47.6 mm to (160.0, 71.1), turned to 270 degrees
- moved C23 45.8 mm to (238.8, 119.4), turned to 0 degrees
- moved P17 41.3 mm to (231.1, 119.4)
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Connections:
- JACK1 pad 1: Net-(JACK1-Pad1) -> (no net)
- JACK1 pad 2: Net-(JACK1-Pad2) -> (no net)
- JACK1 pad 3: Net-(JACK1-Pad3) -> (no net)
- JACK1 pad 6: Net-(JACK1-Pad6) -> (no net)
- JACK1 pad 7: Net-(JACK1-Pad7) -> (no net)
- JACK2 pad 1: Net-(JACK2-Pad1) -> (no net)
- JACK2 pad 2: Net-(JACK2-Pad2) -> (no net)
- JACK2 pad 3: Net-(JACK2-Pad3) -> (no net)
- JACK2 pad 6: Net-(JACK2-Pad6) -> (no net)
- JACK2 pad 7: Net-(JACK2-Pad7) -> (no net)
- JACK3 pad 1: Net-(JACK3-Pad1) -> (no net)
- JACK3 pad 2: Net-(JACK3-Pad2) -> (no net)
- JACK3 pad 3: Net-(JACK3-Pad3) -> (no net)
- JACK3 pad 6: Net-(JACK3-Pad6) -> (no net)
- JACK3 pad 7: Net-(JACK3-Pad7) -> (no net)
- P38 pad 1: GND -> Net-(C46-Pad1)
- P38 pad 2: Net-(P38-Pad2) -> GND
- P38 pad 3: Net-(P38-Pad3) -> Net-(C47-Pad1)
- P38 pad 4: Net-(P38-Pad4) -> Net-(C48-Pad1)
- P38 pad 5: Net-(P38-Pad5) -> GND
- P39 pad 1: GND -> Net-(C50-Pad1)
- P39 pad 2: Net-(P39-Pad2) -> GND
- P39 pad 3: Net-(P39-Pad3) -> Net-(C51-Pad1)
- P39 pad 4: Net-(P39-Pad4) -> Net-(C52-Pad1)
- P39 pad 5: Net-(P39-Pad5) -> GND
- U11 pad 1: Net-(U11-Pad1) -> (no net)
- U11 pad 4: Net-(U11-Pad4) -> (no net)
- U11 pad 7: Net-(U11-Pad7) -> (no net)
- U12 pad 1: Net-(U12-Pad1) -> (no net)
- U12 pad 2: Net-(U12-Pad2) -> (no net)
- U12 pad 3: Net-(U12-Pad3) -> (no net)
- U12 pad 5: Net-(U12-Pad5) -> (no net)
- U12 pad 6: Net-(U12-Pad6) -> (no net)
- U12 pad 7: Net-(U12-Pad7) -> (no net)
- U13 pad 16: VDD -> (no net)
- U14 pad 16: VDD -> (no net)
- U3 pad 35: Net-(U3-Pad35) -> (no net)
- U3 pad 38: Net-(U3-Pad38) -> (no net)
- U3 pad 41: Net-(U3-Pad41) -> (no net)
- U3 pad 48: Net-(U3-Pad48) -> (no net)
- U3 pad 49: Net-(U3-Pad49) -> (no net)
- U30 pad 9: Net-(U30-Pad9) -> (no net)
- U31 pad 11: Net-(P39-Pad4) -> 3/4AOUTR
- U31 pad 12: Net-(P39-Pad5) -> 3/4AOUTL
- U31 pad 13: Net-(P39-Pad3) -> 3/4AINR
- U31 pad 14: Net-(P39-Pad2) -> 3/4AINL
- U31 pad 15: Net-(U31-Pad15) -> (no net)
- U31 pad 16: Net-(U31-Pad16) -> (no net)
- U31 pad 18: Net-(U31-Pad18) -> (no net)
- U5 pad 11: Net-(P38-Pad4) -> 1/2AOUTR
- U5 pad 12: Net-(P38-Pad5) -> 1/2AOUTL
- U5 pad 13: Net-(P38-Pad3) -> 1/2AINR
- U5 pad 14: Net-(P38-Pad2) -> 1/2AINL
- U5 pad 15: Net-(U5-Pad15) -> (no net)
- U5 pad 16: Net-(U5-Pad16) -> (no net)
- U5 pad 18: Net-(U5-Pad18) -> (no net)
- U6 pad 1: Net-(U6-Pad1) -> (no net)
- U6 pad 10: Net-(U6-Pad10) -> (no net)
- U6 pad 11: Net-(U6-Pad11) -> (no net)
- U6 pad 12: Net-(U6-Pad12) -> (no net)
- U6 pad 8: Net-(U6-Pad8) -> (no net)
- U6 pad 9: Net-(U6-Pad9) -> (no net)
- U8 pad 9: Net-(U8-Pad9) -> (no net)
- U9 pad 2: PORT-RX -> Net-(JMP18-Pad2)
Routing:
- net LED_LATCH: track 247.0 -> 28.1 mm, vias 9 -> 1
- net SPI_SCK: track 244.7 -> 32.6 mm, vias 11 -> 1
- net LED_OE: track 236.3 -> 32.9 mm, vias 9 -> 1
- net !LED_RST: track 230.0 -> 27.9 mm, vias 9 -> 0
- net +5V: track 207.6 -> 22.2 mm, vias 8 -> 0
- net EN: track 81.4 -> 0.00 mm, vias 5 -> 0
- net SPI_MOSI: track 81.1 -> 22.1 mm, vias 5 -> 1
- net (no net): track 0.00 -> 53.3 mm, vias 8 -> 1
- net KA3: track 86.8 -> 35.2 mm
- net VDD: track 51.4 -> 0.00 mm
- net KA2: track 79.5 -> 36.2 mm
- net KA1: track 81.4 -> 39.7 mm
- net SPI_MISO: track 43.1 -> 2.80 mm, vias 3 -> 0
- net KA0: track 81.2 -> 41.8 mm
- net B: track 36.7 -> 0.00 mm, vias 3 -> 0
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