File: Test Projects/Teensy_test_layout.kicad_pcb (KiCad board)
At the start: 2 copper layers, 254 x 127 mm, 231 parts, among them P1 CONN_01X02, P10 CONN_01X06, P11 CONN_01X06, P12 CONN_01X06, P13 CONN_01X08, P14 CONN_01X08, P15 CONN_01X08, P16 CONN_01X08, P17 CONN_01X08, P18 CONN_01X08, P19 CONN_01X08, P2 CONN_01X03, P20 CONN_01X08, P21 CONN_01X07, P22 CONN_01X08, P23 CONN_01X08, P24 CONN_01X08, P25 CONN_01X08, P26 CONN_01X08, P27 CONN_01X08, P28 CONN_01X08, P29 CONN_01X08, P3 COLS0, P30 CONN_01X03, P31 PIN20, P32 PIN8, P33 SIO2, P34 ~HOLD~/SIO3, P35 PIN37, P36 PIN29, P37 PIN31, P38 CONN_01X06, P39 CONN_01X06, P4 COLS1, P40 CONN_01X08, P41 CONN_01X08, P42 CONN_01X08, P43 CONN_01X08, P44 CONN_01X08, P45 CONN_01X08, P46 CONN_01X08, P47 CONN_01X08, P48 CONN_01X08, P49 CONN_01X08, P5 CONN_01X06, P50 CONN_01X08, P51 CONN_01X08, P52 CONN_01X08, P53 CONN_01X08, P54 CONN_01X08, P55 CONN_01X08, P56 CONN_01X01, P57 CONN_01X01, P58 VUU, P59 CONN_01X01, P6 CONN_01X06, P60 CONN_01X01, P61 CONN_01X01, P62 UGND, P63 CONN_01X01, P64 DIN1, P65 DOUT1, P66 SDA0, P67 SCL0, P68 MCLK, P69 BCLK, P7 CONN_01X06, P70 LRCLK, P71 DIN0, P72 DOUT0, P73 IN2TTL, P8 CONN_01X06, P9 CONN_01X06, U1 LDO-adj-4term, U10 SF-74x125, U11 2N168, U12 SF-LM358, U13 SF-4052, U14 SF-4052, U15 SF-4052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

Commit message: Routing, 15%
Parts:
- removed C18: C, Capacitors_Tantalum_SMD:TantalC_SizeB_EIA-3528_Reflow
- removed U12: SF-LM358, SparkFun-Footprints:SF-SOIC-8
- added JACK12: POWER_JACKPTH, SparkFun-Footprints:SparkFun-Connectors-POWER_JACK_PTH, F.Cu at (41.9, 25.4)
- added P74: CONN_01X08, Pin_Headers:Pin_Header_Straight_1x08, F.Cu at (129.5, 127.0)
- added P75: CONN_01X08, Pin_Headers:Pin_Header_Straight_1x08, F.Cu at (152.4, 127.0)
- added P76: CONN_01X08, Pin_Headers:Pin_Header_Straight_1x08, F.Cu at (129.5, 147.3)
- added P77: CONN_01X08, Pin_Headers:Pin_Header_Straight_1x08, F.Cu at (152.4, 147.3)
- added P78: CONN_01X08, Pin_Headers:Pin_Header_Straight_1x08, F.Cu at (175.3, 147.3)
- added P79: CONN_01X08, Pin_Headers:Pin_Header_Straight_1x08, F.Cu at (198.1, 147.3)
- added P80: CONN_01X08, Pin_Headers:Pin_Header_Straight_1x08, F.Cu at (221.0, 147.3)
- added P81: CONN_01X08, Pin_Headers:Pin_Header_Straight_1x08, F.Cu at (243.8, 147.3)
- added P82: CONN_01X01, SparkFun-Footprints:PTH_LUG_.05, F.Cu at (181.6, 101.6)
- added P83: CONN_01X01, SparkFun-Footprints:PTH_LUG_.05, F.Cu at (181.6, 121.9)
- added P84: CONN_01X01, SparkFun-Footprints:PTH_LUG_.05, F.Cu at (176.5, 97.8)
- added P85: CONN_01X01, SparkFun-Footprints:PTH_LUG_.05, F.Cu at (181.6, 106.7)
- added P86: CONN_01X01, SparkFun-Footprints:PTH_LUG_.05, F.Cu at (181.6, 127.0)
- added P87: CONN_01X01, SparkFun-Footprints:PTH_LUG_.05, F.Cu at (124.5, 147.3)
- added P88: CONN_01X01, SparkFun-Footprints:PTH_LUG_.05, F.Cu at (124.5, 127.0)
- added R31: 470, Resistors_SMD:R_0603, F.Cu at (129.5, 120.7)
- added R32: 470, Resistors_SMD:R_0603, F.Cu at (129.5, 141.0)
- added R33: 470, Resistors_SMD:R_0603, F.Cu at (132.1, 120.7)
- added R34: 470, Resistors_SMD:R_0603, F.Cu at (132.1, 141.0)
- added R35: 470, Resistors_SMD:R_0603, F.Cu at (134.6, 120.7)
- added R36: 470, Resistors_SMD:R_0603, F.Cu at (134.6, 141.0)
- added R37: 470, Resistors_SMD:R_0603, F.Cu at (137.2, 120.7)
- added R38: 470, Resistors_SMD:R_0603, F.Cu at (137.2, 141.0)
- added R39: 470, Resistors_SMD:R_0603, F.Cu at (139.7, 120.7)
- added R40: 470, Resistors_SMD:R_0603, F.Cu at (139.7, 141.0)
- added R41: 470, Resistors_SMD:R_0603, F.Cu at (142.2, 120.7)
- added R42: 470, Resistors_SMD:R_0603, F.Cu at (142.2, 141.0)
- added R43: 470, Resistors_SMD:R_0603, F.Cu at (144.8, 120.7)
- added R44: 470, Resistors_SMD:R_0603, F.Cu at (144.8, 141.0)
- added R45: 470, Resistors_SMD:R_0603, F.Cu at (147.3, 120.7)
- added R46: 470, Resistors_SMD:R_0603, F.Cu at (147.3, 141.0)
- added R47: 470, Resistors_SMD:R_0603, F.Cu at (152.4, 120.7)
- added R48: 470, Resistors_SMD:R_0603, F.Cu at (152.4, 141.0)
- added R49: 470, Resistors_SMD:R_0603, F.Cu at (154.9, 120.7)
- added R50: 470, Resistors_SMD:R_0603, F.Cu at (154.9, 141.0)
- added R51: 470, Resistors_SMD:R_0603, F.Cu at (157.5, 120.7)
- added R52: 470, Resistors_SMD:R_0603, F.Cu at (157.5, 141.0)
- added R53: 470, Resistors_SMD:R_0603, F.Cu at (160.0, 120.7)
- added R54: 470, Resistors_SMD:R_0603, F.Cu at (160.0, 141.0)
- added R55: 470, Resistors_SMD:R_0603, F.Cu at (162.6, 120.7)
- added R56: 470, Resistors_SMD:R_0603, F.Cu at (162.6, 141.0)
- added R57: 470, Resistors_SMD:R_0603, F.Cu at (165.1, 120.7)
- added R58: 470, Resistors_SMD:R_0603, F.Cu at (165.1, 141.0)
- added R59: 470, Resistors_SMD:R_0603, F.Cu at (167.6, 120.7)
- added R60: 470, Resistors_SMD:R_0603, F.Cu at (167.6, 141.0)
- added R61: 470, Resistors_SMD:R_0603, F.Cu at (170.2, 120.7)
- added R62: 470, Resistors_SMD:R_0603, F.Cu at (170.2, 141.0)
- added R63: 470, Resistors_SMD:R_0603, F.Cu at (175.3, 141.0)
- added R64: 470, Resistors_SMD:R_0603, F.Cu at (221.0, 141.0)
- added R65: 470, Resistors_SMD:R_0603, F.Cu at (177.8, 141.0)
- added R66: 470, Resistors_SMD:R_0603, F.Cu at (223.5, 141.0)
- added R67: 470, Resistors_SMD:R_0603, F.Cu at (180.3, 141.0)
- added R68: 470, Resistors_SMD:R_0603, F.Cu at (226.1, 141.0)
- added R69: 470, Resistors_SMD:R_0603, F.Cu at (182.9, 141.0)
- added R70: 470, Resistors_SMD:R_0603, F.Cu at (228.6, 141.0)
- added R71: 470, Resistors_SMD:R_0603, F.Cu at (185.4, 141.0)
- added R72: 470, Resistors_SMD:R_0603, F.Cu at (231.1, 141.0)
- added R73: 470, Resistors_SMD:R_0603, F.Cu at (188.0, 141.0)
- added R74: 470, Resistors_SMD:R_0603, F.Cu at (233.7, 141.0)
- added R75: 470, Resistors_SMD:R_0603, F.Cu at (190.5, 141.0)
- added R76: 470, Resistors_SMD:R_0603, F.Cu at (236.2, 141.0)
- added R77: 470, Resistors_SMD:R_0603, F.Cu at (193.0, 141.0)
- added R78: 470, Resistors_SMD:R_0603, F.Cu at (238.8, 141.0)
- added R79: 470, Resistors_SMD:R_0603, F.Cu at (198.1, 141.0)
- added R80: 470, Resistors_SMD:R_0603, F.Cu at (243.8, 141.0)
- added R81: 470, Resistors_SMD:R_0603, F.Cu at (200.7, 141.0)
- added R82: 470, Resistors_SMD:R_0603, F.Cu at (246.4, 141.0)
- added R83: 470, Resistors_SMD:R_0603, F.Cu at (203.2, 141.0)
- added R84: 470, Resistors_SMD:R_0603, F.Cu at (248.9, 141.0)
- added R85: 470, Resistors_SMD:R_0603, F.Cu at (205.7, 141.0)
- added R86: 470, Resistors_SMD:R_0603, F.Cu at (251.5, 141.0)
- added R87: 470, Resistors_SMD:R_0603, F.Cu at (208.3, 141.0)
- added R88: 470, Resistors_SMD:R_0603, F.Cu at (254.0, 141.0)
- added R89: 470, Resistors_SMD:R_0603, F.Cu at (210.8, 141.0)
- added R90: 470, Resistors_SMD:R_0603, F.Cu at (256.5, 141.0)
- added R91: 470, Resistors_SMD:R_0603, F.Cu at (213.4, 141.0)
- added R92: 470, Resistors_SMD:R_0603, F.Cu at (259.1, 141.0)
- added R93: 470, Resistors_SMD:R_0603, F.Cu at (215.9, 141.0)
- added R94: 470, Resistors_SMD:R_0603, F.Cu at (261.6, 141.0)
- C10, C11, C12, C13, C14, C37, C38, C39, C40, C41: value C -> 0.1uF
- moved C27 82.3 mm to (242.6, 114.3), turned to 270 degrees
- moved H4 82.3 mm to (195.6, 76.2)
- moved U21 67.6 mm to (228.6, 94.0)
- moved P71 65.2 mm to (152.4, 102.2)
- moved U16 59.3 mm to (271.8, 94.0), turned to 0 degrees
- moved P24 58.4 mm to (129.5, 144.8), turned to 90 degrees
- moved P25 50.8 mm to (152.4, 144.8), turned to 90 degrees
- moved U15 50.6 mm to (248.9, 94.0), turned to 0 degrees
- moved U17 49.8 mm to (184.2, 114.3), turned to 180 degrees
- moved P42 49.8 mm to (209.6, 121.9), turned to 90 degrees
- moved P50 49.8 mm to (209.6, 127.0), turned to 90 degrees
- moved P18 49.8 mm to (209.6, 124.5), turned to 90 degrees
- moved C21 49.7 mm to (228.6, 87.6), turned to 90 degrees
- moved C24 48.6 mm to (190.5, 114.3), turned to 90 degrees
- moved C31 48.4 mm to (134.6, 134.6), turned to 270 degrees
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Connections:
- net /page1/Bulk_IN renamed VBULK
- net Net-(C43-Pad1) renamed VUUIN
- C48 pad 2: 1/2AOUTR -> 1/2AOUTL
- C49 pad 2: 1/2AOUTL -> 1/2AOUTR
- C52 pad 2: 3/4AOUTR -> 3/4AOUTL
- C53 pad 2: 3/4AOUTL -> 3/4AOUTR
- JMP10 pad 1: 1/2AOUTL -> 1/2AOUTR
- JMP11 pad 1: 1/2AOUTR -> 1/2AOUTL
- JMP14 pad 1: 3/4AOUTL -> 3/4AOUTR
- JMP15 pad 1: 3/4AOUTR -> 3/4AOUTL
- P64 pad 1: Net-(JMP6-Pad2) -> I2S_DIN1
- P65 pad 1: Net-(JMP7-Pad2) -> I2S_DOUT1
- P71 pad 1: Net-(JMP2-Pad2) -> I2S_DIN0
- P72 pad 1: Net-(JMP3-Pad2) -> I2S_DOUT0
- U13 pad 16: (no net) -> VDD
- U14 pad 16: (no net) -> VDD
- U23 pad 1: Net-(P22-Pad2) -> Net-(R33-Pad2)
- U23 pad 15: Net-(P22-Pad1) -> Net-(R31-Pad2)
- U23 pad 2: Net-(P22-Pad3) -> Net-(R35-Pad2)
- U23 pad 3: Net-(P22-Pad4) -> Net-(R37-Pad2)
- U23 pad 4: Net-(P22-Pad5) -> Net-(R39-Pad2)
- U23 pad 5: Net-(P22-Pad6) -> Net-(R41-Pad2)
- U23 pad 6: Net-(P22-Pad7) -> Net-(R43-Pad2)
- U23 pad 7: Net-(P22-Pad8) -> Net-(R45-Pad2)
- U24 pad 1: Net-(P23-Pad2) -> Net-(R49-Pad2)
- U24 pad 15: Net-(P23-Pad1) -> Net-(R47-Pad2)
- U24 pad 2: Net-(P23-Pad3) -> Net-(R51-Pad2)
- U24 pad 3: Net-(P23-Pad4) -> Net-(R53-Pad2)
- U24 pad 4: Net-(P23-Pad5) -> Net-(R55-Pad2)
- U24 pad 5: Net-(P23-Pad6) -> Net-(R57-Pad2)
- U24 pad 6: Net-(P23-Pad7) -> Net-(R59-Pad2)
- U24 pad 7: Net-(P23-Pad8) -> Net-(R61-Pad2)
- U25 pad 1: Net-(P24-Pad2) -> Net-(R34-Pad2)
- U25 pad 15: Net-(P24-Pad1) -> Net-(R32-Pad2)
- U25 pad 2: Net-(P24-Pad3) -> Net-(R36-Pad2)
- U25 pad 3: Net-(P24-Pad4) -> Net-(R38-Pad2)
- U25 pad 4: Net-(P24-Pad5) -> Net-(R40-Pad2)
- U25 pad 5: Net-(P24-Pad6) -> Net-(R42-Pad2)
- U25 pad 6: Net-(P24-Pad7) -> Net-(R44-Pad2)
- U25 pad 7: Net-(P24-Pad8) -> Net-(R46-Pad2)
- U26 pad 1: Net-(P25-Pad2) -> Net-(R50-Pad2)
- U26 pad 15: Net-(P25-Pad1) -> Net-(R48-Pad2)
- U26 pad 2: Net-(P25-Pad3) -> Net-(R52-Pad2)
- U26 pad 3: Net-(P25-Pad4) -> Net-(R54-Pad2)
- U26 pad 4: Net-(P25-Pad5) -> Net-(R56-Pad2)
- U26 pad 5: Net-(P25-Pad6) -> Net-(R58-Pad2)
- U26 pad 6: Net-(P25-Pad7) -> Net-(R60-Pad2)
- U26 pad 7: Net-(P25-Pad8) -> Net-(R62-Pad2)
- U27 pad 1: Net-(P26-Pad2) -> Net-(R65-Pad2)
- U27 pad 15: Net-(P26-Pad1) -> Net-(R63-Pad2)
- U27 pad 2: Net-(P26-Pad3) -> Net-(R67-Pad2)
- U27 pad 3: Net-(P26-Pad4) -> Net-(R69-Pad2)
- U27 pad 4: Net-(P26-Pad5) -> Net-(R71-Pad2)
- U27 pad 5: Net-(P26-Pad6) -> Net-(R73-Pad2)
- U27 pad 6: Net-(P26-Pad7) -> Net-(R75-Pad2)
- U27 pad 7: Net-(P26-Pad8) -> Net-(R77-Pad2)
- U28 pad 1: Net-(P27-Pad2) -> Net-(R81-Pad2)
- U28 pad 15: Net-(P27-Pad1) -> Net-(R79-Pad2)
- U28 pad 2: Net-(P27-Pad3) -> Net-(R83-Pad2)
- U28 pad 3: Net-(P27-Pad4) -> Net-(R85-Pad2)
- U28 pad 4: Net-(P27-Pad5) -> Net-(R87-Pad2)
- U28 pad 5: Net-(P27-Pad6) -> Net-(R89-Pad2)
- U28 pad 6: Net-(P27-Pad7) -> Net-(R91-Pad2)
- U28 pad 7: Net-(P27-Pad8) -> Net-(R93-Pad2)
- U29 pad 1: Net-(P28-Pad2) -> Net-(R66-Pad2)
- U29 pad 15: Net-(P28-Pad1) -> Net-(R64-Pad2)
- U29 pad 2: Net-(P28-Pad3) -> Net-(R68-Pad2)
- U29 pad 3: Net-(P28-Pad4) -> Net-(R70-Pad2)
- U29 pad 4: Net-(P28-Pad5) -> Net-(R72-Pad2)
- U29 pad 5: Net-(P28-Pad6) -> Net-(R74-Pad2)
- U29 pad 6: Net-(P28-Pad7) -> Net-(R76-Pad2)
- U29 pad 7: Net-(P28-Pad8) -> Net-(R78-Pad2)
- U30 pad 1: Net-(P29-Pad2) -> Net-(R82-Pad2)
- U30 pad 15: Net-(P29-Pad1) -> Net-(R80-Pad2)
- U30 pad 2: Net-(P29-Pad3) -> Net-(R84-Pad2)
- U30 pad 3: Net-(P29-Pad4) -> Net-(R86-Pad2)
- U30 pad 4: Net-(P29-Pad5) -> Net-(R88-Pad2)
- U30 pad 5: Net-(P29-Pad6) -> Net-(R90-Pad2)
- U30 pad 6: Net-(P29-Pad7) -> Net-(R92-Pad2)
- U30 pad 7: Net-(P29-Pad8) -> Net-(R94-Pad2)
Routing:
- net SPI_SCK: track 32.6 -> 394.6 mm, vias 1 -> 14
- net LED_LATCH: track 28.1 -> 301.6 mm, vias 1 -> 10
- net !LED_RST: track 27.9 -> 299.1 mm, vias 0 -> 9
- net LED_OE: track 32.9 -> 298.6 mm, vias 1 -> 10
- net +5V: track 22.2 -> 242.1 mm, vias 0 -> 8
- net LED_BUS: track 0.00 -> 182.9 mm
- net SPI_MOSI: track 22.1 -> 112.9 mm, vias 1 -> 4
- net Net-(U24-Pad9): track 0.00 -> 62.9 mm, vias 0 -> 2
- net +3V3: track 53.6 -> 10.8 mm, vias 2 -> 0
- net ROW4: track 15.5 -> 52.9 mm
- net (no net): track 53.3 -> 18.0 mm, vias 1 -> 4
- net ROW3: track 14.9 -> 48.6 mm
- net ROW1: track 10.2 -> 41.6 mm
- net SPI_MISO: track 2.80 -> 33.8 mm, vias 0 -> 1
- net ROW2: track 13.2 -> 44.0 mm
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Other:
- board text added: "IN"
- board text added: "OUT"
- board text added: "R"
- board text added: "RN"
- board text added: "S"
- board text added: "SN"
- board text added: "T"
- board text added: "THRU"
- board text added: "TN"

Commit message: layout
Routing:
- net (no net): track 18.0 -> 0.00 mm, vias 4 -> 1
- net Net-(P30-Pad3): track 1.33 -> 10.4 mm, vias 0 -> 2
- net Net-(P30-Pad1): track 1.19 -> 10.1 mm, vias 1 -> 2
- net GND: track 27.3 -> 24.6 mm
- net +5V: track 242.1 -> 239.8 mm
- net Net-(C37-Pad1): track 2.90 -> 4.55 mm
- net Net-(C40-Pad1): track 6.64 -> 7.77 mm

Commit message: more layout
Parts:
- added P89: CONN_01X04, Pin_Headers:Pin_Header_Straight_1x04, F.Cu at (161.3, 104.2)
- P21: value CONN_01X07 -> CONN_01X05; footprint Pin_Headers:Pin_Header_Straight_1x07 -> Pin_Headers:Pin_Header_Straight_1x05
- moved P21 66.3 mm to (109.2, 110.5)
- moved P72 58.2 mm to (147.3, 100.3)
- moved P66 34.5 mm to (119.4, 97.8)
- moved P64 32.8 mm to (124.5, 100.3)
- moved P68 27.9 mm to (114.3, 90.2)
- moved P69 23.2 mm to (114.3, 95.2)
- moved P70 21.2 mm to (114.3, 92.7)
- moved R8 13.8 mm to (117.6, 94.2)
- moved R9 13.8 mm to (120.2, 94.2)
- moved P67 13.0 mm to (116.8, 97.8)
- moved JMP20 12.5 mm to (63.5, 48.9)
- moved C19 10.1 mm to (190.6, 93.5), turned to 90 degrees
- moved C54 10.0 mm to (68.6, 50.2), turned to 180 degrees
- moved U34 9.25 mm to (71.1, 57.1)
- moved JMP18 9.18 mm to (98.4, 57.8)
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Connections:
- U21 pad 10: A -> C
- U21 pad 9: B -> D
- U22 pad 10: A -> C
- U22 pad 9: B -> D
- U3 pad 27: KA -> (no net)
- U3 pad 28: KB -> (no net)
Routing:
- net VDD: track 0.00 -> 346.7 mm, vias 0 -> 22
- net B: track 0.00 -> 271.8 mm, vias 0 -> 8
- net A: track 0.00 -> 271.7 mm, vias 0 -> 8
- net EN: track 0.00 -> 260.7 mm, vias 0 -> 10
- net KA1: track 39.7 -> 233.2 mm, vias 0 -> 6
- net VKK: track 0.15 -> 184.3 mm
- net KGND: track 0.15 -> 183.0 mm
- net KA0: track 41.8 -> 202.8 mm, vias 2 -> 7
- net KA3: track 35.2 -> 161.6 mm, vias 0 -> 3
- net KA2: track 36.2 -> 146.4 mm, vias 0 -> 3
- net +5V: track 239.8 -> 341.4 mm, vias 8 -> 12
- net C: track 0.00 -> 99.9 mm, vias 0 -> 3
- net D: track 0.00 -> 94.7 mm, vias 0 -> 2
- net SCL0: track 0.00 -> 80.6 mm, vias 0 -> 2
- net SDA0: track 0.00 -> 80.2 mm, vias 0 -> 2
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
Commit message: moar layout
Parts:
- added JMP21: 2Jumper, SparkFun-Footprints:SF-2way-open, F.Cu at (172.9, 88.3)
- added JMP22: 2Jumper, SparkFun-Footprints:SF-2way-open, F.Cu at (118.1, 101.0)
- added JMP23: 2Jumper, SparkFun-Footprints:SF-2way-open, F.Cu at (118.1, 98.4)
- added JMP24: 2Jumper, SparkFun-Footprints:SF-2way-open, F.Cu at (112.4, 90.2)
- added JMP25: 2Jumper, SparkFun-Footprints:SF-2way-open, F.Cu at (112.4, 95.2)
- added JMP26: 2Jumper, SparkFun-Footprints:SF-2way-open, F.Cu at (112.4, 92.7)
- added P90: CONN_01X01, Pin_Headers:Pin_Header_Straight_1x01, F.Cu at (45.1, 44.5)
- added P91: SDA0, SparkFun-Footprints:TestHole, F.Cu at (116.2, 101.0)
- added P92: SCL0, SparkFun-Footprints:TestHole, F.Cu at (116.2, 98.4)
- added P93: MCLK, SparkFun-Footprints:TestHole, F.Cu at (110.5, 90.2)
- added P94: BCLK, SparkFun-Footprints:TestHole, F.Cu at (110.5, 95.2)
- added P95: LRCLK, SparkFun-Footprints:TestHole, F.Cu at (110.5, 92.7)
- added P96: DIN1_ISO, SparkFun-Footprints:TestHole, F.Cu at (127.0, 99.7)
- added P97: DOUT1_ISO, SparkFun-Footprints:TestHole, F.Cu at (124.5, 99.7)
- added P98: DIN0_ISO, SparkFun-Footprints:TestHole, F.Cu at (152.4, 99.7)
- added P99: DOUT0_ISO, SparkFun-Footprints:TestHole, F.Cu at (149.9, 99.7)
- P66: value SDA0 -> SDA0_ISO
- P67: value SCL0 -> SCL0_ISO
- P68: value MCLK -> MCLK_ISO
- P69: value BCLK -> BCLK_ISO
- P70: value LRCLK -> LRCLK_ISO
- moved JMP1 38.6 mm to (57.1, 79.4), turned to 90 degrees
- moved P82 22.9 mm to (182.9, 121.9)
- moved P83 22.9 mm to (182.9, 99.1)
- moved P85 22.9 mm to (182.9, 127.0)
- moved P86 22.9 mm to (182.9, 104.1)
- moved P60 18.1 mm to (33.0, 106.7)
- moved P62 17.7 mm to (30.5, 106.7)
- moved P59 14.5 mm to (35.6, 106.7)
- moved P61 14.5 mm to (38.1, 106.7)
- moved P57 7.73 mm to (45.7, 106.7)
- moved P56 7.10 mm to (48.3, 106.7)
- moved P58 6.48 mm to (50.8, 106.7)
- moved P72 6.25 mm to (149.9, 106.0)
- moved P64 6.25 mm to (127.0, 106.0)
- moved P65 6.25 mm to (124.5, 106.0)
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Connections:
- net Net-(JMP2-Pad2) renamed I2S_DIN0_ISO
- net Net-(JMP3-Pad2) renamed I2S_DOUT0_ISO
- net Net-(JMP6-Pad2) renamed I2S_DIN1_ISO
- net Net-(JMP7-Pad2) renamed I2S_DOUT1_ISO
- JACK1 pad 1: (no net) -> Net-(JACK1-Pad1)
- JACK1 pad 2: (no net) -> Net-(JACK1-Pad2)
- JACK1 pad 3: (no net) -> Net-(JACK1-Pad3)
- JACK1 pad 6: (no net) -> Net-(JACK1-Pad6)
- JACK1 pad 7: (no net) -> Net-(JACK1-Pad7)
- JACK12 pad GNDB: (no net) -> Net-(JACK12-PadGNDB)
- JACK2 pad 1: (no net) -> Net-(JACK2-Pad1)
- JACK2 pad 2: (no net) -> Net-(JACK2-Pad2)
- JACK2 pad 3: (no net) -> Net-(JACK2-Pad3)
- JACK2 pad 6: (no net) -> Net-(JACK2-Pad6)
- JACK2 pad 7: (no net) -> Net-(JACK2-Pad7)
- JACK3 pad 1: (no net) -> Net-(JACK3-Pad1)
- JACK3 pad 2: (no net) -> Net-(JACK3-Pad2)
- JACK3 pad 3: (no net) -> Net-(JACK3-Pad3)
- JACK3 pad 6: (no net) -> Net-(JACK3-Pad6)
- JACK3 pad 7: (no net) -> Net-(JACK3-Pad7)
- P44 pad 1: VKK -> VKK2
- P44 pad 2: VKK -> VKK2
- P44 pad 3: VKK -> VKK2
- P44 pad 4: VKK -> VKK2
- P44 pad 5: VKK -> VKK2
- P44 pad 6: VKK -> VKK2
- P44 pad 7: VKK -> VKK2
- P44 pad 8: VKK -> VKK2
- P45 pad 1: VKK -> VKK2
- P45 pad 2: VKK -> VKK2
- P45 pad 3: VKK -> VKK2
- P45 pad 4: VKK -> VKK2
- P45 pad 5: VKK -> VKK2
- P45 pad 6: VKK -> VKK2
- P45 pad 7: VKK -> VKK2
- P45 pad 8: VKK -> VKK2
- P46 pad 1: VKK -> VKK2
- P46 pad 2: VKK -> VKK2
- P46 pad 3: VKK -> VKK2
- P46 pad 4: VKK -> VKK2
- P46 pad 5: VKK -> VKK2
- P46 pad 6: VKK -> VKK2
- P46 pad 7: VKK -> VKK2
- P46 pad 8: VKK -> VKK2
- P47 pad 1: VKK -> VKK2
- P47 pad 2: VKK -> VKK2
- P47 pad 3: VKK -> VKK2
- P47 pad 4: VKK -> VKK2
- P47 pad 5: VKK -> VKK2
- P47 pad 6: VKK -> VKK2
- P47 pad 7: VKK -> VKK2
- P47 pad 8: VKK -> VKK2
- P52 pad 1: KGND -> KGND2
- P52 pad 2: KGND -> KGND2
- P52 pad 3: KGND -> KGND2
- P52 pad 4: KGND -> KGND2
- P52 pad 5: KGND -> KGND2
- P52 pad 6: KGND -> KGND2
- P52 pad 7: KGND -> KGND2
- P52 pad 8: KGND -> KGND2
- P53 pad 1: KGND -> KGND2
- P53 pad 2: KGND -> KGND2
- P53 pad 3: KGND -> KGND2
- P53 pad 4: KGND -> KGND2
- P53 pad 5: KGND -> KGND2
- P53 pad 6: KGND -> KGND2
- P53 pad 7: KGND -> KGND2
- P53 pad 8: KGND -> KGND2
- P54 pad 1: KGND -> KGND2
- P54 pad 2: KGND -> KGND2
- P54 pad 3: KGND -> KGND2
- P54 pad 4: KGND -> KGND2
- P54 pad 5: KGND -> KGND2
- P54 pad 6: KGND -> KGND2
- P54 pad 7: KGND -> KGND2
- P54 pad 8: KGND -> KGND2
- P55 pad 1: KGND -> KGND2
- P55 pad 2: KGND -> KGND2
- P55 pad 3: KGND -> KGND2
- P55 pad 4: KGND -> KGND2
- P55 pad 5: KGND -> KGND2
- P55 pad 6: KGND -> KGND2
- P55 pad 7: KGND -> KGND2
- P55 pad 8: KGND -> KGND2
- P66 pad 1: SDA0 -> SDA_ISO
- P67 pad 1: SCL0 -> SCL_ISO
- P68 pad 1: I2S_MCLK -> MCLK_ISO
- P69 pad 1: I2S_BCLK -> BCLK_ISO
- P70 pad 1: I2S_LRCLK -> LRCLK_ISO
- P83 pad 1: VKK -> VKK2
- P86 pad 1: KGND -> KGND2
- U11 pad 1: (no net) -> Net-(U11-Pad1)
- U11 pad 4: (no net) -> Net-(U11-Pad4)
- U11 pad 7: (no net) -> Net-(U11-Pad7)
- U3 pad 20: Net-(P31-Pad1) -> D
- U3 pad 27: (no net) -> A
- U3 pad 28: (no net) -> B
- U3 pad 29: Net-(P36-Pad1) -> C
- U3 pad 35: (no net) -> Net-(U3-Pad35)
- U3 pad 38: (no net) -> Net-(U3-Pad38)
- U3 pad 41: (no net) -> Net-(U3-Pad41)
- U3 pad 48: (no net) -> Net-(U3-Pad48)
- U3 pad 49: (no net) -> Net-(U3-Pad49)
- U30 pad 9: (no net) -> Net-(U30-Pad9)
- U31 pad 15: (no net) -> Net-(U31-Pad15)
- U31 pad 16: (no net) -> Net-(U31-Pad16)
- U31 pad 18: (no net) -> Net-(U31-Pad18)
- U31 pad 21: I2S_MCLK -> MCLK_ISO
- U31 pad 23: I2S_LRCLK -> LRCLK_ISO
- U31 pad 24: I2S_BCLK -> BCLK_ISO
- U31 pad 27: SDA0 -> SDA_ISO
- U31 pad 29: SCL0 -> SCL_ISO
- U34 pad 1: (no net) -> Net-(U34-Pad1)
- U34 pad 4: (no net) -> Net-(U34-Pad4)
- U34 pad 7: (no net) -> Net-(U34-Pad7)
- U5 pad 15: (no net) -> Net-(U5-Pad15)
- U5 pad 16: (no net) -> Net-(U5-Pad16)
- U5 pad 18: (no net) -> Net-(U5-Pad18)
- U5 pad 21: I2S_MCLK -> MCLK_ISO
- U5 pad 23: I2S_LRCLK -> LRCLK_ISO
- U5 pad 24: I2S_BCLK -> BCLK_ISO
- U5 pad 27: SDA0 -> SDA_ISO
- U5 pad 29: SCL0 -> SCL_ISO
- U6 pad 1: (no net) -> Net-(U6-Pad1)
- U6 pad 10: (no net) -> Net-(U6-Pad10)
- U6 pad 11: (no net) -> Net-(U6-Pad11)
- U6 pad 12: (no net) -> Net-(U6-Pad12)
- U6 pad 8: (no net) -> Net-(U6-Pad8)
- U6 pad 9: (no net) -> Net-(U6-Pad9)
- U8 pad 9: (no net) -> Net-(U8-Pad9)
Routing:
- net VKK: track 184.3 -> 91.4 mm
- net KGND: track 183.0 -> 90.2 mm
- net VKK2: track 0.00 -> 90.3 mm
- net KGND2: track 0.00 -> 90.3 mm
- net SCL0: track 80.6 -> 5.52 mm, vias 2 -> 1
- net +1V8: track 72.5 -> 147.0 mm, vias 2 -> 3
- net SDA0: track 80.2 -> 9.27 mm, vias 2 -> 1
- net I2S_BCLK: track 72.3 -> 1.50 mm, vias 2 -> 0
- net I2S_LRCLK: track 72.2 -> 1.50 mm, vias 2 -> 0
- net I2S_MCLK: track 71.6 -> 1.50 mm, vias 2 -> 0
- net +3V3: track 89.4 -> 148.4 mm, vias 4 -> 5
- net VBULK: track 20.3 -> 77.2 mm, vias 0 -> 3
- net SDA_ISO: track 0.00 -> 49.2 mm, vias 0 -> 2
- net SCL_ISO: track 0.00 -> 49.1 mm, vias 0 -> 2
- net BCLK_ISO: track 0.00 -> 48.6 mm, vias 0 -> 2
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- added copper zone on F.Cu, net +1V8
- added copper zone on F.Cu, net +3V3_REG
- added copper zone on F.Cu, net +5V
- added copper zone on B.Cu, net UGND
- added copper zone on F.Cu, net UGND
- added copper zone on F.Cu, net VUU

Commit message: layout
Parts:
- added JMP27: 2Jumper, SparkFun-Footprints:SF-2way-open, F.Cu at (161.5, 98.8)
- added JMP28: 2Jumper, SparkFun-Footprints:SF-2way-open, F.Cu at (136.1, 98.8)
- added P100: SPI_MOSI, SparkFun-Footprints:TestHole, F.Cu at (83.8, 127.0)
- added P101: SPI_MISO, SparkFun-Footprints:TestHole, F.Cu at (88.9, 127.0)
- added P102: SPI_SCK, SparkFun-Footprints:TestHole, F.Cu at (91.4, 127.0)
- added REF**: SVIA, SparkFun-Footprints:SVIA, F.Cu at (276.9, 27.9)
- added REF**: SVIA, SparkFun-Footprints:SVIA, F.Cu at (182.9, 27.9)
- added REF**: SVIA, SparkFun-Footprints:SVIA, F.Cu at (172.7, 27.9)
- added REF**: SVIA, SparkFun-Footprints:SVIA, F.Cu at (162.6, 27.9)
- added REF**: SVIA, SparkFun-Footprints:SVIA, F.Cu at (152.4, 27.9)
- added REF**: SVIA, SparkFun-Footprints:SVIA, F.Cu at (142.2, 27.9)
- added REF**: SVIA, SparkFun-Footprints:SVIA, F.Cu at (132.1, 27.9)
- added REF**: SVIA, SparkFun-Footprints:SVIA, F.Cu at (121.9, 27.9)
- added REF**: SVIA, SparkFun-Footprints:SVIA, F.Cu at (88.9, 27.9)
- added REF**: SVIA, SparkFun-Footprints:SVIA, F.Cu at (111.8, 27.9)
- added REF**: SVIA, SparkFun-Footprints:SVIA, F.Cu at (99.1, 27.9)
- added REF**: SVIA, SparkFun-Footprints:SVIA, F.Cu at (264.2, 27.9)
- added REF**: SVIA, SparkFun-Footprints:SVIA, F.Cu at (68.6, 27.9)
- added REF**: SVIA, SparkFun-Footprints:SVIA, F.Cu at (78.7, 27.9)
- added REF**: SVIA, SparkFun-Footprints:SVIA, F.Cu at (58.4, 27.9)
- added REF**: SVIA, SparkFun-Footprints:SVIA, F.Cu at (45.7, 27.9)
- added REF**: SVIA, SparkFun-Footprints:SVIA, F.Cu at (167.1, 89.2)
- added REF**: SVIA, SparkFun-Footprints:SVIA, F.Cu at (160.5, 97.3)
- added REF**: SVIA, SparkFun-Footprints:SVIA, F.Cu at (159.4, 90.8)
- added REF**: SVIA, SparkFun-Footprints:SVIA, F.Cu at (153.7, 90.8)
- added REF**: SVIA, SparkFun-Footprints:SVIA, F.Cu at (160.0, 87.4)
- added REF**: SVIA, SparkFun-Footprints:SVIA, F.Cu at (164.8, 87.6)
- added REF**: SVIA, SparkFun-Footprints:SVIA, F.Cu at (254.0, 27.9)
- added REF**: SVIA, SparkFun-Footprints:SVIA, F.Cu at (156.8, 87.6)
- added REF**: SVIA, SparkFun-Footprints:SVIA, F.Cu at (154.9, 88.3)
- added REF**: SVIA, SparkFun-Footprints:SVIA, F.Cu at (163.2, 94.0)
- added REF**: SVIA, SparkFun-Footprints:SVIA, F.Cu at (169.5, 94.6)
- added REF**: SVIA, SparkFun-Footprints:SVIA, F.Cu at (169.5, 87.6)
- added REF**: SVIA, SparkFun-Footprints:SVIA, F.Cu at (169.5, 80.6)
- added REF**: SVIA, SparkFun-Footprints:SVIA, F.Cu at (169.5, 74.3)
- added REF**: SVIA, SparkFun-Footprints:SVIA, F.Cu at (161.3, 74.3)
- added REF**: SVIA, SparkFun-Footprints:SVIA, F.Cu at (150.5, 74.3)
- added REF**: SVIA, SparkFun-Footprints:SVIA, F.Cu at (150.5, 80.6)
- added REF**: SVIA, SparkFun-Footprints:SVIA, F.Cu at (243.8, 27.9)
- added REF**: SVIA, SparkFun-Footprints:SVIA, F.Cu at (150.5, 90.8)
- added REF**: SVIA, SparkFun-Footprints:SVIA, F.Cu at (139.7, 88.3)
- added REF**: SVIA, SparkFun-Footprints:SVIA, F.Cu at (129.5, 88.3)
- added REF**: SVIA, SparkFun-Footprints:SVIA, F.Cu at (131.4, 87.6)
- added REF**: SVIA, SparkFun-Footprints:SVIA, F.Cu at (134.6, 87.0)
- added REF**: SVIA, SparkFun-Footprints:SVIA, F.Cu at (137.2, 87.6)
- added REF**: SVIA, SparkFun-Footprints:SVIA, F.Cu at (144.1, 87.0)
- added REF**: SVIA, SparkFun-Footprints:SVIA, F.Cu at (144.1, 80.6)
- added REF**: SVIA, SparkFun-Footprints:SVIA, F.Cu at (144.1, 94.6)
- added REF**: SVIA, SparkFun-Footprints:SVIA, F.Cu at (138.4, 94.0)
- added REF**: SVIA, SparkFun-Footprints:SVIA, F.Cu at (233.7, 27.9)
- added REF**: SVIA, SparkFun-Footprints:SVIA, F.Cu at (134.0, 96.5)
- added REF**: SVIA, SparkFun-Footprints:SVIA, F.Cu at (134.0, 90.8)
- added REF**: SVIA, SparkFun-Footprints:SVIA, F.Cu at (128.9, 90.8)
- added REF**: SVIA, SparkFun-Footprints:SVIA, F.Cu at (125.1, 90.8)
- added REF**: SVIA, SparkFun-Footprints:SVIA, F.Cu at (125.1, 81.3)
- added REF**: SVIA, SparkFun-Footprints:SVIA, F.Cu at (125.1, 74.3)
- added REF**: SVIA, SparkFun-Footprints:SVIA, F.Cu at (135.9, 74.3)
- added REF**: SVIA, SparkFun-Footprints:SVIA, F.Cu at (144.1, 74.3)
- added REF**: SVIA, SparkFun-Footprints:SVIA, F.Cu at (139.7, 75.6)
- added REF**: SVIA, SparkFun-Footprints:SVIA, F.Cu at (132.1, 75.6)
- added REF**: SVIA, SparkFun-Footprints:SVIA, F.Cu at (223.5, 27.9)
- added REF**: SVIA, SparkFun-Footprints:SVIA, F.Cu at (125.1, 87.0)
- added REF**: SVIA, SparkFun-Footprints:SVIA, F.Cu at (150.5, 87.0)
- added REF**: SVIA, SparkFun-Footprints:SVIA, F.Cu at (27.9, 27.9)
- added REF**: SVIA, SparkFun-Footprints:SVIA, F.Cu at (213.4, 27.9)
- added REF**: SVIA, SparkFun-Footprints:SVIA, F.Cu at (203.2, 27.9)
- added REF**: SVIA, SparkFun-Footprints:SVIA, F.Cu at (193.0, 27.9)
- added REF**1101: Single PTH, SparkFun-Footprints:proto, F.Cu at (38.1, 119.4)
- added REF**1101: Single PTH, SparkFun-Footprints:proto, F.Cu at (221.0, 78.7)
- added REF**1101: Single PTH, SparkFun-Footprints:proto, F.Cu at (205.7, 78.7)
- added REF**1101: Single PTH, SparkFun-Footprints:proto, F.Cu at (175.3, 78.7)
- added REF**1101: Single PTH, SparkFun-Footprints:proto, F.Cu at (190.5, 78.7)
- added REF**1101: Single PTH, SparkFun-Footprints:proto, F.Cu at (251.5, 78.7)
- added REF**1101: Single PTH, SparkFun-Footprints:proto, F.Cu at (236.2, 78.7)
- added REF**1101: Single PTH, SparkFun-Footprints:proto, F.Cu at (266.7, 73.7)
- added REF**1101: Single PTH, SparkFun-Footprints:proto, F.Cu at (221.0, 73.7)
- added REF**1101: Single PTH, SparkFun-Footprints:proto, F.Cu at (205.7, 73.7)
- added REF**1101: Single PTH, SparkFun-Footprints:proto, F.Cu at (175.3, 73.7)
- added REF**1101: Single PTH, SparkFun-Footprints:proto, F.Cu at (106.7, 124.5)
- added REF**1101: Single PTH, SparkFun-Footprints:proto, F.Cu at (190.5, 73.7)
- added REF**1101: Single PTH, SparkFun-Footprints:proto, F.Cu at (251.5, 73.7)
- added REF**1101: Single PTH, SparkFun-Footprints:proto, F.Cu at (236.2, 73.7)
- added REF**1101: Single PTH, SparkFun-Footprints:proto, F.Cu at (221.0, 58.4)
- added REF**1101: Single PTH, SparkFun-Footprints:proto, F.Cu at (205.7, 58.4)
- added REF**1101: Single PTH, SparkFun-Footprints:proto, F.Cu at (266.7, 58.4)
- added REF**1101: Single PTH, SparkFun-Footprints:proto, F.Cu at (251.5, 58.4)
- added REF**1101: Single PTH, SparkFun-Footprints:proto, F.Cu at (236.2, 58.4)
- added REF**1101: Single PTH, SparkFun-Footprints:proto, F.Cu at (190.5, 58.4)
- added REF**1101: Single PTH, SparkFun-Footprints:proto, F.Cu at (175.3, 58.4)
- added REF**1101: Single PTH, SparkFun-Footprints:proto, F.Cu at (96.5, 124.5)
- added REF**1101: Single PTH, SparkFun-Footprints:proto, F.Cu at (129.5, 58.4)
- added REF**1101: Single PTH, SparkFun-Footprints:proto, F.Cu at (160.0, 58.4)
- added REF**1101: Single PTH, SparkFun-Footprints:proto, F.Cu at (144.8, 58.4)
- added REF**1101: Single PTH, SparkFun-Footprints:proto, F.Cu at (221.0, 63.5)
- added REF**1101: Single PTH, SparkFun-Footprints:proto, F.Cu at (205.7, 63.5)
- added REF**1101: Single PTH, SparkFun-Footprints:proto, F.Cu at (266.7, 63.5)
- added REF**1101: Single PTH, SparkFun-Footprints:proto, F.Cu at (251.5, 63.5)
- added REF**1101: Single PTH, SparkFun-Footprints:proto, F.Cu at (236.2, 63.5)
- added REF**1101: Single PTH, SparkFun-Footprints:proto, F.Cu at (190.5, 63.5)
- added REF**1101: Single PTH, SparkFun-Footprints:proto, F.Cu at (175.3, 63.5)
- added REF**1101: Single PTH, SparkFun-Footprints:proto, F.Cu at (43.2, 119.4)
- added REF**1101: Single PTH, SparkFun-Footprints:proto, F.Cu at (129.5, 63.5)
- added REF**1101: Single PTH, SparkFun-Footprints:proto, F.Cu at (160.0, 63.5)
- added REF**1101: Single PTH, SparkFun-Footprints:proto, F.Cu at (144.8, 63.5)
- added REF**1101: Single PTH, SparkFun-Footprints:proto, F.Cu at (266.7, 68.6)
- added REF**1101: Single PTH, SparkFun-Footprints:proto, F.Cu at (251.5, 68.6)
- added REF**1101: Single PTH, SparkFun-Footprints:proto, F.Cu at (236.2, 68.6)
- added REF**1101: Single PTH, SparkFun-Footprints:proto, F.Cu at (221.0, 68.6)
- added REF**1101: Single PTH, SparkFun-Footprints:proto, F.Cu at (205.7, 68.6)
- added REF**1101: Single PTH, SparkFun-Footprints:proto, F.Cu at (190.5, 68.6)
- added REF**1101: Single PTH, SparkFun-Footprints:proto, F.Cu at (175.3, 68.6)
- added REF**1101: Single PTH, SparkFun-Footprints:proto, F.Cu at (78.7, 66.0)
- added REF**1101: Single PTH, SparkFun-Footprints:proto, F.Cu at (160.0, 68.6)
- added REF**1101: Single PTH, SparkFun-Footprints:proto, F.Cu at (144.8, 68.6)
- added REF**1101: Single PTH, SparkFun-Footprints:proto, F.Cu at (129.5, 68.6)
- added REF**1101: Single PTH, SparkFun-Footprints:proto, F.Cu at (114.3, 68.6)
- added REF**1101: Single PTH, SparkFun-Footprints:proto, F.Cu at (99.1, 68.6)
- added REF**1101: Single PTH, SparkFun-Footprints:proto, F.Cu at (99.1, 63.5)
- added REF**1101: Single PTH, SparkFun-Footprints:proto, F.Cu at (111.8, 63.5)
- added REF**1101: Single PTH, SparkFun-Footprints:proto, F.Cu at (111.8, 58.4)
- added REF**1101: Single PTH, SparkFun-Footprints:proto, F.Cu at (266.7, 78.7)
- added REF**1102: Single PTH, SparkFun-Footprints:proto, F.Cu at (43.2, 114.3)
- added REF**1102: Single PTH, SparkFun-Footprints:proto, F.Cu at (96.5, 121.9)
- added REF**1102: Single PTH, SparkFun-Footprints:proto, F.Cu at (43.2, 116.8)
- added REF**1102: Single PTH, SparkFun-Footprints:proto, F.Cu at (43.2, 121.9)
- added REF**1102: Single PTH, SparkFun-Footprints:proto, F.Cu at (86.4, 66.0)
- added REF**1102: Single PTH, SparkFun-Footprints:proto, F.Cu at (99.1, 66.0)
- added REF**1102: Single PTH, SparkFun-Footprints:proto, F.Cu at (111.8, 66.0)
- added REF**1102: Single PTH, SparkFun-Footprints:proto, F.Cu at (111.8, 61.0)
- added REF**1102: Single PTH, SparkFun-Footprints:proto, F.Cu at (266.7, 81.3)
- added REF**1102: Single PTH, SparkFun-Footprints:proto, F.Cu at (221.0, 81.3)
- added REF**1102: Single PTH, SparkFun-Footprints:proto, F.Cu at (205.7, 81.3)
- added REF**1102: Single PTH, SparkFun-Footprints:proto, F.Cu at (38.1, 114.3)
- added REF**1102: Single PTH, SparkFun-Footprints:proto, F.Cu at (175.3, 81.3)
- added REF**1102: Single PTH, SparkFun-Footprints:proto, F.Cu at (190.5, 81.3)
- added REF**1102: Single PTH, SparkFun-Footprints:proto, F.Cu at (251.5, 81.3)
- added REF**1102: Single PTH, SparkFun-Footprints:proto, F.Cu at (236.2, 81.3)
- added REF**1102: Single PTH, SparkFun-Footprints:proto, F.Cu at (266.7, 76.2)
- added REF**1102: Single PTH, SparkFun-Footprints:proto, F.Cu at (221.0, 76.2)
- added REF**1102: Single PTH, SparkFun-Footprints:proto, F.Cu at (205.7, 76.2)
- added REF**1102: Single PTH, SparkFun-Footprints:proto, F.Cu at (175.3, 76.2)
- added REF**1102: Single PTH, SparkFun-Footprints:proto, F.Cu at (190.5, 76.2)
- added REF**1102: Single PTH, SparkFun-Footprints:proto, F.Cu at (251.5, 76.2)
- added REF**1102: Single PTH, SparkFun-Footprints:proto, F.Cu at (38.1, 116.8)
- added REF**1102: Single PTH, SparkFun-Footprints:proto, F.Cu at (236.2, 76.2)
- added REF**1102: Single PTH, SparkFun-Footprints:proto, F.Cu at (221.0, 61.0)
- added REF**1102: Single PTH, SparkFun-Footprints:proto, F.Cu at (205.7, 61.0)
- added REF**1102: Single PTH, SparkFun-Footprints:proto, F.Cu at (266.7, 61.0)
- added REF**1102: Single PTH, SparkFun-Footprints:proto, F.Cu at (251.5, 61.0)
- added REF**1102: Single PTH, SparkFun-Footprints:proto, F.Cu at (236.2, 61.0)
- added REF**1102: Single PTH, SparkFun-Footprints:proto, F.Cu at (190.5, 61.0)
- added REF**1102: Single PTH, SparkFun-Footprints:proto, F.Cu at (175.3, 61.0)
- added REF**1102: Single PTH, SparkFun-Footprints:proto, F.Cu at (129.5, 61.0)
- added REF**1102: Single PTH, SparkFun-Footprints:proto, F.Cu at (160.0, 61.0)
- added REF**1102: Single PTH, SparkFun-Footprints:proto, F.Cu at (38.1, 121.9)
- added REF**1102: Single PTH, SparkFun-Footprints:proto, F.Cu at (144.8, 61.0)
- added REF**1102: Single PTH, SparkFun-Footprints:proto, F.Cu at (221.0, 66.0)
- added REF**1102: Single PTH, SparkFun-Footprints:proto, F.Cu at (205.7, 66.0)
- added REF**1102: Single PTH, SparkFun-Footprints:proto, F.Cu at (266.7, 66.0)
- added REF**1102: Single PTH, SparkFun-Footprints:proto, F.Cu at (251.5, 66.0)
- added REF**1102: Single PTH, SparkFun-Footprints:proto, F.Cu at (236.2, 66.0)
- added REF**1102: Single PTH, SparkFun-Footprints:proto, F.Cu at (190.5, 66.0)
- added REF**1102: Single PTH, SparkFun-Footprints:proto, F.Cu at (175.3, 66.0)
- added REF**1102: Single PTH, SparkFun-Footprints:proto, F.Cu at (129.5, 66.0)
- added REF**1102: Single PTH, SparkFun-Footprints:proto, F.Cu at (160.0, 66.0)
- added REF**1102: Single PTH, SparkFun-Footprints:proto, F.Cu at (106.7, 129.5)
- added REF**1102: Single PTH, SparkFun-Footprints:proto, F.Cu at (144.8, 66.0)
- added REF**1102: Single PTH, SparkFun-Footprints:proto, F.Cu at (266.7, 71.1)
- added REF**1102: Single PTH, SparkFun-Footprints:proto, F.Cu at (251.5, 71.1)
- added REF**1102: Single PTH, SparkFun-Footprints:proto, F.Cu at (236.2, 71.1)
- added REF**1102: Single PTH, SparkFun-Footprints:proto, F.Cu at (221.0, 71.1)
- added REF**1102: Single PTH, SparkFun-Footprints:proto, F.Cu at (205.7, 71.1)
- added REF**1102: Single PTH, SparkFun-Footprints:proto, F.Cu at (190.5, 71.1)
- added REF**1102: Single PTH, SparkFun-Footprints:proto, F.Cu at (175.3, 71.1)
- added REF**1102: Single PTH, SparkFun-Footprints:proto, F.Cu at (160.0, 71.1)
- added REF**1102: Single PTH, SparkFun-Footprints:proto, F.Cu at (144.8, 71.1)
- added REF**1102: Single PTH, SparkFun-Footprints:proto, F.Cu at (96.5, 129.5)
- added REF**1102: Single PTH, SparkFun-Footprints:proto, F.Cu at (129.5, 71.1)
- added REF**1102: Single PTH, SparkFun-Footprints:proto, F.Cu at (114.3, 71.1)
- added REF**1102: Single PTH, SparkFun-Footprints:proto, F.Cu at (99.1, 71.1)
- added REF**1102: Single PTH, SparkFun-Footprints:proto, F.Cu at (106.7, 127.0)
- added REF**1102: Single PTH, SparkFun-Footprints:proto, F.Cu at (106.7, 121.9)
- added REF**1102: Single PTH, SparkFun-Footprints:proto, F.Cu at (96.5, 127.0)
- added REF**1103: Single PTH, SparkFun-Footprints:proto, F.Cu at (114.3, 73.7)
- added REF**1103: Single PTH, SparkFun-Footprints:proto, F.Cu at (99.1, 73.7)
- added REF**1104: Single PTH, SparkFun-Footprints:proto, F.Cu at (114.3, 76.2)
- added REF**1104: Single PTH, SparkFun-Footprints:proto, F.Cu at (99.1, 76.2)
- added REF**1105: Single PTH, SparkFun-Footprints:proto, F.Cu at (114.3, 78.7)
- added REF**1105: Single PTH, SparkFun-Footprints:proto, F.Cu at (99.1, 78.7)
- added REF**1106: Single PTH, SparkFun-Footprints:proto, F.Cu at (114.3, 81.3)
- added REF**1106: Single PTH, SparkFun-Footprints:proto, F.Cu at (99.1, 81.3)
- added REF**1107: Single PTH, SparkFun-Footprints:proto, F.Cu at (114.3, 83.8)
- added REF**1107: Single PTH, SparkFun-Footprints:proto, F.Cu at (99.1, 83.8)
- added REF**111: Single PTH, SparkFun-Footprints:proto, F.Cu at (68.6, 68.6)
- added REF**111: Single PTH, SparkFun-Footprints:proto, F.Cu at (76.2, 68.6)
- added REF**1111: Single PTH, SparkFun-Footprints:proto, F.Cu at (40.6, 119.4)
- added REF**1111: Single PTH, SparkFun-Footprints:proto, F.Cu at (269.2, 78.7)
- added REF**1111: Single PTH, SparkFun-Footprints:proto, F.Cu at (223.5, 78.7)
- added REF**1111: Single PTH, SparkFun-Footprints:proto, F.Cu at (193.0, 78.7)
- added REF**1111: Single PTH, SparkFun-Footprints:proto, F.Cu at (177.8, 78.7)
- added REF**1111: Single PTH, SparkFun-Footprints:proto, F.Cu at (208.3, 78.7)
- added REF**1111: Single PTH, SparkFun-Footprints:proto, F.Cu at (238.8, 78.7)
- added REF**1111: Single PTH, SparkFun-Footprints:proto, F.Cu at (254.0, 73.7)
- added REF**1111: Single PTH, SparkFun-Footprints:proto, F.Cu at (269.2, 73.7)
- added REF**1111: Single PTH, SparkFun-Footprints:proto, F.Cu at (223.5, 73.7)
- added REF**1111: Single PTH, SparkFun-Footprints:proto, F.Cu at (193.0, 73.7)
- added REF**1111: Single PTH, SparkFun-Footprints:proto, F.Cu at (109.2, 124.5)
- added REF**1111: Single PTH, SparkFun-Footprints:proto, F.Cu at (177.8, 73.7)
- added REF**1111: Single PTH, SparkFun-Footprints:proto, F.Cu at (208.3, 73.7)
- added REF**1111: Single PTH, SparkFun-Footprints:proto, F.Cu at (238.8, 73.7)
- added REF**1111: Single PTH, SparkFun-Footprints:proto, F.Cu at (223.5, 58.4)
- added REF**1111: Single PTH, SparkFun-Footprints:proto, F.Cu at (208.3, 58.4)
- added REF**1111: Single PTH, SparkFun-Footprints:proto, F.Cu at (254.0, 58.4)
- added REF**1111: Single PTH, SparkFun-Footprints:proto, F.Cu at (269.2, 58.4)
- added REF**1111: Single PTH, SparkFun-Footprints:proto, F.Cu at (238.8, 58.4)
- added REF**1111: Single PTH, SparkFun-Footprints:proto, F.Cu at (193.0, 58.4)
- added REF**1111: Single PTH, SparkFun-Footprints:proto, F.Cu at (177.8, 58.4)
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Connections:
- C10 pad 2: GND -> ISOGND12
- C11 pad 2: GND -> ISOGND12
- C12 pad 2: GND -> ISOGND12
- C13 pad 2: GND -> ISOGND12
- C14 pad 2: GND -> ISOGND12
- C37 pad 2: GND -> ISOGND34
- C38 pad 2: GND -> ISOGND34
- C39 pad 2: GND -> ISOGND34
- C40 pad 2: GND -> ISOGND34
- C41 pad 2: GND -> ISOGND34
- JMP4 pad 1: GND -> ISOGND12
- JMP5 pad 1: GND -> ISOGND34
- P21 pad 5: KEN -> EN
- P31 pad 1: Net-(P31-Pad1) -> +5V
- P36 pad 1: Net-(P36-Pad1) -> GND
- P38 pad 2: GND -> ISOGND12
- P38 pad 5: GND -> ISOGND12
- P39 pad 2: GND -> ISOGND34
- P39 pad 5: GND -> ISOGND34
- R21 pad 2: GND -> ISOGND12
- R22 pad 2: GND -> ISOGND12
- R23 pad 2: GND -> ISOGND12
- R24 pad 2: GND -> ISOGND12
- R25 pad 2: GND -> ISOGND34
- R26 pad 2: GND -> ISOGND34
- R27 pad 2: GND -> ISOGND34
- R28 pad 2: GND -> ISOGND34
- U31 pad 1: GND -> ISOGND34
- U31 pad 3: GND -> ISOGND34
- U31 pad 32: GND -> ISOGND34
- U31 pad 33: GND -> ISOGND34
- U31 pad 7: GND -> ISOGND34
- U5 pad 1: GND -> ISOGND12
- U5 pad 3: GND -> ISOGND12
- U5 pad 32: GND -> ISOGND12
- U5 pad 33: GND -> ISOGND12
- U5 pad 7: GND -> ISOGND12
Routing:
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- added copper zone on B.Cu, net ISOGND12
- added copper zone on F.Cu, net ISOGND12
- added copper zone on B.Cu, net ISOGND34
- added copper zone on F.Cu, net ISOGND34
Other:
- board text added: "+1v8"
- board text added: "+3v3"
- board text added: "+3v3 source"
- board text added: "+5v"
- board text added: "1"
- board text added: "10"
- board text added: "11"
- board text added: "12"
- board text added: "13"
- board text added: "14"
- board text added: "15"
- board text added: "16"
- board text added: "17"
- board text added: "2"
- board text added: "25"
- board text added: "3"
- board text added: "33"
- board text added: "4"
- board text added: "41"
- board text added: "49"
- board text added: "5"
- board text added: "57"
- board text added: "6"
- board text added: "7"
- board text added: "8"
- board text added: "9"
- board text added: "A"
- board text added: "A11"
- board text added: "A12"
- board text added: "A13"
- board text added: "A14"
- board text added: "B"
- board text added: "BCLK"
- board text added: "C"
- board text added: "CODEC 1/2"
- board text added: "CODEC 3/4"
- board text added: "Columns"
- board text added: "D"
- board text added: "DIN"
- board text added: "DOUT"
- board text added: "GND"
- board text added: "L"
- board text added: "LRCLK"
- board text added: "MCLK"
- board text added: "MISO"
- board text added: "MOSI"
- board text added: "Mux Select"
- board text added: "N"
- board text added: "PORT 0"
- board text added: "PORT 1"
- board text added: "PROTO-8"
- board text added: "Rows"
- board text added: "SCK"
- board text added: "SCL"
- board text added: "SDA"
- board text added: "SIO2"
- board text added: "SIO3"
- board text added: "UCC"
- board text added: "UGND"
- board text added: "VUUIN"
