File: Test Projects/Teensy_test_layout.kicad_pcb (KiCad board)
At the start: 2 copper layers, 254 x 127 mm, 1193 parts, among them P1 CONN_01X02, P10 CONN_01X06, P100 SPI_MOSI, P101 SPI_MISO, P102 SPI_SCK, P11 CONN_01X06, P12 CONN_01X06, P13 CONN_01X08, P14 CONN_01X08, P15 CONN_01X08, P16 CONN_01X08, P17 CONN_01X08, P18 CONN_01X08, P19 CONN_01X08, P2 CONN_01X03, P20 CONN_01X08, P21 CONN_01X05, P22 CONN_01X08, P23 CONN_01X08, P24 CONN_01X08, P25 CONN_01X08, P26 CONN_01X08, P27 CONN_01X08, P28 CONN_01X08, P29 CONN_01X08, P3 COLS0, P30 CONN_01X03, P31 CONN_01X01, P32 PIN8, P33 SIO2, P34 ~HOLD~/SIO3, P35 PIN37, P36 CONN_01X01, P37 PIN31, P38 CONN_01X06, P39 CONN_01X06, P4 COLS1, P40 CONN_01X08, P41 CONN_01X08, P42 CONN_01X08, P43 CONN_01X08, P44 CONN_01X08, P45 CONN_01X08, P46 CONN_01X08, P47 CONN_01X08, P48 CONN_01X08, P49 CONN_01X08, P5 CONN_01X06, P50 CONN_01X08, P51 CONN_01X08, P52 CONN_01X08, P53 CONN_01X08, P54 CONN_01X08, P55 CONN_01X08, P56 CONN_01X01, P57 CONN_01X01, P58 VUU, P59 CONN_01X01, P6 CONN_01X06, P60 CONN_01X01, P61 CONN_01X01, P62 UGND, P63 CONN_01X01, P64 DIN1, P65 DOUT1, P66 SDA0_ISO, P67 SCL0_ISO, P68 MCLK_ISO, P69 BCLK_ISO, P7 CONN_01X06, P70 LRCLK_ISO, P71 DIN0, P72 DOUT0, P73 IN2TTL, P74 CONN_01X08, P75 CONN_01X08, P76 CONN_01X08, P77 CONN_01X08, P78 CONN_01X08, P79 CONN_01X08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

Commit message: layout
Parts:
- added C18: 68uF, Capacitors_Tantalum_SMD:TantalC_SizeC_EIA-6032_Reflow, F.Cu at (175.3, 92.7)
- added C55: 1uF, Capacitors_SMD:C_0603, F.Cu at (171.4, 90.7)
- added C56: 100u, Capacitors_SMD:c_elec_10x10.5, F.Cu at (35.6, 53.3)
- added C57: 100u, Capacitors_SMD:c_elec_10x10.5, F.Cu at (47.0, 53.3)
- added C58: 1u, Capacitors_SMD:C_1206, F.Cu at (27.9, 50.8)
- added C59: 1u, Capacitors_SMD:C_1206, F.Cu at (27.9, 44.5)
- added C60: 68uF, Capacitors_Tantalum_SMD:TantalC_SizeC_EIA-6032_Reflow, F.Cu at (123.2, 137.2)
- added C61: 1uF, Capacitors_SMD:C_0603, F.Cu at (126.2, 136.1)
- added C62: 22p, Capacitors_SMD:C_0603, F.Cu at (154.4, 156.3)
- added C63: 22p, Capacitors_SMD:C_0603, F.Cu at (138.0, 156.1)
- added C64: 22p, Capacitors_SMD:C_0603, F.Cu at (142.0, 156.1)
- added C65: 22p, Capacitors_SMD:C_0603, F.Cu at (145.9, 156.1)
- added C66: 22p, Capacitors_SMD:C_0603, F.Cu at (161.4, 156.3)
- added C67: 22p, Capacitors_SMD:C_0603, F.Cu at (149.9, 156.1)
- added C68: 22p, Capacitors_SMD:C_0603, F.Cu at (158.0, 156.1)
- added C69: 22p, Capacitors_SMD:C_0603, F.Cu at (102.0, 156.0)
- added C70: 22p, Capacitors_SMD:C_0603, F.Cu at (98.4, 157.2)
- added C71: 22p, Capacitors_SMD:C_0603, F.Cu at (96.0, 155.8)
- added JMP29: 2Jumper, SparkFun-Footprints:SF-2way-open, F.Cu at (118.9, 97.5)
- added P103: CONN_01X01, SparkFun-Footprints:PTH_LUG_.05, F.Cu at (172.7, 83.8)
- added P104: CONN_01X01, SparkFun-Footprints:TestHole, F.Cu at (55.9, 94.0)
- added P105: CONN_01X01, SparkFun-Footprints:TestHole, F.Cu at (55.9, 86.4)
- added P106: CONN_01X01, SparkFun-Footprints:PTH_LUG_.05, F.Cu at (129.5, 134.6)
- added P107: CONN_01X01, SparkFun-Footprints:PTH_LUG_.05, F.Cu at (119.4, 142.2)
- added P108: CONN_01X01, SparkFun-Footprints:PTH_LUG_.05, F.Cu at (175.3, 104.1)
- added P109: SCL_ISO, SparkFun-Footprints:TestHole, F.Cu at (117.0, 97.5)
- added P110: SDA_ISO, SparkFun-Footprints:TestHole, F.Cu at (117.0, 100.1)
- added P111: SCL_ISO2, SparkFun-Footprints:TestHole, F.Cu at (120.8, 97.5)
- added P112: SDA_ISO2, SparkFun-Footprints:TestHole, F.Cu at (120.8, 100.1)
- added R100: 50, Resistors_SMD:R_0603, F.Cu at (94.8, 162.2)
- added R95: 1, Resistors_SMD:R_0603, F.Cu at (171.7, 87.6)
- added R96: 1, Resistors_SMD:R_2512, F.Cu at (35.6, 44.5)
- added R97: 1, Resistors_SMD:R_0603, F.Cu at (126.7, 132.1)
- added R98: 50, Resistors_SMD:R_0603, F.Cu at (102.7, 162.2)
- added R99: 50, Resistors_SMD:R_0603, F.Cu at (98.8, 162.2)
- moved JMP21 54.5 mm to (118.9, 100.1)
- moved ROWS1 27.4 mm to (58.4, 121.9), turned to 90 degrees
- moved P66 24.3 mm to (144.3, 103.0)
- moved P67 24.3 mm to (144.3, 100.5)
- moved P90 24.3 mm to (27.9, 61.0)
- moved JMP22 24.2 mm to (142.2, 103.0)
- moved JMP23 24.2 mm to (142.2, 100.5)
- moved P91 24.1 mm to (140.2, 103.0)
- moved P92 24.1 mm to (140.2, 100.5)
- moved P1 11.4 mm to (47.0, 34.3), turned to 0 degrees
- moved P31 10.5 mm to (55.9, 78.7)
- moved C1 10.2 mm to (31.8, 94.0)
- moved C43 10.2 mm to (31.8, 109.9)
- moved REF**1102 10.2 mm to (43.2, 132.1)
- moved REF**1102 10.2 mm to (38.1, 132.1)
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Connections:
- JACK1 pad 1: Net-(JACK1-Pad1) -> (no net)
- JACK1 pad 2: Net-(JACK1-Pad2) -> (no net)
- JACK1 pad 3: Net-(JACK1-Pad3) -> (no net)
- JACK1 pad 6: Net-(JACK1-Pad6) -> (no net)
- JACK1 pad 7: Net-(JACK1-Pad7) -> (no net)
- JACK12 pad GNDB: Net-(JACK12-PadGNDB) -> (no net)
- JACK12 pad PWR: VBULK -> PWR
- JACK2 pad 1: Net-(JACK2-Pad1) -> (no net)
- JACK2 pad 2: Net-(JACK2-Pad2) -> (no net)
- JACK2 pad 3: Net-(JACK2-Pad3) -> (no net)
- JACK2 pad 6: Net-(JACK2-Pad6) -> (no net)
- JACK2 pad 7: Net-(JACK2-Pad7) -> (no net)
- JACK3 pad 1: Net-(JACK3-Pad1) -> (no net)
- JACK3 pad 2: Net-(JACK3-Pad2) -> (no net)
- JACK3 pad 3: Net-(JACK3-Pad3) -> (no net)
- JACK3 pad 6: Net-(JACK3-Pad6) -> (no net)
- JACK3 pad 7: Net-(JACK3-Pad7) -> (no net)
- JMP21 pad 1: +5V -> SDA0
- JMP21 pad 2: VDD -> SDA34
- JMP22 pad 1: SDA0 -> SDA34
- JMP22 pad 2: SDA_ISO -> SDA12
- JMP23 pad 1: SCL0 -> SCL34
- JMP23 pad 2: SCL_ISO -> SCL12
- P1 pad 1: VBULK -> GND
- P1 pad 2: GND -> PWR
- P101 pad 1: SPI_MISO -> Net-(P101-Pad1)
- P66 pad 1: SDA_ISO -> SDA12
- P67 pad 1: SCL_ISO -> SCL12
- P91 pad 1: SDA0 -> SDA34
- P92 pad 1: SCL0 -> SCL34
- U11 pad 1: Net-(U11-Pad1) -> (no net)
- U11 pad 4: Net-(U11-Pad4) -> (no net)
- U11 pad 7: Net-(U11-Pad7) -> (no net)
- U3 pad 14: SPI_SCK -> Net-(R98-Pad1)
- U3 pad 21: KEN -> (no net)
- U3 pad 35: Net-(U3-Pad35) -> (no net)
- U3 pad 38: Net-(U3-Pad38) -> (no net)
- U3 pad 41: Net-(U3-Pad41) -> (no net)
- U3 pad 48: Net-(U3-Pad48) -> (no net)
- U3 pad 49: Net-(U3-Pad49) -> (no net)
- U3 pad 7: SPI_MOSI -> Net-(R99-Pad1)
- U30 pad 9: Net-(U30-Pad9) -> (no net)
- U31 pad 15: Net-(U31-Pad15) -> (no net)
- U31 pad 16: Net-(U31-Pad16) -> (no net)
- U31 pad 18: Net-(U31-Pad18) -> (no net)
- U31 pad 27: SDA_ISO -> SDA34
- U31 pad 29: SCL_ISO -> SCL34
- U32 pad 2: SPI_MISO -> Net-(P101-Pad1)
- U34 pad 1: Net-(U34-Pad1) -> (no net)
- U34 pad 4: Net-(U34-Pad4) -> (no net)
- U34 pad 7: Net-(U34-Pad7) -> (no net)
- U5 pad 15: Net-(U5-Pad15) -> (no net)
- U5 pad 16: Net-(U5-Pad16) -> (no net)
- U5 pad 18: Net-(U5-Pad18) -> (no net)
- U5 pad 27: SDA_ISO -> SDA12
- U5 pad 29: SCL_ISO -> SCL12
- U6 pad 1: Net-(U6-Pad1) -> (no net)
- U6 pad 10: Net-(U6-Pad10) -> (no net)
- U6 pad 11: Net-(U6-Pad11) -> (no net)
- U6 pad 12: Net-(U6-Pad12) -> (no net)
- U6 pad 8: Net-(U6-Pad8) -> (no net)
- U6 pad 9: Net-(U6-Pad9) -> (no net)
- U8 pad 9: Net-(U8-Pad9) -> (no net)
Routing:
- net SDA_ISO: track 48.0 -> 0.00 mm, vias 2 -> 0
- net SCL_ISO: track 47.5 -> 0.00 mm, vias 2 -> 0
- net ROW4: track 52.9 -> 11.8 mm
- net ROW3: track 48.6 -> 12.9 mm
- net ROW2: track 44.0 -> 12.9 mm
- net SDA34: track 0.00 -> 29.8 mm, vias 0 -> 1
- net SCL34: track 0.00 -> 29.1 mm, vias 0 -> 1
- net ROW1: track 41.6 -> 13.3 mm
- net EN: track 362.3 -> 385.5 mm, vias 14 -> 15
- net KEN: track 23.2 -> 0.00 mm, vias 1 -> 0
- net +5V: track 523.4 -> 501.9 mm
- net SDA12: track 0.00 -> 18.1 mm, vias 0 -> 1
- net SCL12: track 0.00 -> 17.5 mm, vias 0 -> 1
- net PWR: track 0.00 -> 15.1 mm
- net Net-(C18-Pad1): track 0.00 -> 10.2 mm
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- added copper zone on F.Cu, net VBULK
Other:
- board text added: "+3v3 reg"
- board text added: "VUU"
- board text removed: "+3v3 source"
- board text removed: "UCC"

Commit message: Finished artwork
Parts:
- removed the REF** at (182.9, 27.9)
- removed the REF** at (172.7, 27.9)
- removed the REF** at (162.6, 27.9)
- removed the REF** at (152.4, 27.9)
- removed the REF** at (142.2, 27.9)
- removed the REF** at (132.1, 27.9)
- removed the REF** at (121.9, 27.9)
- removed the REF** at (88.9, 27.9)
- removed the REF** at (111.8, 27.9)
- removed the REF** at (99.1, 27.9)
- removed the REF** at (68.6, 27.9)
- removed the REF** at (78.7, 27.9)
- removed the REF** at (58.4, 27.9)
- removed the REF** at (45.7, 27.9)
- removed the REF** at (254.0, 27.9)
- removed the REF** at (243.8, 27.9)
- removed the REF** at (233.7, 27.9)
- removed the REF** at (223.5, 27.9)
- removed the REF** at (213.4, 27.9)
- removed the REF** at (203.2, 27.9)
- added G***: LOGO, SparkFun-Footprints:PROTO8LOGO, F.Cu at (83.7, 90.8)
- added G***: LOGO, SparkFun-Footprints:biglogoslant, B.Cu at (158.0, 101.9)
- added R101: 4.7k, Resistors_SMD:R_0603, F.Cu at (91.4, 144.8)
- added R102: 4.7k, Resistors_SMD:R_0603, F.Cu at (108.0, 144.8)
- added REF**: SVIA, SparkFun-Footprints:SVIA, F.Cu at (47.0, 57.3)
- added REF**: SVIA, SparkFun-Footprints:SVIA, F.Cu at (146.7, 94.0)
- added REF**: SVIA, SparkFun-Footprints:SVIA, F.Cu at (88.1, 119.6)
- added REF**: SVIA, SparkFun-Footprints:SVIA, F.Cu at (95.5, 117.6)
- added REF**: SVIA, SparkFun-Footprints:SVIA, F.Cu at (104.4, 115.1)
- added REF**: SVIA, SparkFun-Footprints:SVIA, F.Cu at (106.2, 112.3)
- added REF**: SVIA, SparkFun-Footprints:SVIA, F.Cu at (117.3, 130.0)
- added REF**: SVIA, SparkFun-Footprints:SVIA, F.Cu at (102.1, 142.0)
- added REF**: SVIA, SparkFun-Footprints:SVIA, F.Cu at (101.1, 148.1)
- added REF**: SVIA, SparkFun-Footprints:SVIA, F.Cu at (92.2, 139.7)
- added REF**: SVIA, SparkFun-Footprints:SVIA, F.Cu at (96.0, 140.0)
- added REF**: SVIA, SparkFun-Footprints:SVIA, F.Cu at (99.1, 138.7)
- added REF**: SVIA, SparkFun-Footprints:SVIA, F.Cu at (147.3, 88.3)
- added REF**: SVIA, SparkFun-Footprints:SVIA, F.Cu at (90.7, 134.1)
- added REF**: SVIA, SparkFun-Footprints:SVIA, F.Cu at (84.8, 129.5)
- added REF**: SVIA, SparkFun-Footprints:SVIA, F.Cu at (85.9, 134.1)
- added REF**: SVIA, SparkFun-Footprints:SVIA, F.Cu at (85.9, 137.7)
- added REF**: SVIA, SparkFun-Footprints:SVIA, F.Cu at (82.8, 137.7)
- added REF**: SVIA, SparkFun-Footprints:SVIA, F.Cu at (74.7, 132.1)
- added REF**: SVIA, SparkFun-Footprints:SVIA, F.Cu at (79.0, 129.0)
- added REF**: SVIA, SparkFun-Footprints:SVIA, F.Cu at (80.8, 141.2)
- added REF**: SVIA, SparkFun-Footprints:SVIA, F.Cu at (70.6, 135.9)
- added REF**: SVIA, SparkFun-Footprints:SVIA, F.Cu at (60.7, 140.0)
- added REF**: SVIA, SparkFun-Footprints:SVIA, F.Cu at (147.3, 83.8)
- added REF**: SVIA, SparkFun-Footprints:SVIA, F.Cu at (56.9, 133.9)
- added REF**: SVIA, SparkFun-Footprints:SVIA, F.Cu at (55.4, 136.1)
- added REF**: SVIA, SparkFun-Footprints:SVIA, F.Cu at (47.8, 138.2)
- added REF**: SVIA, SparkFun-Footprints:SVIA, F.Cu at (62.2, 130.0)
- added REF**: SVIA, SparkFun-Footprints:SVIA, F.Cu at (29.2, 136.9)
- added REF**: SVIA, SparkFun-Footprints:SVIA, F.Cu at (33.3, 147.8)
- added REF**: SVIA, SparkFun-Footprints:SVIA, F.Cu at (86.9, 150.4)
- added REF**: SVIA, SparkFun-Footprints:SVIA, F.Cu at (109.7, 150.6)
- added REF**: SVIA, SparkFun-Footprints:SVIA, F.Cu at (120.4, 150.6)
- added REF**: SVIA, SparkFun-Footprints:SVIA, F.Cu at (172.5, 150.4)
- added REF**: SVIA, SparkFun-Footprints:SVIA, F.Cu at (147.3, 76.2)
- added REF**: SVIA, SparkFun-Footprints:SVIA, F.Cu at (217.9, 150.4)
- added REF**: SVIA, SparkFun-Footprints:SVIA, F.Cu at (276.9, 140.7)
- added REF**: SVIA, SparkFun-Footprints:SVIA, F.Cu at (266.7, 145.8)
- added REF**: SVIA, SparkFun-Footprints:SVIA, F.Cu at (176.3, 129.0)
- added REF**: SVIA, SparkFun-Footprints:SVIA, F.Cu at (165.1, 98.8)
- added REF**: SVIA, SparkFun-Footprints:SVIA, F.Cu at (167.6, 98.8)
- added REF**: SVIA, SparkFun-Footprints:SVIA, F.Cu at (169.9, 96.8)
- added REF**: SVIA, SparkFun-Footprints:SVIA, F.Cu at (172.5, 95.0)
- added REF**: SVIA, SparkFun-Footprints:SVIA, F.Cu at (175.3, 98.0)
- added REF**: SVIA, SparkFun-Footprints:SVIA, F.Cu at (174.5, 84.8)
- added REF**: SVIA, SparkFun-Footprints:SVIA, F.Cu at (93.5, 123.7)
- added REF**: SVIA, SparkFun-Footprints:SVIA, F.Cu at (176.5, 87.9)
- added REF**: SVIA, SparkFun-Footprints:SVIA, F.Cu at (180.6, 86.9)
- added REF**: SVIA, SparkFun-Footprints:SVIA, F.Cu at (198.6, 85.1)
- added REF**: SVIA, SparkFun-Footprints:SVIA, F.Cu at (193.3, 89.4)
- added REF**: SVIA, SparkFun-Footprints:SVIA, F.Cu at (198.6, 90.9)
- added REF**: SVIA, SparkFun-Footprints:SVIA, F.Cu at (200.7, 93.0)
- added REF**: SVIA, SparkFun-Footprints:SVIA, F.Cu at (221.0, 93.7)
- added REF**: SVIA, SparkFun-Footprints:SVIA, F.Cu at (216.7, 87.6)
- added REF**: SVIA, SparkFun-Footprints:SVIA, F.Cu at (214.9, 89.2)
- added REF**: SVIA, SparkFun-Footprints:SVIA, F.Cu at (224.3, 86.4)
- added REF**: SVIA, SparkFun-Footprints:SVIA, F.Cu at (90.9, 120.9)
- added REF**: SVIA, SparkFun-Footprints:SVIA, F.Cu at (237.2, 86.6)
- added REF**: SVIA, SparkFun-Footprints:SVIA, F.Cu at (240.5, 89.7)
- added REF**: SVIA, SparkFun-Footprints:SVIA, F.Cu at (249.9, 91.9)
- added REF**: SVIA, SparkFun-Footprints:SVIA, F.Cu at (261.4, 87.9)
- added REF**: SVIA, SparkFun-Footprints:SVIA, F.Cu at (263.7, 93.7)
- added REF**: SVIA, SparkFun-Footprints:SVIA, F.Cu at (275.6, 93.0)
- added REF**: SVIA, SparkFun-Footprints:SVIA, F.Cu at (173.2, 104.9)
- added REF**: SVIA, SparkFun-Footprints:SVIA, F.Cu at (181.1, 114.6)
- added REF**: SVIA, SparkFun-Footprints:SVIA, F.Cu at (176.0, 113.3)
- added REF**: SVIA, SparkFun-Footprints:SVIA, F.Cu at (181.4, 109.2)
- added REF**: SVIA, SparkFun-Footprints:SVIA, F.Cu at (93.3, 107.2)
- added REF**: SVIA, SparkFun-Footprints:SVIA, F.Cu at (193.0, 111.0)
- added REF**: SVIA, SparkFun-Footprints:SVIA, F.Cu at (193.5, 109.0)
- added REF**: SVIA, SparkFun-Footprints:SVIA, F.Cu at (198.6, 111.5)
- added REF**: SVIA, SparkFun-Footprints:SVIA, F.Cu at (199.9, 116.6)
- added REF**: SVIA, SparkFun-Footprints:SVIA, F.Cu at (205.5, 119.1)
- added REF**: SVIA, SparkFun-Footprints:SVIA, F.Cu at (217.7, 114.3)
- added REF**: SVIA, SparkFun-Footprints:SVIA, F.Cu at (228.3, 118.9)
- added REF**: SVIA, SparkFun-Footprints:SVIA, F.Cu at (237.0, 109.7)
- added REF**: SVIA, SparkFun-Footprints:SVIA, F.Cu at (237.5, 117.6)
- added REF**: SVIA, SparkFun-Footprints:SVIA, F.Cu at (237.7, 113.0)
- added REF**: SVIA, SparkFun-Footprints:SVIA, F.Cu at (93.5, 114.6)
- added REF**: SVIA, SparkFun-Footprints:SVIA, F.Cu at (250.7, 113.5)
- added REF**: SVIA, SparkFun-Footprints:SVIA, F.Cu at (252.7, 115.8)
- added REF**: SVIA, SparkFun-Footprints:SVIA, F.Cu at (263.4, 115.1)
- added REF**: SVIA, SparkFun-Footprints:SVIA, F.Cu at (275.6, 115.3)
- added REF**: SVIA, SparkFun-Footprints:SVIA, F.Cu at (129.5, 131.1)
- added REF**: SVIA, SparkFun-Footprints:SVIA, F.Cu at (171.2, 122.7)
- added REF**: SVIA, SparkFun-Footprints:SVIA, F.Cu at (149.9, 128.0)
- added REF**: SVIA, SparkFun-Footprints:SVIA, F.Cu at (172.7, 142.5)
- added REF**: SVIA, SparkFun-Footprints:SVIA, F.Cu at (149.9, 142.2)
- added REF**: SVIA, SparkFun-Footprints:SVIA, F.Cu at (172.5, 114.3)
- added REF**: SVIA, SparkFun-Footprints:SVIA, F.Cu at (94.7, 103.3)
- added REF**: SVIA, SparkFun-Footprints:SVIA, F.Cu at (171.7, 119.4)
- added REF**: SVIA, SparkFun-Footprints:SVIA, F.Cu at (151.4, 112.5)
- added REF**: SVIA, SparkFun-Footprints:SVIA, F.Cu at (146.8, 117.3)
- added REF**: SVIA, SparkFun-Footprints:SVIA, F.Cu at (139.4, 115.1)
- added REF**: SVIA, SparkFun-Footprints:SVIA, F.Cu at (120.1, 115.8)
- added REF**: SVIA, SparkFun-Footprints:SVIA, F.Cu at (122.7, 115.8)
- added REF**: SVIA, SparkFun-Footprints:SVIA, F.Cu at (128.0, 121.9)
- added REF**: SVIA, SparkFun-Footprints:SVIA, F.Cu at (125.0, 121.9)
- added REF**: SVIA, SparkFun-Footprints:SVIA, F.Cu at (149.9, 120.7)
- added REF**: SVIA, SparkFun-Footprints:SVIA, F.Cu at (240.3, 139.2)
- added REF**: SVIA, SparkFun-Footprints:SVIA, F.Cu at (194.1, 118.6)
- added REF**: SVIA, SparkFun-Footprints:SVIA, F.Cu at (216.4, 138.4)
- added REF**: SVIA, SparkFun-Footprints:SVIA, F.Cu at (195.1, 138.9)
- added REF**: SVIA, SparkFun-Footprints:SVIA, F.Cu at (125.2, 143.3)
- added REF**: SVIA, SparkFun-Footprints:SVIA, F.Cu at (126.7, 139.2)
- added REF**: SVIA, SparkFun-Footprints:SVIA, F.Cu at (129.5, 137.4)
- added REF**: SVIA, SparkFun-Footprints:SVIA, F.Cu at (132.3, 135.6)
- added REF**: SVIA, SparkFun-Footprints:SVIA, F.Cu at (141.5, 135.4)
- added REF**: SVIA, SparkFun-Footprints:SVIA, F.Cu at (151.6, 132.1)
- added REF**: SVIA, SparkFun-Footprints:SVIA, F.Cu at (148.3, 138.4)
- added REF**: SVIA, SparkFun-Footprints:SVIA, F.Cu at (171.7, 138.7)
- added REF**: SVIA, SparkFun-Footprints:SVIA, F.Cu at (35.6, 57.3)
- added REF**: SVIA, SparkFun-Footprints:SVIA, F.Cu at (40.6, 27.9)
- added REF**: SVIA, SparkFun-Footprints:SVIA, F.Cu at (173.7, 135.4)
- added REF**: SVIA, SparkFun-Footprints:SVIA, F.Cu at (176.0, 133.6)
- added REF**: SVIA, SparkFun-Footprints:SVIA, F.Cu at (198.4, 133.6)
- added REF**: SVIA, SparkFun-Footprints:SVIA, F.Cu at (260.9, 136.7)
- added REF**: SVIA, SparkFun-Footprints:SVIA, F.Cu at (234.4, 136.4)
- added REF**: SVIA, SparkFun-Footprints:SVIA, F.Cu at (53.3, 33.0)
- added REF**: SVIA, SparkFun-Footprints:SVIA, F.Cu at (251.5, 50.8)
- added REF**: SVIA, SparkFun-Footprints:SVIA, F.Cu at (231.1, 50.8)
- added REF**: SVIA, SparkFun-Footprints:SVIA, F.Cu at (210.8, 45.7)
- added REF**: SVIA, SparkFun-Footprints:SVIA, F.Cu at (190.5, 50.8)
- added REF**: SVIA, SparkFun-Footprints:SVIA, F.Cu at (170.2, 50.8)
- added REF**: SVIA, SparkFun-Footprints:SVIA, F.Cu at (149.9, 45.7)
- added REF**: SVIA, SparkFun-Footprints:SVIA, F.Cu at (129.5, 50.8)
- added REF**: SVIA, SparkFun-Footprints:SVIA, F.Cu at (111.8, 50.8)
- added REF**: SVIA, SparkFun-Footprints:SVIA, F.Cu at (55.9, 95.9)
- added REF**: SVIA, SparkFun-Footprints:SVIA, F.Cu at (276.9, 50.8)
- added REF**: SVIA, SparkFun-Footprints:SVIA, F.Cu at (274.3, 27.9)
- added REF**: SVIA, SparkFun-Footprints:SVIA, F.Cu at (261.6, 27.9)
- added REF**: SVIA, SparkFun-Footprints:SVIA, F.Cu at (241.3, 27.9)
- added REF**: SVIA, SparkFun-Footprints:SVIA, F.Cu at (221.0, 27.9)
- added REF**: SVIA, SparkFun-Footprints:SVIA, F.Cu at (200.7, 27.9)
- added REF**: SVIA, SparkFun-Footprints:SVIA, F.Cu at (180.3, 27.9)
- added REF**: SVIA, SparkFun-Footprints:SVIA, F.Cu at (160.0, 27.9)
- added REF**: SVIA, SparkFun-Footprints:SVIA, F.Cu at (139.7, 27.9)
- added REF**: SVIA, SparkFun-Footprints:SVIA, F.Cu at (119.4, 27.9)
- added REF**: SVIA, SparkFun-Footprints:SVIA, F.Cu at (65.4, 90.8)
- added REF**: SVIA, SparkFun-Footprints:SVIA, F.Cu at (27.9, 33.0)
- added REF**: SVIA, SparkFun-Footprints:SVIA, F.Cu at (38.7, 117.5)
- added REF**: SVIA, SparkFun-Footprints:SVIA, F.Cu at (45.7, 120.0)
- added REF**: SVIA, SparkFun-Footprints:SVIA, F.Cu at (52.1, 120.0)
- added REF**: SVIA, SparkFun-Footprints:SVIA, F.Cu at (52.1, 109.9)
- added REF**: SVIA, SparkFun-Footprints:SVIA, F.Cu at (45.7, 109.9)
- added REF**: SVIA, SparkFun-Footprints:SVIA, F.Cu at (45.7, 104.8)
- added REF**: SVIA, SparkFun-Footprints:SVIA, F.Cu at (52.1, 102.9)
- added REF**: SVIA, SparkFun-Footprints:SVIA, F.Cu at (38.7, 102.9)
- added REF**: SVIA, SparkFun-Footprints:SVIA, F.Cu at (30.5, 114.9)
- added REF**: SVIA, SparkFun-Footprints:SVIA, F.Cu at (60.3, 87.6)
- added REF**: SVIA, SparkFun-Footprints:SVIA, F.Cu at (30.5, 102.9)
- added REF**: SVIA, SparkFun-Footprints:SVIA, F.Cu at (51.3, 99.3)
- added REF**: SVIA, SparkFun-Footprints:SVIA, F.Cu at (50.0, 89.2)
- added REF**: SVIA, SparkFun-Footprints:SVIA, F.Cu at (51.1, 85.9)
- added REF**: SVIA, SparkFun-Footprints:SVIA, F.Cu at (50.8, 61.2)
- added REF**: SVIA, SparkFun-Footprints:SVIA, F.Cu at (51.1, 73.7)
- added REF**: SVIA, SparkFun-Footprints:SVIA, F.Cu at (54.4, 83.8)
- added REF**: SVIA, SparkFun-Footprints:SVIA, F.Cu at (60.2, 67.3)
- added REF**: SVIA, SparkFun-Footprints:SVIA, F.Cu at (60.5, 73.9)
- added REF**: SVIA, SparkFun-Footprints:SVIA, F.Cu at (60.2, 80.0)
- added REF**: SVIA, SparkFun-Footprints:SVIA, F.Cu at (55.2, 90.8)
- added REF**: SVIA, SparkFun-Footprints:SVIA, F.Cu at (64.8, 65.3)
- added REF**: SVIA, SparkFun-Footprints:SVIA, F.Cu at (63.0, 86.9)
- added REF**: SVIA, SparkFun-Footprints:SVIA, F.Cu at (61.0, 103.1)
- added REF**: SVIA, SparkFun-Footprints:SVIA, F.Cu at (61.0, 97.0)
- added REF**: SVIA, SparkFun-Footprints:SVIA, F.Cu at (65.3, 67.8)
- added REF**: SVIA, SparkFun-Footprints:SVIA, F.Cu at (69.3, 65.0)
- added REF**: SVIA, SparkFun-Footprints:SVIA, F.Cu at (58.2, 58.9)
- added REF**: SVIA, SparkFun-Footprints:SVIA, F.Cu at (90.4, 54.9)
- added REF**: SVIA, SparkFun-Footprints:SVIA, F.Cu at (104.4, 59.9)
- added REF**: SVIA, SparkFun-Footprints:SVIA, F.Cu at (82.5, 60.7)
- added REF**: SVIA, SparkFun-Footprints:SVIA, F.Cu at (71.1, 88.9)
- added REF**: SVIA, SparkFun-Footprints:SVIA, F.Cu at (85.9, 57.9)
- added REF**: SVIA, SparkFun-Footprints:SVIA, F.Cu at (82.5, 48.8)
- added REF**: SVIA, SparkFun-Footprints:SVIA, F.Cu at (74.2, 49.3)
- added REF**: SVIA, SparkFun-Footprints:SVIA, F.Cu at (78.0, 52.1)
- added REF**: SVIA, SparkFun-Footprints:SVIA, F.Cu at (106.9, 44.5)
- added REF**: SVIA, SparkFun-Footprints:SVIA, F.Cu at (99.1, 41.7)
- added REF**: SVIA, SparkFun-Footprints:SVIA, F.Cu at (79.2, 42.4)
- added REF**: SVIA, SparkFun-Footprints:SVIA, F.Cu at (58.4, 42.2)
- added REF**: SVIA, SparkFun-Footprints:SVIA, F.Cu at (28.4, 38.9)
- added REF**: SVIA, SparkFun-Footprints:SVIA, F.Cu at (33.0, 55.9)
- added REF**: SVIA, SparkFun-Footprints:SVIA, F.Cu at (120.0, 88.9)
- added REF**: SVIA, SparkFun-Footprints:SVIA, F.Cu at (49.5, 55.9)
- added REF**: SVIA, SparkFun-Footprints:SVIA, F.Cu at (47.0, 53.3)
- added REF**: SVIA, SparkFun-Footprints:SVIA, F.Cu at (44.5, 55.9)
- added REF**: SVIA, SparkFun-Footprints:SVIA, F.Cu at (38.1, 55.9)
- added REF**: SVIA, SparkFun-Footprints:SVIA, F.Cu at (35.6, 53.3)
- added REF**: SVIA, SparkFun-Footprints:SVIA, F.Cu at (32.5, 60.7)
- added REF**: SVIA, SparkFun-Footprints:SVIA, F.Cu at (27.2, 55.1)
- added REF**: SVIA, SparkFun-Footprints:SVIA, F.Cu at (27.2, 65.0)
- added REF**: SVIA, SparkFun-Footprints:SVIA, F.Cu at (27.2, 76.7)
- added REF**: SVIA, SparkFun-Footprints:SVIA, F.Cu at (27.9, 88.1)
- added REF**: SVIA, SparkFun-Footprints:SVIA, F.Cu at (147.3, 101.6)
- added REF**: SVIA, SparkFun-Footprints:SVIA, F.Cu at (27.9, 99.3)
- added REF**: SVIA, SparkFun-Footprints:SVIA, F.Cu at (65.5, 96.8)
- added REF**: SVIA, SparkFun-Footprints:SVIA, F.Cu at (66.3, 104.6)
- added REF**: SVIA, SparkFun-Footprints:SVIA, F.Cu at (58.4, 106.7)
- added REF**: SVIA, SparkFun-Footprints:SVIA, F.Cu at (58.4, 101.1)
- added REF**: SVIA, SparkFun-Footprints:SVIA, F.Cu at (70.9, 112.0)
- added REF**: SVIA, SparkFun-Footprints:SVIA, F.Cu at (70.9, 109.2)
- added REF**: SVIA, SparkFun-Footprints:SVIA, F.Cu at (76.2, 111.8)
- added REF**: SVIA, SparkFun-Footprints:SVIA, F.Cu at (78.7, 111.8)
- added REF**: SVIA, SparkFun-Footprints:SVIA, F.Cu at (84.3, 117.1)
- added REF**1102: Single PTH, SparkFun-Footprints:proto, F.Cu at (106.7, 132.1)
- added REF**1102: Single PTH, SparkFun-Footprints:proto, F.Cu at (96.5, 132.1)
- added REF**1112: Single PTH, SparkFun-Footprints:proto, F.Cu at (99.1, 132.1)
- added REF**1122: Single PTH, SparkFun-Footprints:proto, F.Cu at (101.6, 132.1)
- added REF**1132: Single PTH, SparkFun-Footprints:proto, F.Cu at (104.1, 132.1)
- moved REF** 116.1 mm to (218.4, 134.6)
- moved REF** 112.6 mm to (242.3, 135.1)
- moved REF** 107.7 mm to (195.8, 135.6)
- moved C67 81.3 mm to (94.0, 97.2), turned to 90 degrees
- moved C66 80.5 mm to (115.6, 90.2)
- moved C65 69.5 mm to (117.5, 92.7), turned to 90 degrees
- moved C64 68.7 mm to (115.6, 92.7), turned to 90 degrees
- moved R98 67.6 mm to (89.5, 95.9)
- moved C63 66.1 mm to (97.9, 103.5)
- moved C62 60.4 mm to (128.9, 101.6), turned to 270 degrees
- moved C68 54.7 mm to (154.3, 101.6), turned to 270 degrees
- moved R99 47.9 mm to (78.7, 118.7), turned to 270 degrees
- moved C70 41.4 mm to (81.9, 119.3), turned to 0 degrees
- moved C69 40.4 mm to (89.5, 117.5), turned to 180 degrees
- moved R100 32.3 mm to (90.8, 130.2), turned to 90 degrees
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Connections:
- net Net-(R98-Pad1) renamed SPI_SCK_SRC
- net Net-(R99-Pad1) renamed SPI_MOSI_SRC
- C64 pad 1: I2S_LRCLK -> LRCLK_ISO
- C65 pad 1: I2S_BCLK -> BCLK_ISO
- C66 pad 1: I2S_MCLK -> MCLK_ISO
- JACK1 pad 6: (no net) -> CHASSIS
- JACK1 pad 7: (no net) -> CHASSIS
- JACK2 pad 6: (no net) -> CHASSIS
- JACK2 pad 7: (no net) -> CHASSIS
- JACK3 pad 6: (no net) -> CHASSIS
- JACK3 pad 7: (no net) -> CHASSIS
- P101 pad 1: Net-(P101-Pad1) -> SPI_MISO
- R100 pad 1: Net-(P101-Pad1) -> SPI_MISO_SRC
- REF** pad : GND -> CHASSIS
- U32 pad 2: Net-(P101-Pad1) -> SPI_MISO_SRC
- U6 pad 1: (no net) -> Net-(R102-Pad2)
- U6 pad 8: (no net) -> Net-(R101-Pad2)
Routing:
- net VDD: track 295.4 -> 338.9 mm, vias 12 -> 22
- net LED_OE: track 312.6 -> 287.6 mm, vias 11 -> 12
- net !LED_RST: track 310.8 -> 289.3 mm, vias 10 -> 11
- net +3V3_REG: track 28.9 -> 43.5 mm, vias 0 -> 9
- net +1V8: track 155.8 -> 169.2 mm, vias 4 -> 12
- net VUU: track 24.9 -> 37.7 mm, vias 0 -> 6
- net +3V3: track 286.5 -> 297.7 mm, vias 13 -> 15
- net SPI_SCK: track 380.2 -> 389.9 mm, vias 12 -> 14
- net A: track 356.9 -> 366.6 mm
- net Net-(R102-Pad2): track 0.00 -> 9.13 mm
- net B: track 351.6 -> 360.2 mm
- net KA0: track 200.1 -> 207.8 mm
- net BCLK_ISO: track 51.7 -> 59.0 mm
- net KA1: track 204.6 -> 211.0 mm
- net Net-(C45-Pad1): track 10.9 -> 4.74 mm
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- added copper zone on B.Cu, net +1V8
- added copper zone on B.Cu, net +3V3_REG
- added copper zone on B.Cu, net +5V
- added copper zone on B.Cu, net CHASSIS
- added copper zone on F.Cu, net CHASSIS
- added copper zone on B.Cu, net VUU
Other:
- board text added: "..."
- board text added: "0000"
- board text added: "0001"
- board text added: "0010"
- board text added: "0100"
- board text added: "1110"
- board text added: "1111"
- board text added: "4/10 R43"
- board text added: "5/10 R43"
- board text added: "5/12 R43"
- board text added: "6/12 R43"
- board text added: "6/14 R43"
- board text added: "8/16 R43"
- board text added: "A10"
- board text added: "AEN"
- board text added: "BUS"
- board text added: "BUTTONS"
- board text added: "Co-Teensy"
- board text added: "DCBA"
- board text added: "DISK"
- board text added: "KGND"
- board text added: "KNOBS"
- board text added: "LEDS"
- board text added: "LSB"
- board text added: "MEM"
- board text added: "MSB"
- board text added: "Teensy"
- board text added: "Teensy Audio Carrier"
- board text added: "Teensy Audio Carrier Marshall Taylor V1.0 2016"
- board text added: "VDD"
- board text added: "VKK"
- board text removed: "A14"
- board text removed: "PROTO-8"

Commit message: went to production
Parts:
- removed the REF** at (147.3, 76.2)
- removed the REF** at (169.9, 96.8)
- added G***: Mushroom, SparkFun-Footprints:Mushroom, F.Cu at (147.7, 84.5)
- added JMP30: 2Jumper, SparkFun-Footprints:SF-2way-open, F.Cu at (56.1, 103.6)
- added P113: CONN_01X05, Pin_Headers:Pin_Header_Straight_1x05, F.Cu at (265.4, 132.1)
- added P114: CONN_01X01, SparkFun-Footprints:TestHole, F.Cu at (66.0, 96.5)
- added P115: CONN_01X01, SparkFun-Footprints:TestHole, F.Cu at (61.0, 96.5)
- added REF**: SVIA, SparkFun-Footprints:SVIA, F.Cu at (128.3, 111.5)
- added REF**: SVIA, SparkFun-Footprints:SVIA, F.Cu at (125.7, 101.1)
- added REF**: SVIA, SparkFun-Footprints:SVIA, F.Cu at (111.6, 101.2)
- added REF**: SVIA, SparkFun-Footprints:SVIA, F.Cu at (118.1, 105.5)
- added REF**: SVIA, SparkFun-Footprints:SVIA, F.Cu at (97.0, 111.4)
- added REF**: SVIA, SparkFun-Footprints:SVIA, F.Cu at (99.4, 111.4)
- added REF**: SVIA, SparkFun-Footprints:SVIA, F.Cu at (63.2, 133.3)
- added REF**: SVIA, SparkFun-Footprints:SVIA, F.Cu at (156.2, 132.1)
- added REF**: SVIA, SparkFun-Footprints:SVIA, F.Cu at (260.6, 137.9)
- added REF**: SVIA, SparkFun-Footprints:SVIA, F.Cu at (97.7, 93.2)
- added REF**: SVIA, SparkFun-Footprints:SVIA, F.Cu at (123.3, 88.0)
- added REF**: SVIA, SparkFun-Footprints:SVIA, F.Cu at (54.7, 130.2)
- added REF**: SVIA, SparkFun-Footprints:SVIA, F.Cu at (158.2, 106.8)
- added REF**: SVIA, SparkFun-Footprints:SVIA, F.Cu at (153.8, 104.5)
- added REF**: SVIA, SparkFun-Footprints:SVIA, F.Cu at (122.7, 101.1)
- added REF**: SVIA, SparkFun-Footprints:SVIA, F.Cu at (136.0, 101.7)
- added REF**: SVIA, SparkFun-Footprints:SVIA, F.Cu at (133.7, 105.7)
- U3: footprint teensy footprints:Teensy_3.2_Route -> teensy footprints:Teensy_3.2_Grid
- moved REF** 7.64 mm to (268.5, 137.2)
- moved REF** 4.70 mm to (148.8, 88.3)
- moved REF** 2.62 mm to (62.2, 94.7)
- moved REF** 2.29 mm to (278.1, 52.7)
- moved REF** 1.65 mm to (64.0, 97.4)
- moved REF** 1.48 mm to (57.1, 100.3)
- moved REF** 1.27 mm to (151.8, 90.8)
- moved REF** 0.95 mm to (146.4, 88.3)
- moved REF** 0.85 mm to (61.8, 129.3)
- moved REF** 0.64 mm to (125.7, 90.8)
- moved REF** 0.64 mm to (125.7, 81.3)
- moved REF** 0.64 mm to (125.7, 74.3)
- moved REF** 0.64 mm to (125.7, 87.0)
- moved REF** 0.63 mm to (151.1, 74.3)
- moved REF** 0.63 mm to (151.1, 80.6)
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Connections:
- U3 pad 21: (no net) -> EN
- U3 pad 35: (no net) -> AGND
- U3 pad 48: (no net) -> AREF
- U30 pad 9: (no net) -> Net-(P113-Pad1)
Routing:
- net GND: track 7.66 -> 25.5 mm
- net LED_OE: track 287.6 -> 303.2 mm, vias 12 -> 13
- net SPI_SCK: track 389.9 -> 404.9 mm
- net LED_LATCH: track 316.4 -> 329.2 mm
- net !LED_RST: track 289.3 -> 299.7 mm
- net AGND: track 0.00 -> 9.45 mm, vias 0 -> 1
- net Net-(C45-Pad1): track 4.74 -> 11.2 mm
- net AREF: track 0.00 -> 6.13 mm
- net Net-(P113-Pad1): track 0.00 -> 5.98 mm
- net VBULK: track 76.4 -> 80.8 mm
- net I2S_DOUT1: track 46.8 -> 50.1 mm
- net +3V3: track 297.7 -> 300.6 mm
- net VDD: track 338.9 -> 341.4 mm
- net BOE: track 55.6 -> 58.1 mm
- net +5V: track 501.1 -> 503.6 mm
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Other:
- rule via_min_size: 0.508 -> 0.381
- board text added: "DATA"
- board text added: "LED_LATCH"
- board text added: "LED_OE"
- board text added: "LED_~RST"
- board text added: "SPI_SCK"
- board text added: "Teensy Audio Carrier For PJRC Audio Adaptor Board Expansion Marshall Taylor V1.0 2016"
- board text removed: "Teensy Audio Carrier Marshall Taylor V1.0 2016"
