File: Test Projects/page3.sch (KiCad schematic (older format))
At the start: 1 part, among them U2 Teensy_3.2

Commit message: Tested a few layout sections
Connections:
- net BCLK: now also U2.28 (28,A17); no longer U2.29 (29,SCL1,A18)
- net LEDSER: now reaches U2.31 (31,TX2,A20)
- new net LEDCLK: U2.29 (29,SCL1,A18)
Changed lines of the file:
@@
 Wire Wire Line
 	4950 4800 4850 4800
-Text GLabel 4650 5100 0    50   Input ~ 0
+Text GLabel 4850 5100 0    50   Input ~ 0
 BSER
-Text GLabel 4650 5200 0    50   Input ~ 0
+Text GLabel 4850 5200 0    50   Input ~ 0
 LEDSER
-Text GLabel 4450 5000 0    50   Input ~ 0
+Text GLabel 4850 5000 0    50   Input ~ 0
 LEDCLK
-Text GLabel 4450 4900 0    50   Input ~ 0
+Text GLabel 4850 4900 0    50   Input ~ 0
 BCLK
 Wire Wire Line
-	4450 5000 4950 5000
+	4850 5000 4950 5000
 Wire Wire Line
-	4550 5000 4550 4900
+	4850 5100 4950 5100
 Wire Wire Line
-	4650 5100 4950 5100
+	4950 5200 4850 5200
 Wire Wire Line
-	4750 5200 4650 5200
-Connection ~ 4750 5100
-Wire Wire Line
-	4550 4900 4450 4900
-Connection ~ 4550 5000
-Wire Wire Line
-	4750 5200 4750 5100
+	4950 4900 4850 4900
 $EndSCHEMATC

Commit message: Continued proto 1 layout
Parts:
- added P22, P23, P24, P25, P26: CONN_01X05, Pin_Headers:Pin_Header_Straight_1x05, symbol CONN_01X05
Connections:
- net labels added: KEN
- wire segments 15 -> 16
Changed lines of the file:
@@
 Wire Wire Line
 	4950 4900 4850 4900
+Text GLabel 4850 3600 0    50   Input ~ 0
+KEN
+Wire Wire Line
+	4950 3600 4850 3600
+$Comp
+L CONN_01X05 P22
+U 1 1 568AC10F
+P 7400 2300
+F 0 "P22" H 7400 2600 50  0000 C CNN
+F 1 "CONN_01X05" V 7500 2300 50  0000 C CNN
+F 2 "Pin_Headers:Pin_Header_Straight_1x05" H 7400 2300 50  0001 C CNN
+F 3 "" H 7400 2300 50  0000 C CNN
+	1    7400 2300
+	1    0    0    -1
+$EndComp
+$Comp
+L CONN_01X05 P23
+U 1 1 568AC1B3
+P 7800 2300
+F 0 "P23" H 7800 2600 50  0000 C CNN
+F 1 "CONN_01X05" V 7900 2300 50  0000 C CNN
+F 2 "Pin_Headers:Pin_Header_Straight_1x05" H 7800 2300 50  0001 C CNN
+F 3 "" H 7800 2300 50  0000 C CNN
+	1    7800 2300
+	1    0    0    -1
+$EndComp
+$Comp
+L CONN_01X05 P24
+U 1 1 568AC266
+P 8200 2300
+F 0 "P24" H 8200 2600 50  0000 C CNN
+F 1 "CONN_01X05" V 8300 2300 50  0000 C CNN
+F 2 "Pin_Headers:Pin_Header_Straight_1x05" H 8200 2300 50  0001 C CNN
+F 3 "" H 8200 2300 50  0000 C CNN
+	1    8200 2300
+	1    0    0    -1
+$EndComp
+$Comp
+L CONN_01X05 P25
+U 1 1 568AC26C
+P 8600 2300
+F 0 "P25" H 8600 2600 50  0000 C CNN
+F 1 "CONN_01X05" V 8700 2300 50  0000 C CNN
+F 2 "Pin_Headers:Pin_Header_Straight_1x05" H 8600 2300 50  0001 C CNN
+F 3 "" H 8600 2300 50  0000 C CNN
+	1    8600 2300
+	1    0    0    -1
+$EndComp
+$Comp
+L CONN_01X05 P26
+U 1 1 568AC28F
+P 8950 2300
+F 0 "P26" H 8950 2600 50  0000 C CNN
+F 1 "CONN_01X05" V 9050 2300 50  0000 C CNN
+F 2 "Pin_Headers:Pin_Header_Straight_1x05" H 8950 2300 50  0001 C CNN
+F 3 "" H 8950 2300 50  0000 C CNN
+	1    8950 2300
+	1    0    0    -1
+$EndComp
 $EndSCHEMATC

Commit message: Moved to 10x5 size
Parts:
- removed P22, P23, P24, P25, P26: CONN_01X05, Pin_Headers:Pin_Header_Straight_1x05, symbol CONN_01X05
- removed U2: Teensy_3.2, teensy footprints:Teensy_3.2_Route, symbol Teensy_3.2
Connections:
- net labels removed: BCLK, BSER, KA, KA0, KA1, KA2, KA3, KB, KEN, LEDCLK, LEDSER, PIN14, PIN22, PIN23, SCL0, SDA0
- wire segments 16 -> 0
Changed lines of the file:
@@
 Comment4 ""
 $EndDescr
-$Comp
-L Teensy_3.2 U2
-U 3 1 56886BDD
-P 5750 4100
-F 0 "U2" V 6200 4100 50  0000 C CNN
-F 1 "Teensy_3.2" V 6100 4100 50  0000 C CNN
-F 2 "teensy footprints:Teensy_3.2_Route" H 5450 4400 50  0001 C CNN
-F 3 "" H 5450 4400 50  0000 C CNN
-	3    5750 4100
-	1    0    0    -1
-$EndComp
-Text GLabel 4850 3700 0    50   Input ~ 0
-PIN22
-Text GLabel 4850 3800 0    50   Input ~ 0
-PIN23
-Text GLabel 4850 3300 0    50   Input ~ 0
-SDA0
-Text GLabel 4850 3400 0    50   Input ~ 0
-SCL0
-Wire Wire Line
-	4850 3300 4950 3300
-Wire Wire Line
-	4950 3400 4850 3400
-Wire Wire Line
-	4850 3700 4950 3700
-Wire Wire Line
-	4950 3800 4850 3800
-Text GLabel 4850 2900 0    50   Input ~ 0
-PIN14
-Wire Wire Line
-	4850 2900 4950 2900
-Text GLabel 4850 4000 0    50   Input ~ 0
-KA0
-Text GLabel 4850 4100 0    50   Input ~ 0
-KA1
-Text GLabel 4850 4200 0    50   Input ~ 0
-KA2
-Text GLabel 4850 4300 0    50   Input ~ 0
-KA3
-Wire Wire Line
-	4950 4000 4850 4000
-Wire Wire Line
-	4850 4100 4950 4100
-Wire Wire Line
-	4950 4200 4850 4200
-Wire Wire Line
-	4850 4300 4950 4300
-Text GLabel 4850 4700 0    50   Input ~ 0
-KA
-Text GLabel 4850 4800 0    50   Input ~ 0
-KB
-Wire Wire Line
-	4850 4700 4950 4700
-Wire Wire Line
-	4950 4800 4850 4800
-Text GLabel 4850 5100 0    50   Input ~ 0
-BSER
-Text GLabel 4850 5200 0    50   Input ~ 0
-LEDSER
-Text GLabel 4850 5000 0    50   Input ~ 0
-LEDCLK
-Text GLabel 4850 4900 0    50   Input ~ 0
-BCLK
-Wire Wire Line
-	4850 5000 4950 5000
-Wire Wire Line
-	4850 5100 4950 5100
-Wire Wire Line
-	4950 5200 4850 5200
-Wire Wire Line
-	4950 4900 4850 4900
-Text GLabel 4850 3600 0    50   Input ~ 0
-KEN
-Wire Wire Line
-	4950 3600 4850 3600
-$Comp
-L CONN_01X05 P22
-U 1 1 568AC10F
-P 7400 2300
-F 0 "P22" H 7400 2600 50  0000 C CNN
-F 1 "CONN_01X05" V 7500 2300 50  0000 C CNN
-F 2 "Pin_Headers:Pin_Header_Straight_1x05" H 7400 2300 50  0001 C CNN
-F 3 "" H 7400 2300 50  0000 C CNN
-	1    7400 2300
-	1    0    0    -1
-$EndComp
-$Comp
-L CONN_01X05 P23
-U 1 1 568AC1B3
-P 7800 2300
-F 0 "P23" H 7800 2600 50  0000 C CNN
-F 1 "CONN_01X05" V 7900 2300 50  0000 C CNN
-F 2 "Pin_Headers:Pin_Header_Straight_1x05" H 7800 2300 50  0001 C CNN
-F 3 "" H 7800 2300 50  0000 C CNN
-	1    7800 2300
-	1    0    0    -1
-$EndComp
-$Comp
-L CONN_01X05 P24
-U 1 1 568AC266
-P 8200 2300
-F 0 "P24" H 8200 2600 50  0000 C CNN
-F 1 "CONN_01X05" V 8300 2300 50  0000 C CNN
-F 2 "Pin_Headers:Pin_Header_Straight_1x05" H 8200 2300 50  0001 C CNN
-F 3 "" H 8200 2300 50  0000 C CNN
-	1    8200 2300
-	1    0    0    -1
-$EndComp
-$Comp
-L CONN_01X05 P25
-U 1 1 568AC26C
-P 8600 2300
-F 0 "P25" H 8600 2600 50  0000 C CNN
-F 1 "CONN_01X05" V 8700 2300 50  0000 C CNN
-F 2 "Pin_Headers:Pin_Header_Straight_1x05" H 8600 2300 50  0001 C CNN
-F 3 "" H 8600 2300 50  0000 C CNN
-	1    8600 2300
-	1    0    0    -1
-$EndComp
-$Comp
-L CONN_01X05 P26
-U 1 1 568AC28F
-P 8950 2300
-F 0 "P26" H 8950 2600 50  0000 C CNN
-F 1 "CONN_01X05" V 9050 2300 50  0000 C CNN
-F 2 "Pin_Headers:Pin_Header_Straight_1x05" H 8950 2300 50  0001 C CNN
-F 3 "" H 8950 2300 50  0000 C CNN
-	1    8950 2300
-	1    0    0    -1
-$EndComp
 $EndSCHEMATC

Commit message: Added holes, moved layout
Parts:
- added P13, P14, P15, P16, P17, P18, P19, P20, P40, P41, P42, P43, P44, P45, P46, P47, P48, P49, P50, P51, P52, P53, P54, P55: CONN_01X08, Pin_Headers:Pin_Header_Straight_1x08, symbol CONN_01X08
Connections:
- new net K1: P13.1 (P1)
- new net K10: P14.2 (P2)
- new net K11: P14.3 (P3)
- new net K12: P14.4 (P4)
- new net K13: P14.5 (P5)
- new net K14: P14.6 (P6)
- new net K15: P14.7 (P7)
- new net K16: P14.8 (P8)
- new net K17: P15.1 (P1)
- new net K18: P15.2 (P2)
- new net K19: P15.3 (P3)
- new net K2: P13.2 (P2)
- new net K20: P15.4 (P4)
- new net K21: P15.5 (P5)
- new net K22: P15.6 (P6)
- new net K23: P15.7 (P7)
- new net K24: P15.8 (P8)
- new net K25: P16.1 (P1)
- new net K26: P16.2 (P2)
- new net K27: P16.3 (P3)
- new net K28: P16.4 (P4)
- new net K29: P16.5 (P5)
- new net K3: P13.3 (P3)
- new net K30: P16.6 (P6)
- new net K31: P16.7 (P7)
- new net K32: P16.8 (P8)
- new net K33: P17.1 (P1)
- new net K34: P17.2 (P2)
- new net K35: P17.3 (P3)
- new net K36: P17.4 (P4)
- new net K37: P17.5 (P5)
- new net K38: P17.6 (P6)
- new net K39: P17.7 (P7)
- new net K4: P13.4 (P4)
- new net K40: P17.8 (P8)
- new net K41: P18.1 (P1)
- new net K42: P18.2 (P2)
- new net K43: P18.3 (P3)
- new net K44: P18.4 (P4)
- new net K45: P18.5 (P5)
- new net K46: P18.6 (P6)
- new net K47: P18.7 (P7)
- new net K48: P18.8 (P8)
- new net K49: P19.1 (P1)
- new net K5: P13.5 (P5)
- new net K50: P19.2 (P2)
- new net K51: P19.3 (P3)
- new net K52: P19.4 (P4)
- new net K53: P19.5 (P5)
- new net K54: P19.6 (P6)
- new net K55: P19.7 (P7)
- new net K56: P19.8 (P8)
- new net K57: P20.1 (P1)
- new net K58: P20.2 (P2)
- new net K59: P20.3 (P3)
- new net K6: P13.6 (P6)
- new net K60: P20.4 (P4)
- new net K61: P20.5 (P5)
- new net K62: P20.6 (P6)
- new net K63: P20.7 (P7)
- new net K64: P20.8 (P8)
- new net K7: P13.7 (P7)
- new net K8: P13.8 (P8)
- new net K9: P14.1 (P1)
- new net KGND: P48.1 (P1), P48.2 (P2), P48.3 (P3), P48.4 (P4), P48.5 (P5), P48.6 (P6), P48.7 (P7), P48.8 (P8), P49.1 (P1), P49.2 (P2), P49.3 (P3), P49.4 (P4), P49.5 (P5), P49.6 (P6), P49.7 (P7), P49.8 (P8), P50.1 (P1), P50.2 (P2), P50.3 (P3), P50.4 (P4), P50.5 (P5), P50.6 (P6), P50.7 (P7), P50.8 (P8), P51.1 (P1), P51.2 (P2), P51.3 (P3), P51.4 (P4), P51.5 (P5), P51.6 (P6), P51.7 (P7), P51.8 (P8), P52.1 (P1), P52.2 (P2), P52.3 (P3), P52.4 (P4), P52.5 (P5), P52.6 (P6), P52.7 (P7), P52.8 (P8), P53.1 (P1), P53.2 (P2), P53.3 (P3), P53.4 (P4), P53.5 (P5), P53.6 (P6), P53.7 (P7), P53.8 (P8), P54.1 (P1), P54.2 (P2), P54.3 (P3), P54.4 (P4), P54.5 (P5), P54.6 (P6), P54.7 (P7), P54.8 (P8), P55.1 (P1), P55.2 (P2), P55.3 (P3), P55.4 (P4), P55.5 (P5), P55.6 (P6), P55.7 (P7), P55.8 (P8)
- new net VKK: P40.1 (P1), P40.2 (P2), P40.3 (P3), P40.4 (P4), P40.5 (P5), P40.6 (P6), P40.7 (P7), P40.8 (P8), P41.1 (P1), P41.2 (P2), P41.3 (P3), P41.4 (P4), P41.5 (P5), P41.6 (P6), P41.7 (P7), P41.8 (P8), P42.1 (P1), P42.2 (P2), P42.3 (P3), P42.4 (P4), P42.5 (P5), P42.6 (P6), P42.7 (P7), P42.8 (P8), P43.1 (P1), P43.2 (P2), P43.3 (P3), P43.4 (P4), P43.5 (P5), P43.6 (P6), P43.7 (P7), P43.8 (P8), P44.1 (P1), P44.2 (P2), P44.3 (P3), P44.4 (P4), P44.5 (P5), P44.6 (P6), P44.7 (P7), P44.8 (P8), P45.1 (P1), P45.2 (P2), P45.3 (P3), P45.4 (P4), P45.5 (P5), P45.6 (P6), P45.7 (P7), P45.8 (P8), P46.1 (P1), P46.2 (P2), P46.3 (P3), P46.4 (P4), P46.5 (P5), P46.6 (P6), P46.7 (P7), P46.8 (P8), P47.1 (P1), P47.2 (P2), P47.3 (P3), P47.4 (P4), P47.5 (P5), P47.6 (P6), P47.7 (P7), P47.8 (P8)

Commit message: Routing, 15%
Parts:
- added P82, P83, P84, P85, P86: CONN_01X01, SparkFun-Footprints:PTH_LUG_.05, symbol CONN_01X01
Connections:
- net KGND: now also P85.1 (P1), P86.1 (P1)
- net VKK: now also P82.1 (P1), P83.1 (P1)
- new net GND: P84.1 (P1)
Changed lines of the file:
@@
 EESchema Schematic File Version 2
+LIBS:Teensy_test_layout-rescue
 LIBS:power
 LIBS:device
@@
 LIBS:SparkFun-Mounting
 LIBS:SparkFun-Opto
+LIBS:SparkFun-Connectors
 LIBS:Teensy_test_layout-cache
 EELAYER 25 0
@@
 Text GLabel 5650 3250 0    60   Input ~ 0
 KGND
+Text GLabel 6200 2000 0    50   Input ~ 0
+VKK
+Text GLabel 6200 2200 0    50   Input ~ 0
+VKK
+Text GLabel 6200 3250 0    60   Input ~ 0
+KGND
+Text GLabel 6200 3450 0    60   Input ~ 0
+KGND
+$Comp
+L CONN_01X01 P82
+U 1 1 56A7BE80
+P 6500 2000
+F 0 "P82" H 6500 2100 50  0000 C CNN
+F 1 "CONN_01X01" V 6600 2000 50  0001 C CNN
+F 2 "SparkFun-Footprints:PTH_LUG_.05" H 6500 2000 50  0001 C CNN
+F 3 "" H 6500 2000 50  0000 C CNN
+	1    6500 2000
+	1    0    0    -1
+$EndComp
+$Comp
+L CONN_01X01 P83
+U 1 1 56A7C0E5
+P 6500 2200
+F 0 "P83" H 6500 2300 50  0000 C CNN
+F 1 "CONN_01X01" V 6600 2200 50  0001 C CNN
+F 2 "SparkFun-Footprints:PTH_LUG_.05" H 6500 2200 50  0001 C CNN
+F 3 "" H 6500 2200 50  0000 C CNN
+	1    6500 2200
+	1    0    0    -1
+$EndComp
+$Comp
+L CONN_01X01 P84
+U 1 1 56A7C147
+P 6500 2400
+F 0 "P84" H 6500 2500 50  0000 C CNN
+F 1 "CONN_01X01" V 6600 2400 50  0001 C CNN
+F 2 "SparkFun-Footprints:PTH_LUG_.05" H 6500 2400 50  0001 C CNN
+F 3 "" H 6500 2400 50  0000 C CNN
+	1    6500 2400
+	1    0    0    -1
+$EndComp
+$Comp
+L CONN_01X01 P85
+U 1 1 56A7C1B4
+P 6500 3250
+F 0 "P85" H 6500 3350 50  0000 C CNN
+F 1 "CONN_01X01" V 6600 3250 50  0001 C CNN
+F 2 "SparkFun-Footprints:PTH_LUG_.05" H 6500 3250 50  0001 C CNN
+F 3 "" H 6500 3250 50  0000 C CNN
+	1    6500 3250
+	1    0    0    -1
+$EndComp
+$Comp
+L CONN_01X01 P86
+U 1 1 56A7C236
+P 6500 3450
+F 0 "P86" H 6500 3550 50  0000 C CNN
+F 1 "CONN_01X01" V 6600 3450 50  0001 C CNN
+F 2 "SparkFun-Footprints:PTH_LUG_.05" H 6500 3450 50  0001 C CNN
+F 3 "" H 6500 3450 50  0000 C CNN
+	1    6500 3450
+	1    0    0    -1
+$EndComp
+$Comp
+L GND #PWR032
+U 1 1 56A7CCB1
+P 6200 2500
+F 0 "#PWR032" H 6200 2250 50  0001 C CNN
+F 1 "GND" H 6200 2350 50  0000 C CNN
+F 2 "" H 6200 2500 50  0000 C CNN
+F 3 "" H 6200 2500 50  0000 C CNN
+	1    6200 2500
+	1    0    0    -1
+$EndComp
+Wire Wire Line
+	6200 2500 6200 2400
+Wire Wire Line
+	6200 2400 6300 2400
+Wire Wire Line
+	6200 2200 6300 2200
+Wire Wire Line
+	6200 2000 6300 2000
+Wire Wire Line
+	6200 3250 6300 3250
+Wire Wire Line
+	6200 3450 6300 3450
 $EndSCHEMATC

Commit message: moar layout
Connections:
- net KGND: no longer P52.1 (P1), P52.2 (P2), P52.3 (P3), P52.4 (P4), P52.5 (P5), P52.6 (P6), P52.7 (P7), P52.8 (P8), P53.1 (P1), P53.2 (P2), P53.3 (P3), P53.4 (P4), P53.5 (P5), P53.6 (P6), P53.7 (P7), P53.8 (P8), P54.1 (P1), P54.2 (P2), P54.3 (P3), P54.4 (P4), P54.5 (P5), P54.6 (P6), P54.7 (P7), P54.8 (P8), P55.1 (P1), P55.2 (P2), P55.3 (P3), P55.4 (P4), P55.5 (P5), P55.6 (P6), P55.7 (P7), P55.8 (P8), P86.1 (P1)
- net VKK: no longer P44.1 (P1), P44.2 (P2), P44.3 (P3), P44.4 (P4), P44.5 (P5), P44.6 (P6), P44.7 (P7), P44.8 (P8), P45.1 (P1), P45.2 (P2), P45.3 (P3), P45.4 (P4), P45.5 (P5), P45.6 (P6), P45.7 (P7), P45.8 (P8), P46.1 (P1), P46.2 (P2), P46.3 (P3), P46.4 (P4), P46.5 (P5), P46.6 (P6), P46.7 (P7), P46.8 (P8), P47.1 (P1), P47.2 (P2), P47.3 (P3), P47.4 (P4), P47.5 (P5), P47.6 (P6), P47.7 (P7), P47.8 (P8), P83.1 (P1)
- new net KGND2: P52.1 (P1), P52.2 (P2), P52.3 (P3), P52.4 (P4), P52.5 (P5), P52.6 (P6), P52.7 (P7), P52.8 (P8), P53.1 (P1), P53.2 (P2), P53.3 (P3), P53.4 (P4), P53.5 (P5), P53.6 (P6), P53.7 (P7), P53.8 (P8), P54.1 (P1), P54.2 (P2), P54.3 (P3), P54.4 (P4), P54.5 (P5), P54.6 (P6), P54.7 (P7), P54.8 (P8), P55.1 (P1), P55.2 (P2), P55.3 (P3), P55.4 (P4), P55.5 (P5), P55.6 (P6), P55.7 (P7), P55.8 (P8), P86.1 (P1)
- new net VKK2: P44.1 (P1), P44.2 (P2), P44.3 (P3), P44.4 (P4), P44.5 (P5), P44.6 (P6), P44.7 (P7), P44.8 (P8), P45.1 (P1), P45.2 (P2), P45.3 (P3), P45.4 (P4), P45.5 (P5), P45.6 (P6), P45.7 (P7), P45.8 (P8), P46.1 (P1), P46.2 (P2), P46.3 (P3), P46.4 (P4), P46.5 (P5), P46.6 (P6), P46.7 (P7), P46.8 (P8), P47.1 (P1), P47.2 (P2), P47.3 (P3), P47.4 (P4), P47.5 (P5), P47.6 (P6), P47.7 (P7), P47.8 (P8), P83.1 (P1)
Changed lines of the file:
@@
 LIBS:SparkFun-Mounting
 LIBS:SparkFun-Opto
-LIBS:SparkFun-Connectors
 LIBS:Teensy_test_layout-cache
 EELAYER 25 0
@@
 VKK
 Text GLabel 3850 2000 0    50   Input ~ 0
-VKK
+VKK2
 Text GLabel 4450 2000 0    50   Input ~ 0
-VKK
+VKK2
 Text GLabel 5050 2000 0    50   Input ~ 0
-VKK
+VKK2
 Text GLabel 5650 2000 0    50   Input ~ 0
-VKK
+VKK2
 Text GLabel 1200 3250 0    60   Input ~ 0
 KGND
@@
 KGND
 Text GLabel 3850 3250 0    60   Input ~ 0
-KGND
+KGND2
 Text GLabel 4450 3250 0    60   Input ~ 0
-KGND
+KGND2
 Text GLabel 5050 3250 0    60   Input ~ 0
-KGND
+KGND2
 Text GLabel 5650 3250 0    60   Input ~ 0
-KGND
+KGND2
 Text GLabel 6200 2000 0    50   Input ~ 0
 VKK
 Text GLabel 6200 2200 0    50   Input ~ 0
-VKK
+VKK2
 Text GLabel 6200 3250 0    60   Input ~ 0
 KGND
 Text GLabel 6200 3450 0    60   Input ~ 0
-KGND
+KGND2
 $Comp
 L CONN_01X01 P82
