File: Test Projects/page3.sch (KiCad schematic (older format))
At the start: 29 parts, among them P13 CONN_01X08, P14 CONN_01X08, P15 CONN_01X08, P16 CONN_01X08, P17 CONN_01X08, P18 CONN_01X08, P19 CONN_01X08, P20 CONN_01X08, P40 CONN_01X08, P41 CONN_01X08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

Commit message: layout
Parts:
- added C18, C60: 68uF, Capacitors_Tantalum_SMD:TantalC_SizeC_EIA-6032_Reflow, symbol C
- added C55, C61: 1uF, Capacitors_SMD:C_0603, symbol C
- added P103, P106, P107: CONN_01X01, SparkFun-Footprints:PTH_LUG_.05, symbol CONN_01X01
- added R95, R97: 1, Resistors_SMD:R_0603, symbol R
Connections:
- net GND: now also C18.2, C55.2, C60.2, C61.2, P107.1 (P1)
- new net: C18.1, C55.1, P103.1 (P1), R95.1
- new net: C60.1, C61.1, P106.1 (P1), R97.1
- new net +3v3: R95.2
- new net +5V: R97.2
Other:
- moved on the sheet: P84
Changed lines of the file:
@@
 L CONN_01X01 P84
 U 1 1 56A7C147
-P 6500 2400
-F 0 "P84" H 6500 2500 50  0000 C CNN
-F 1 "CONN_01X01" V 6600 2400 50  0001 C CNN
-F 2 "SparkFun-Footprints:PTH_LUG_.05" H 6500 2400 50  0001 C CNN
-F 3 "" H 6500 2400 50  0000 C CNN
-	1    6500 2400
+P 8700 2400
+F 0 "P84" H 8700 2500 50  0000 C CNN
+F 1 "CONN_01X01" V 8800 2400 50  0001 C CNN
+F 2 "SparkFun-Footprints:PTH_LUG_.05" H 8700 2400 50  0001 C CNN
+F 3 "" H 8700 2400 50  0000 C CNN
+	1    8700 2400
 	1    0    0    -1
 $EndComp
@@
 $EndComp
 $Comp
-L GND #PWR033
+L GND #PWR040
 U 1 1 56A7CCB1
-P 6200 2500
-F 0 "#PWR033" H 6200 2250 50  0001 C CNN
-F 1 "GND" H 6200 2350 50  0000 C CNN
-F 2 "" H 6200 2500 50  0000 C CNN
-F 3 "" H 6200 2500 50  0000 C CNN
-	1    6200 2500
-	1    0    0    -1
-$EndComp
-Wire Wire Line
-	6200 2500 6200 2400
-Wire Wire Line
-	6200 2400 6300 2400
+P 8400 2500
+F 0 "#PWR040" H 8400 2250 50  0001 C CNN
+F 1 "GND" H 8400 2350 50  0000 C CNN
+F 2 "" H 8400 2500 50  0000 C CNN
+F 3 "" H 8400 2500 50  0000 C CNN
+	1    8400 2500
+	1    0    0    -1
+$EndComp
+Wire Wire Line
+	8400 2500 8400 2400
+Wire Wire Line
+	8400 2400 8500 2400
 Wire Wire Line
 	6200 2200 6300 2200
@@
 Wire Wire Line
 	6200 3450 6300 3450
+$Comp
+L CONN_01X01 P103
+U 1 1 56B038F2
+P 8700 2000
+F 0 "P103" H 8700 2100 50  0000 C CNN
+F 1 "CONN_01X01" V 8800 2000 50  0001 C CNN
+F 2 "SparkFun-Footprints:PTH_LUG_.05" H 8700 2000 50  0001 C CNN
+F 3 "" H 8700 2000 50  0000 C CNN
+	1    8700 2000
+	1    0    0    -1
+$EndComp
+Text GLabel 7250 2000 0    60   Input ~ 0
++3v3
+$Comp
+L C C18
+U 1 1 56B039EF
+P 7700 2250
+F 0 "C18" H 7725 2350 50  0000 L CNN
+F 1 "68uF" H 7725 2150 50  0000 L CNN
+F 2 "Capacitors_Tantalum_SMD:TantalC_SizeC_EIA-6032_Reflow" H 7738 2100 50  0001 C CNN
+F 3 "" H 7700 2250 50  0000 C CNN
+	1    7700 2250
+	1    0    0    -1
+$EndComp
+$Comp
+L GND #PWR041
+U 1 1 56B03E1C
+P 7700 2500
+F 0 "#PWR041" H 7700 2250 50  0001 C CNN
+F 1 "GND" H 7700 2350 50  0000 C CNN
+F 2 "" H 7700 2500 50  0000 C CNN
+F 3 "" H 7700 2500 50  0000 C CNN
+	1    7700 2500
+	1    0    0    -1
+$EndComp
+$Comp
+L R R95
+U 1 1 56B03E67
+P 7500 2000
+F 0 "R95" V 7580 2000 50  0000 C CNN
+F 1 "1" V 7500 2000 50  0000 C CNN
+F 2 "Resistors_SMD:R_0603" V 7430 2000 50  0001 C CNN
+F 3 "" H 7500 2000 50  0000 C CNN
+	1    7500 2000
+	0    1    1    0
+$EndComp
+Wire Wire Line
+	7250 2000 7350 2000
+Wire Wire Line
+	7700 2500 7700 2400
+Wire Wire Line
+	7650 2000 8500 2000
+Wire Wire Line
+	7700 2100 7700 2000
+Connection ~ 7700 2000
+$Comp
+L C C55
+U 1 1 56B04874
+P 8050 2250
+F 0 "C55" H 8075 2350 50  0000 L CNN
+F 1 "1uF" H 8075 2150 50  0000 L CNN
+F 2 "Capacitors_SMD:C_0603" H 8088 2100 50  0001 C CNN
+F 3 "" H 8050 2250 50  0000 C CNN
+	1    8050 2250
+	1    0    0    -1
+$EndComp
+$Comp
+L GND #PWR042
+U 1 1 56B04B01
+P 8050 2500
+F 0 "#PWR042" H 8050 2250 50  0001 C CNN
+F 1 "GND" H 8050 2350 50  0000 C CNN
+F 2 "" H 8050 2500 50  0000 C CNN
+F 3 "" H 8050 2500 50  0000 C CNN
+	1    8050 2500
+	1    0    0    -1
+$EndComp
+Wire Wire Line
+	8050 2100 8050 2000
+Connection ~ 8050 2000
+Wire Wire Line
+	8050 2500 8050 2400
+$Comp
+L CONN_01X01 P107
+U 1 1 56B07216
+P 8700 3450
+F 0 "P107" H 8700 3550 50  0000 C CNN
+F 1 "CONN_01X01" V 8800 3450 50  0001 C CNN
+F 2 "SparkFun-Footprints:PTH_LUG_.05" H 8700 3450 50  0001 C CNN
+F 3 "" H 8700 3450 50  0000 C CNN
+	1    8700 3450
+	1    0    0    -1
+$EndComp
+$Comp
+L GND #PWR043
+U 1 1 56B0721C
+P 8400 3550
+F 0 "#PWR043" H 8400 3300 50  0001 C CNN
+F 1 "GND" H 8400 3400 50  0000 C CNN
+F 2 "" H 8400 3550 50  0000 C CNN
+F 3 "" H 8400 3550 50  0000 C CNN
+	1    8400 3550
+	1    0    0    -1
+$EndComp
+Wire Wire Line
+	8400 3550 8400 3450
+Wire Wire Line
+	8400 3450 8500 3450
+$Comp
+L CONN_01X01 P106
+U 1 1 56B07224
+P 8700 3050
+F 0 "P106" H 8700 3150 50  0000 C CNN
+F 1 "CONN_01X01" V 8800 3050 50  0001 C CNN
+F 2 "SparkFun-Footprints:PTH_LUG_.05" H 8700 3050 50  0001 C CNN
+F 3 "" H 8700 3050 50  0000 C CNN
+	1    8700 3050
+	1    0    0    -1
+$EndComp
+Text GLabel 7250 3050 0    60   Input ~ 0
++5V
+$Comp
+L C C60
+U 1 1 56B0722B
+P 7700 3300
+F 0 "C60" H 7725 3400 50  0000 L CNN
+F 1 "68uF" H 7725 3200 50  0000 L CNN
+F 2 "Capacitors_Tantalum_SMD:TantalC_SizeC_EIA-6032_Reflow" H 7738 3150 50  0001 C CNN
+F 3 "" H 7700 3300 50  0000 C CNN
+	1    7700 3300
+	1    0    0    -1
+$EndComp
+$Comp
+L GND #PWR044
+U 1 1 56B07231
+P 7700 3550
+F 0 "#PWR044" H 7700 3300 50  0001 C CNN
+F 1 "GND" H 7700 3400 50  0000 C CNN
+F 2 "" H 7700 3550 50  0000 C CNN
+F 3 "" H 7700 3550 50  0000 C CNN
+	1    7700 3550
+	1    0    0    -1
+$EndComp
+$Comp
+L R R97
+U 1 1 56B07237
+P 7500 3050
+F 0 "R97" V 7580 3050 50  0000 C CNN
+F 1 "1" V 7500 3050 50  0000 C CNN
+F 2 "Resistors_SMD:R_0603" V 7430 3050 50  0001 C CNN
+F 3 "" H 7500 3050 50  0000 C CNN
+	1    7500 3050
+	0    1    1    0
+$EndComp
+Wire Wire Line
+	7250 3050 7350 3050
+Wire Wire Line
+	7700 3550 7700 3450
+Wire Wire Line
+	7650 3050 8500 3050
+Wire Wire Line
+	7700 3150 7700 3050
+Connection ~ 7700 3050
+$Comp
+L C C61
+U 1 1 56B07242
+P 8050 3300
+F 0 "C61" H 8075 3400 50  0000 L CNN
+F 1 "1uF" H 8075 3200 50  0000 L CNN
+F 2 "Capacitors_SMD:C_0603" H 8088 3150 50  0001 C CNN
+F 3 "" H 8050 3300 50  0000 C CNN
+	1    8050 3300
+	1    0    0    -1
+$EndComp
+$Comp
+L GND #PWR045
+U 1 1 56B07248
+P 8050 3550
+F 0 "#PWR045" H 8050 3300 50  0001 C CNN
+F 1 "GND" H 8050 3400 50  0000 C CNN
+F 2 "" H 8050 3550 50  0000 C CNN
+F 3 "" H 8050 3550 50  0000 C CNN
+	1    8050 3550
+	1    0    0    -1
+$EndComp
+Wire Wire Line
+	8050 3150 8050 3050
+Connection ~ 8050 3050
+Wire Wire Line
+	8050 3550 8050 3450
 $EndSCHEMATC
