File: Test Projects/page7.sch (KiCad schematic (older format))
At the start: 73 parts, among them P2 CONN_01X03, P30 CONN_01X03, P38 CONN_01X06, P39 CONN_01X06, P64 DIN1, P65 DOUT1, P66 SDA0_ISO, P67 SCL0_ISO, P68 MCLK_ISO, P69 BCLK_ISO, P70 LRCLK_ISO, P71 DIN0, P72 DOUT0, P91 SDA0, P92 SCL0, P93 MCLK, P94 BCLK, P95 LRCLK, P96 DIN1_ISO, P97 DOUT1_ISO, P98 DIN0_ISO, P99 DOUT0_ISO, U31 SGTL5000, U5 SGTL5000

Commit message: layout
Parts:
- added C62, C63, C64, C65, C66, C67, C68: 22p, Capacitors_SMD:C_0603, symbol C
- added JMP21, JMP29: 2Jumper, SparkFun-Footprints:SF-2way-open, symbol 2Jumper
- added P109: SCL_ISO, SparkFun-Footprints:TestHole, symbol CONN_01X01
- added P110: SDA_ISO, SparkFun-Footprints:TestHole, symbol CONN_01X01
- added P111: SCL_ISO2, SparkFun-Footprints:TestHole, symbol CONN_01X01
- added P112: SDA_ISO2, SparkFun-Footprints:TestHole, symbol CONN_01X01
Connections:
- net GND: now also C62.2, C63.2, C64.2, C65.2, C66.2, C67.2, C68.2
- net I2S_BCLK: now also C65.1
- net I2S_DIN0_ISO: now also C68.1
- net I2S_DIN1_ISO: now also C62.1
- net I2S_DOUT0: now also C67.1
- net I2S_DOUT1: now also C63.1
- net I2S_LRCLK: now also C64.1
- net I2S_MCLK: now also C66.1
- net SCL0: now also JMP29.1, P109.1 (P1); no longer JMP23.1, P92.1 (P1)
- net SDA0: now also JMP21.1, P110.1 (P1); no longer JMP22.1, P91.1 (P1)
- net SCL_ISO renamed SCL12
- net SCL12: no longer U31.29 (SCL)
- net SDA_ISO renamed SDA12
- net SDA12: no longer U31.27 (SDA)
- new net SCL34: JMP23.1, JMP29.2, P111.1 (P1), P92.1 (P1), U31.29 (SCL)
- new net SDA34: JMP21.2, JMP22.1, P112.1 (P1), P91.1 (P1), U31.27 (SDA)
Other:
- moved on the sheet: C37, C38, C39, C40, C41, C46, C47, C48, C49, C50, C51, C52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

Commit message: Finished artwork
Connections:
- net BCLK_ISO: now also C65.1
- net I2S_BCLK: no longer C65.1
- net I2S_LRCLK: no longer C64.1
- net I2S_MCLK: no longer C66.1
- net LRCLK_ISO: now also C64.1
- net MCLK_ISO: now also C66.1
Changed lines of the file:
@@
 I2S_DOUT0
 $Comp
-L +1V8 #PWR0127
+L +1V8 #PWR0129
 U 1 1 569EDC07
 P 4500 3550
-F 0 "#PWR0127" H 4500 3400 50  0001 C CNN
+F 0 "#PWR0129" H 4500 3400 50  0001 C CNN
 F 1 "+1V8" H 4500 3690 50  0000 C CNN
 F 2 "" H 4500 3550 50  0000 C CNN
@@
 $EndComp
 $Comp
-L +3V3 #PWR0128
+L +3V3 #PWR0130
 U 1 1 569EDC0D
 P 4850 3550
-F 0 "#PWR0128" H 4850 3400 50  0001 C CNN
+F 0 "#PWR0130" H 4850 3400 50  0001 C CNN
 F 1 "+3V3" H 4850 3690 50  0000 C CNN
 F 2 "" H 4850 3550 50  0000 C CNN
@@
 $EndComp
 $Comp
-L +3V3 #PWR0129
+L +3V3 #PWR0131
 U 1 1 569EDC13
 P 5050 3550
-F 0 "#PWR0129" H 5050 3400 50  0001 C CNN
+F 0 "#PWR0131" H 5050 3400 50  0001 C CNN
 F 1 "+3V3" H 5050 3690 50  0000 C CNN
 F 2 "" H 5050 3550 50  0000 C CNN
@@
 $EndComp
 $Comp
-L +3V3 #PWR0130
+L +3V3 #PWR0132
 U 1 1 569EDC19
 P 3350 6050
-F 0 "#PWR0130" H 3350 5900 50  0001 C CNN
+F 0 "#PWR0132" H 3350 5900 50  0001 C CNN
 F 1 "+3V3" H 3350 6190 50  0000 C CNN
 F 2 "" H 3350 6050 50  0000 C CNN
@@
 I2S_DOUT1
 $Comp
-L +1V8 #PWR0131
+L +1V8 #PWR0133
 U 1 1 569EE133
 P 9350 2550
-F 0 "#PWR0131" H 9350 2400 50  0001 C CNN
+F 0 "#PWR0133" H 9350 2400 50  0001 C CNN
 F 1 "+1V8" H 9350 2690 50  0000 C CNN
 F 2 "" H 9350 2550 50  0000 C CNN
@@
 $EndComp
 $Comp
-L +3V3 #PWR0132
+L +3V3 #PWR0134
 U 1 1 569EE139
 P 9700 2550
-F 0 "#PWR0132" H 9700 2400 50  0001 C CNN
+F 0 "#PWR0134" H 9700 2400 50  0001 C CNN
 F 1 "+3V3" H 9700 2690 50  0000 C CNN
 F 2 "" H 9700 2550 50  0000 C CNN
@@
 $EndComp
 $Comp
-L +3V3 #PWR0133
+L +3V3 #PWR0135
 U 1 1 569EE13F
 P 9900 2550
-F 0 "#PWR0133" H 9900 2400 50  0001 C CNN
+F 0 "#PWR0135" H 9900 2400 50  0001 C CNN
 F 1 "+3V3" H 9900 2690 50  0000 C CNN
 F 2 "" H 9900 2550 50  0000 C CNN
@@
 $EndComp
 $Comp
-L +3V3 #PWR0134
+L +3V3 #PWR0136
 U 1 1 569EE145
 P 8200 5050
-F 0 "#PWR0134" H 8200 4900 50  0001 C CNN
+F 0 "#PWR0136" H 8200 4900 50  0001 C CNN
 F 1 "+3V3" H 8200 5190 50  0000 C CNN
 F 2 "" H 8200 5050 50  0000 C CNN
@@
 $EndComp
 $Comp
-L GND #PWR0135
+L GND #PWR0137
 U 1 1 56AEF939
 P 4800 7500
-F 0 "#PWR0135" H 4800 7250 50  0001 C CNN
+F 0 "#PWR0137" H 4800 7250 50  0001 C CNN
 F 1 "GND" H 4800 7350 50  0000 C CNN
 F 2 "" H 4800 7500 50  0000 C CNN
@@
 $EndComp
 $Comp
-L GND #PWR0136
+L GND #PWR0138
 U 1 1 56AEFA07
 P 8100 6200
-F 0 "#PWR0136" H 8100 5950 50  0001 C CNN
+F 0 "#PWR0138" H 8100 5950 50  0001 C CNN
 F 1 "GND" H 8100 6050 50  0000 C CNN
 F 2 "" H 8100 6200 50  0000 C CNN
@@
 	4150 6200 3950 6200
 Wire Wire Line
-	3950 6750 3950 6200
+	3950 6200 3950 6750
 Wire Wire Line
 	3500 6400 3600 6400
@@
 	9000 5200 8800 5200
 Wire Wire Line
-	8800 5750 8800 5200
+	8800 5200 8800 5750
 Wire Wire Line
 	8350 5400 8450 5400
@@
 Connection ~ 8050 4050
 Text GLabel 1000 6400 0    50   Input ~ 0
-I2S_MCLK
+MCLK_ISO
 Text GLabel 1000 6600 0    50   Input ~ 0
-I2S_BCLK
+BCLK_ISO
 Text GLabel 1000 6800 0    50   Input ~ 0
-I2S_LRCLK
+LRCLK_ISO
 $Comp
 L C C64
@@
 $EndComp
 $Comp
-L GND #PWR0137
+L GND #PWR0139
 U 1 1 56B1CDC7
 P 1150 7250
-F 0 "#PWR0137" H 1150 7000 50  0001 C CNN
+F 0 "#PWR0139" H 1150 7000 50  0001 C CNN
 F 1 "GND" H 1150 7100 50  0000 C CNN
 F 2 "" H 1150 7250 50  0000 C CNN
@@
 $EndComp
 $Comp
-L GND #PWR0138
+L GND #PWR0140
 U 1 1 56B1CEB0
 P 1500 7250
-F 0 "#PWR0138" H 1500 7000 50  0001 C CNN
+F 0 "#PWR0140" H 1500 7000 50  0001 C CNN
 F 1 "GND" H 1500 7100 50  0000 C CNN
 F 2 "" H 1500 7250 50  0000 C CNN
@@
 $EndComp
 $Comp
-L GND #PWR0139
+L GND #PWR0141
 U 1 1 56B1CF99
 P 1850 7250
-F 0 "#PWR0139" H 1850 7000 50  0001 C CNN
+F 0 "#PWR0141" H 1850 7000 50  0001 C CNN
 F 1 "GND" H 1850 7100 50  0000 C CNN
 F 2 "" H 1850 7250 50  0000 C CNN
@@
 $EndComp
 $Comp
-L GND #PWR0140
+L GND #PWR0142
 U 1 1 56B1DFF3
 P 2300 7500
-F 0 "#PWR0140" H 2300 7250 50  0001 C CNN
+F 0 "#PWR0142" H 2300 7250 50  0001 C CNN
 F 1 "GND" H 2300 7350 50  0000 C CNN
 F 2 "" H 2300 7500 50  0000 C CNN
@@
 $EndComp
 $Comp
-L GND #PWR0141
+L GND #PWR0143
 U 1 1 56B1E9D4
 P 3900 7500
-F 0 "#PWR0141" H 3900 7250 50  0001 C CNN
+F 0 "#PWR0143" H 3900 7250 50  0001 C CNN
 F 1 "GND" H 3900 7350 50  0000 C CNN
 F 2 "" H 3900 7500 50  0000 C CNN
@@
 $EndComp
 $Comp
-L GND #PWR0142
+L GND #PWR0144
 U 1 1 56B1F4B9
 P 6550 6100
-F 0 "#PWR0142" H 6550 5850 50  0001 C CNN
+F 0 "#PWR0144" H 6550 5850 50  0001 C CNN
 F 1 "GND" H 6550 5950 50  0000 C CNN
 F 2 "" H 6550 6100 50  0000 C CNN
@@
 $EndComp
 $Comp
-L GND #PWR0143
+L GND #PWR0145
 U 1 1 56B1F4C9
 P 7650 5700
-F 0 "#PWR0143" H 7650 5450 50  0001 C CNN
+F 0 "#PWR0145" H 7650 5450 50  0001 C CNN
 F 1 "GND" H 7650 5550 50  0000 C CNN
 F 2 "" H 7650 5700 50  0000 C CNN
