File: Test Projects/page1.sch (KiCad schematic (older format))
At the start: 36 parts, among them P1 CONN_01X02, P56 CONN_01X01, P57 CONN_01X01, P58 VUU, P59 CONN_01X01, P60 CONN_01X01, P61 CONN_01X01, P62 UGND, P63 CONN_01X01, U1 LDO-adj-4term, U2 LDO-adj-4term, U3 Teensy_3.2, U33 LDO-adj-4term, U4 LDO-adj-4term

Commit message: moar layout
Parts:
- added P90: CONN_01X01, Pin_Headers:Pin_Header_Straight_1x01, symbol CONN_01X01
Connections:
- net VBULK: now also P90.1 (P1)
Changed lines of the file:
@@
 LIBS:SparkFun-Mounting
 LIBS:SparkFun-Opto
-LIBS:SparkFun-Connectors
 LIBS:Teensy_test_layout-cache
 EELAYER 25 0
@@
 	1    0    0    -1
 $EndComp
+$Comp
+L CONN_01X01 P90
+U 1 1 56ABFA3B
+P 2400 700
+F 0 "P90" H 2400 800 50  0000 C CNN
+F 1 "CONN_01X01" H 2500 700 50  0001 L CNN
+F 2 "Pin_Headers:Pin_Header_Straight_1x01" H 2400 700 50  0001 C CNN
+F 3 "" H 2400 700 50  0000 C CNN
+	1    2400 700
+	1    0    0    -1
+$EndComp
+Wire Wire Line
+	2000 1150 2000 700
+Wire Wire Line
+	2000 700  2200 700
+Connection ~ 2000 1150
 $EndSCHEMATC

Commit message: layout
Parts:
- added P31, P36: CONN_01X01, SparkFun-Footprints:TestHole, symbol CONN_01X01
Connections:
- net +5V: now also P31.1 (P1)
- net GND: now also P36.1 (P1)
Changed lines of the file:
@@
 LIBS:SparkFun-Mounting
 LIBS:SparkFun-Opto
+LIBS:SparkFun-Connectors
 LIBS:Teensy_test_layout-cache
 EELAYER 25 0
@@
 	2000 700  2200 700
 Connection ~ 2000 1150
+$Comp
+L CONN_01X01 P31
+U 1 1 56AEC633
+P 5200 3050
+F 0 "P31" H 5200 3150 50  0000 C CNN
+F 1 "CONN_01X01" H 5300 3050 50  0001 L CNN
+F 2 "SparkFun-Footprints:TestHole" H 5200 3050 50  0001 C CNN
+F 3 "" H 5200 3050 50  0000 C CNN
+	1    5200 3050
+	1    0    0    -1
+$EndComp
+Wire Wire Line
+	5000 3050 4700 3050
+Connection ~ 4700 3050
+$Comp
+L CONN_01X01 P36
+U 1 1 56AFD601
+P 5200 3250
+F 0 "P36" H 5200 3350 50  0000 C CNN
+F 1 "CONN_01X01" H 5300 3250 50  0001 L CNN
+F 2 "SparkFun-Footprints:TestHole" H 5200 3250 50  0001 C CNN
+F 3 "" H 5200 3250 50  0000 C CNN
+	1    5200 3250
+	1    0    0    -1
+$EndComp
+$Comp
+L GND #PWR019
+U 1 1 56AFDE83
+P 4900 3300
+F 0 "#PWR019" H 4900 3050 50  0001 C CNN
+F 1 "GND" H 4900 3150 50  0000 C CNN
+F 2 "" H 4900 3300 50  0000 C CNN
+F 3 "" H 4900 3300 50  0000 C CNN
+	1    4900 3300
+	1    0    0    -1
+$EndComp
+Wire Wire Line
+	5000 3250 4900 3250
+Wire Wire Line
+	4900 3250 4900 3300
 $EndSCHEMATC

Commit message: layout
Parts:
- added C56, C57: 100u, Capacitors_SMD:c_elec_10x10.5, symbol C
- added C58, C59: 1u, Capacitors_SMD:C_1206, symbol C
- added P104, P105: CONN_01X01, SparkFun-Footprints:TestHole, symbol CONN_01X01
- added R96: 1, Resistors_SMD:R_2512, symbol R
Connections:
- net +1V8: now also P104.1 (P1)
- net +3V3_REG: now also P105.1 (P1)
- net GND: now also P1.1 (P1), C56.2, C57.2, C58.2, C59.2; no longer P1.2 (P2)
- net VBULK: now also C56.1, C57.1, C58.1, C59.1, R96.1; no longer JACK12.PWR, P1.1 (P1)
- new net PWR: JACK12.PWR, P1.2 (P2), R96.2
Other:
- moved on the sheet: P1
Changed lines of the file:
@@
-$EndComp
-$Comp
-L CONN_01X02 P1
-U 1 1 56886EEF
-P 1650 2800
-F 0 "P1" H 1650 2950 50  0000 C CNN
-F 1 "CONN_01X02" V 1750 2800 50  0000 C CNN
-F 2 "Pin_Headers:Pin_Header_Straight_1x02" H 1650 2800 50  0001 C CNN
-F 3 "" H 1650 2800 50  0000 C CNN
-	1    1650 2800
-	-1   0    0    -1
 $EndComp
 $Comp
@@
 $EndComp
 Wire Wire Line
-	1850 2750 2400 2750
-Wire Wire Line
 	3200 2750 3800 2750
 Wire Wire Line
@@
 $Comp
 L GND #PWR01
-U 1 1 56887438
-P 1950 2950
-F 0 "#PWR01" H 1950 2700 50  0001 C CNN
-F 1 "GND" H 1950 2800 50  0000 C CNN
-F 2 "" H 1950 2950 50  0000 C CNN
-F 3 "" H 1950 2950 50  0000 C CNN
-	1    1950 2950
-	1    0    0    -1
-$EndComp
-$Comp
-L GND #PWR02
 U 1 1 56887462
 P 3400 3800
-F 0 "#PWR02" H 3400 3550 50  0001 C CNN
+F 0 "#PWR01" H 3400 3550 50  0001 C CNN
 F 1 "GND" H 3400 3650 50  0000 C CNN
 F 2 "" H 3400 3800 50  0000 C CNN
@@
 $EndComp
 $Comp
-L GND #PWR03
+L GND #PWR02
 U 1 1 56887485
 P 3400 5600
-F 0 "#PWR03" H 3400 5350 50  0001 C CNN
+F 0 "#PWR02" H 3400 5350 50  0001 C CNN
 F 1 "GND" H 3400 5450 50  0000 C CNN
 F 2 "" H 3400 5600 50  0000 C CNN
@@
 $EndComp
 $Comp
-L GND #PWR04
+L GND #PWR03
 U 1 1 568874A8
 P 4900 5200
-F 0 "#PWR04" H 4900 4950 50  0001 C CNN
+F 0 "#PWR03" H 4900 4950 50  0001 C CNN
 F 1 "GND" H 4900 5050 50  0000 C CNN
 F 2 "" H 4900 5200 50  0000 C CNN
@@
 Wire Wire Line
 	3400 3750 3400 3800
-Wire Wire Line
-	1850 2850 1950 2850
-Wire Wire Line
-	1950 2850 1950 2950
 $Comp
 L C C5
@@
 $EndComp
 $Comp
-L GND #PWR05
+L GND #PWR04
 U 1 1 56887D2E
 P 3800 3350
-F 0 "#PWR05" H 3800 3100 50  0001 C CNN
+F 0 "#PWR04" H 3800 3100 50  0001 C CNN
 F 1 "GND" H 3800 3200 50  0000 C CNN
 F 2 "" H 3800 3350 50  0000 C CNN
@@
 $EndComp
 $Comp
-L GND #PWR06
+L GND #PWR05
 U 1 1 56887D63
 P 3800 5050
-F 0 "#PWR06" H 3800 4800 50  0001 C CNN
+F 0 "#PWR05" H 3800 4800 50  0001 C CNN
 F 1 "GND" H 3800 4900 50  0000 C CNN
 F 2 "" H 3800 5050 50  0000 C CNN
@@
 $EndComp
 $Comp
-L GND #PWR07
+L GND #PWR06
 U 1 1 56887D98
 P 2800 5650
-F 0 "#PWR07" H 2800 5400 50  0001 C CNN
+F 0 "#PWR06" H 2800 5400 50  0001 C CNN
 F 1 "GND" H 2800 5500 50  0000 C CNN
 F 2 "" H 2800 5650 50  0000 C CNN
@@
 $EndComp
 $Comp
-L GND #PWR08
+L GND #PWR07
 U 1 1 56887DCD
 P 2200 4950
-F 0 "#PWR08" H 2200 4700 50  0001 C CNN
+F 0 "#PWR07" H 2200 4700 50  0001 C CNN
 F 1 "GND" H 2200 4800 50  0000 C CNN
 F 2 "" H 2200 4950 50  0000 C CNN
@@
 $EndComp
 $Comp
-L GND #PWR09
+L GND #PWR08
 U 1 1 56887E02
 P 2200 3250
-F 0 "#PWR09" H 2200 3000 50  0001 C CNN
+F 0 "#PWR08" H 2200 3000 50  0001 C CNN
 F 1 "GND" H 2200 3100 50  0000 C CNN
 F 2 "" H 2200 3250 50  0000 C CNN
@@
 Connection ~ 2800 3350
 $Comp
-L GND #PWR010
+L GND #PWR09
 U 1 1 56888143
 P 2800 3850
-F 0 "#PWR010" H 2800 3600 50  0001 C CNN
+F 0 "#PWR09" H 2800 3600 50  0001 C CNN
 F 1 "GND" H 2800 3700 50  0000 C CNN
 F 2 "" H 2800 3850 50  0000 C CNN
@@
 Connection ~ 3400 1150
 $Comp
-L GND #PWR011
+L GND #PWR010
 U 1 1 5687E4D5
 P 3400 2300
-F 0 "#PWR011" H 3400 2050 50  0001 C CNN
+F 0 "#PWR010" H 3400 2050 50  0001 C CNN
 F 1 "GND" H 3400 2150 50  0000 C CNN
 F 2 "" H 3400 2300 50  0000 C CNN
@@
 $EndComp
 $Comp
-L GND #PWR012
+L GND #PWR011
 U 1 1 5687E4E8
 P 3800 1950
-F 0 "#PWR012" H 3800 1700 50  0001 C CNN
+F 0 "#PWR011" H 3800 1700 50  0001 C CNN
 F 1 "GND" H 3800 1800 50  0000 C CNN
 F 2 "" H 3800 1950 50  0000 C CNN
@@
 Connection ~ 2800 1850
 $Comp
-L GND #PWR013
+L GND #PWR012
 U 1 1 5687E4F2
 P 2800 2350
-F 0 "#PWR013" H 2800 2100 50  0001 C CNN
+F 0 "#PWR012" H 2800 2100 50  0001 C CNN
 F 1 "GND" H 2800 2200 50  0000 C CNN
 F 2 "" H 2800 2350 50  0000 C CNN
@@
 $EndComp
 $Comp
-L GND #PWR014
+L GND #PWR013
 U 1 1 5687E561
 P 2200 1850
-F 0 "#PWR014" H 2200 1600 50  0001 C CNN
+F 0 "#PWR013" H 2200 1600 50  0001 C CNN
 F 1 "GND" H 2200 1700 50  0000 C CNN
 F 2 "" H 2200 1850 50  0000 C CNN
@@
 	3300 2850 3300 2750
 Connection ~ 3300 2750
-Connection ~ 1950 2750
-$Comp
-L +3V3 #PWR015
+$Comp
+L +3V3 #PWR014
 U 1 1 5687F792
 P 4200 3800
-F 0 "#PWR015" H 4200 3650 50  0001 C CNN
+F 0 "#PWR014" H 4200 3650 50  0001 C CNN
 F 1 "+3V3" H 4200 3940 50  0000 C CNN
 F 2 "" H 4200 3800 50  0000 C CNN
@@
 $EndComp
 $Comp
-L +1V8 #PWR016
+L +1V8 #PWR015
 U 1 1 5687F99A
 P 3800 1000
-F 0 "#PWR016" H 3800 850 50  0001 C CNN
+F 0 "#PWR015" H 3800 850 50  0001 C CNN
 F 1 "+1V8" H 3800 1140 50  0000 C CNN
 F 2 "" H 3800 1000 50  0000 C CNN
@@
 $EndComp
 $Comp
-L +5V #PWR017
+L +5V #PWR016
 U 1 1 56881FFF
 P 3800 2600
-F 0 "#PWR017" H 3800 2450 50  0001 C CNN
+F 0 "#PWR016" H 3800 2450 50  0001 C CNN
 F 1 "+5V" H 3800 2740 50  0000 C CNN
 F 2 "" H 3800 2600 50  0000 C CNN
@@
 VUUIN
 $Comp
-L GND #PWR018
+L GND #PWR017
 U 1 1 56A70829
 P 2300 6850
-F 0 "#PWR018" H 2300 6600 50  0001 C CNN
+F 0 "#PWR017" H 2300 6600 50  0001 C CNN
 F 1 "GND" H 2300 6700 50  0000 C CNN
 F 2 "" H 2300 6850 50  0000 C CNN
@@
 $EndComp
 Wire Wire Line
-	2100 6400 2300 6400
+	2100 6400 2950 6400
 Wire Wire Line
 	2300 6400 2300 5900
@@
 	2300 6600 2100 6600
 Text GLabel 2250 5900 0    50   Input ~ 0
-VBULK
+PWR
 Text GLabel 1950 1850 0    50   UnSpc ~ 0
 VBULK
@@
 $EndComp
 $Comp
-L GND #PWR019
+L GND #PWR018
 U 1 1 56AFDE83
 P 4900 3300
-F 0 "#PWR019" H 4900 3050 50  0001 C CNN
+F 0 "#PWR018" H 4900 3050 50  0001 C CNN
 F 1 "GND" H 4900 3150 50  0000 C CNN
 F 2 "" H 4900 3300 50  0000 C CNN
@@
 Wire Wire Line
 	4900 3250 4900 3300
+Connection ~ 2300 6400
+$Comp
+L CONN_01X02 P1
+U 1 1 56886EEF
+P 3100 6050
+F 0 "P1" H 3100 6200 50  0000 C CNN
+F 1 "CONN_01X02" V 3200 6050 50  0000 C CNN
+F 2 "Pin_Headers:Pin_Header_Straight_1x02" H 3100 6050 50  0001 C CNN
+F 3 "" H 3100 6050 50  0000 C CNN
+	1    3100 6050
+	1    0    0    1
+$EndComp
+Wire Wire Line
+	2700 6400 2700 6000
+Wire Wire Line
+	2700 6000 2900 6000
+Wire Wire Line
+	2900 6100 2850 6100
+Wire Wire Line
+	2850 6100 2850 6150
+$Comp
+L GND #PWR019
+U 1 1 56B0918E
+P 2850 6150
+F 0 "#PWR019" H 2850 5900 50  0001 C CNN
+F 1 "GND" H 2850 6000 50  0000 C CNN
+F 2 "" H 2850 6150 50  0000 C CNN
+F 3 "" H 2850 6150 50  0000 C CNN
+	1    2850 6150
+	1    0    0    -1
+$EndComp
+$Comp
+L R R96
+U 1 1 56B098CC
+P 3100 6400
+F 0 "R96" V 3180 6400 50  0000 C CNN
+F 1 "1" V 3100 6400 50  0000 C CNN
+F 2 "Resistors_SMD:R_2512" V 3030 6400 50  0001 C CNN
+F 3 "" H 3100 6400 50  0000 C CNN
+	1    3100 6400
+	0    1    1    0
+$EndComp
+$Comp
+L C C56
+U 1 1 56B09987
+P 3500 6600
+F 0 "C56" H 3525 6700 50  0000 L CNN
+F 1 "100u" H 3525 6500 50  0000 L CNN
+F 2 "Capacitors_SMD:c_elec_10x10.5" H 3538 6450 50  0001 C CNN
+F 3 "" H 3500 6600 50  0000 C CNN
+	1    3500 6600
+	1    0    0    -1
+$EndComp
+$Comp
+L C C57
+U 1 1 56B09A63
+P 3750 6600
+F 0 "C57" H 3775 6700 50  0000 L CNN
+F 1 "100u" H 3775 6500 50  0000 L CNN
+F 2 "Capacitors_SMD:c_elec_10x10.5" H 3788 6450 50  0001 C CNN
+F 3 "" H 3750 6600 50  0000 C CNN
+	1    3750 6600
+	1    0    0    -1
+$EndComp
+$Comp
+L C C58
+U 1 1 56B09AFB
+P 4000 6600
+F 0 "C58" H 4025 6700 50  0000 L CNN
+F 1 "1u" H 4025 6500 50  0000 L CNN
+F 2 "Capacitors_SMD:C_1206" H 4038 6450 50  0001 C CNN
+F 3 "" H 4000 6600 50  0000 C CNN
+	1    4000 6600
+	1    0    0    -1
+$EndComp
+$Comp
+L C C59
+U 1 1 56B09B92
+P 4250 6600
+F 0 "C59" H 4275 6700 50  0000 L CNN
+F 1 "1u" H 4275 6500 50  0000 L CNN
+F 2 "Capacitors_SMD:C_1206" H 4288 6450 50  0001 C CNN
+F 3 "" H 4250 6600 50  0000 C CNN
+	1    4250 6600
+	1    0    0    -1
+$EndComp
+$Comp
+L GND #PWR020
+U 1 1 56B09C2C
+P 3500 6850
+F 0 "#PWR020" H 3500 6600 50  0001 C CNN
+F 1 "GND" H 3500 6700 50  0000 C CNN
+F 2 "" H 3500 6850 50  0000 C CNN
+F 3 "" H 3500 6850 50  0000 C CNN
+	1    3500 6850
+	1    0    0    -1
+$EndComp
+$Comp
+L GND #PWR021
+U 1 1 56B09CBB
+P 3750 6850
+F 0 "#PWR021" H 3750 6600 50  0001 C CNN
+F 1 "GND" H 3750 6700 50  0000 C CNN
+F 2 "" H 3750 6850 50  0000 C CNN
+F 3 "" H 3750 6850 50  0000 C CNN
+	1    3750 6850
+	1    0    0    -1
+$EndComp
+$Comp
+L GND #PWR022
+U 1 1 56B09D4A
+P 4000 6850
+F 0 "#PWR022" H 4000 6600 50  0001 C CNN
+F 1 "GND" H 4000 6700 50  0000 C CNN
+F 2 "" H 4000 6850 50  0000 C CNN
+F 3 "" H 4000 6850 50  0000 C CNN
+	1    4000 6850
+	1    0    0    -1
+$EndComp
+$Comp
+L GND #PWR023
+U 1 1 56B09DD9
+P 4250 6850
+F 0 "#PWR023" H 4250 6600 50  0001 C CNN
+F 1 "GND" H 4250 6700 50  0000 C CNN
+F 2 "" H 4250 6850 50  0000 C CNN
+F 3 "" H 4250 6850 50  0000 C CNN
+	1    4250 6850
+	1    0    0    -1
+$EndComp
+Connection ~ 2700 6400
+Wire Wire Line
+	3250 6400 4600 6400
+Wire Wire Line
+	4250 6400 4250 6450
+Wire Wire Line
+	4000 6450 4000 6400
+Connection ~ 4000 6400
+Wire Wire Line
+	3750 6450 3750 6400
+Connection ~ 3750 6400
+Wire Wire Line
+	3500 6450 3500 6400
+Connection ~ 3500 6400
+Wire Wire Line
+	3500 6750 3500 6850
+Wire Wire Line
+	3750 6750 3750 6850
+Wire Wire Line
+	4000 6750 4000 6850
+Wire Wire Line
+	4250 6750 4250 6850
+Connection ~ 4250 6400
+Text GLabel 4600 6400 2    50   Input ~ 0
+VBULK
+$Comp
+L CONN_01X01 P104
+U 1 1 56B0CF49
+P 4250 1250
+F 0 "P104" H 4250 1350 50  0000 C CNN
+F 1 "CONN_01X01" H 4350 1250 50  0001 L CNN
+F 2 "SparkFun-Footprints:TestHole" H 4250 1250 50  0001 C CNN
+F 3 "" H 4250 1250 50  0000 C CNN
+	1    4250 1250
+	1    0    0    -1
+$EndComp
+$Comp
+L CONN_01X01 P105
+U 1 1 56B0D2EB
+P 4100 4350
+F 0 "P105" H 4100 4450 50  0000 C CNN
+F 1 "CONN_01X01" H 4200 4350 50  0001 L CNN
+F 2 "SparkFun-Footprints:TestHole" H 4100 4350 50  0001 C CNN
+F 3 "" H 4100 4350 50  0000 C CNN
+	1    4100 4350
+	1    0    0    -1
+$EndComp
+Wire Wire Line
+	3900 4350 3800 4350
+Connection ~ 3800 4350
+Wire Wire Line
+	4050 1250 3800 1250
+Connection ~ 3800 1250
+Wire Wire Line
+	1950 2750 2400 2750
 $EndSCHEMATC

Commit message: went to production
Parts:
- added JMP30: 2Jumper, SparkFun-Footprints:SF-2way-open, symbol 2Jumper
- added P114, P115: CONN_01X01, SparkFun-Footprints:TestHole, symbol CONN_01X01
- U3: footprint teensy footprints:Teensy_3.2_Route -> teensy footprints:Teensy_3.2_Grid
Connections:
- net GND: now also JMP30.1
- net AGND: now reaches U3.35 (AGND)
- net AGND: now also JMP30.2, P115.1 (P1)
- net AREF: now reaches U3.48 (AREF)
- net AREF: now also P114.1 (P1)
Changed lines of the file:
@@
 F 0 "U3" V 6200 4400 50  0000 C CNN
 F 1 "Teensy_3.2" V 6100 4400 50  0000 C CNN
-F 2 "teensy footprints:Teensy_3.2_Route" H 5450 4700 50  0001 C CNN
+F 2 "teensy footprints:Teensy_3.2_Grid" H 5450 4700 50  0001 C CNN
 F 3 "" H 5450 4700 50  0000 C CNN
 	1    5750 4400
@@
 Connection ~ 3400 5150
 Wire Wire Line
-	3200 4450 3800 4450
+	3800 4450 3200 4450
 Wire Wire Line
 	3400 4450 3400 4550
@@
 $EndComp
 Wire Wire Line
-	2200 2850 2200 2750
+	2200 2750 2200 2850
 Connection ~ 2200 2750
 Wire Wire Line
@@
 Wire Wire Line
 	1950 2750 2400 2750
+$Comp
+L CONN_01X01 P115
+U 1 1 56B7744C
+P 4350 4750
+F 0 "P115" H 4350 4850 50  0000 C CNN
+F 1 "CONN_01X01" H 4450 4750 50  0001 L CNN
+F 2 "SparkFun-Footprints:TestHole" H 4350 4750 50  0001 C CNN
+F 3 "" H 4350 4750 50  0000 C CNN
+	1    4350 4750
+	-1   0    0    1
+$EndComp
+$Comp
+L CONN_01X01 P114
+U 1 1 56B7756D
+P 4150 4650
+F 0 "P114" H 4150 4750 50  0000 C CNN
+F 1 "CONN_01X01" H 4250 4650 50  0001 L CNN
+F 2 "SparkFun-Footprints:TestHole" H 4150 4650 50  0001 C CNN
+F 3 "" H 4150 4650 50  0000 C CNN
+	1    4150 4650
+	-1   0    0    1
+$EndComp
+Wire Wire Line
+	4950 4650 4350 4650
+Wire Wire Line
+	4550 4750 4950 4750
+Text GLabel 4600 4650 1    30   Input ~ 0
+AREF
+Text GLabel 4700 4750 1    30   Input ~ 0
+AGND
+$Comp
+L 2Jumper JMP30
+U 1 1 56B7BA60
+P 4600 5150
+F 0 "JMP30" H 4600 5245 60  0000 C CNN
+F 1 "2Jumper" H 4600 5335 60  0001 C CNN
+F 2 "SparkFun-Footprints:SF-2way-open" H 5755 5220 60  0001 C CNN
+F 3 "" H 5755 5220 60  0000 C CNN
+	1    4600 5150
+	0    -1   -1   0
+$EndComp
+$Comp
+L GND #PWR024
+U 1 1 56B7C292
+P 4600 5450
+F 0 "#PWR024" H 4600 5200 50  0001 C CNN
+F 1 "GND" H 4600 5300 50  0000 C CNN
+F 2 "" H 4600 5450 50  0000 C CNN
+F 3 "" H 4600 5450 50  0000 C CNN
+	1    4600 5450
+	1    0    0    -1
+$EndComp
+Wire Wire Line
+	4600 4950 4600 4750
+Connection ~ 4600 4750
+Wire Wire Line
+	4600 5350 4600 5450
 $EndSCHEMATC
