File: Test Projects/page2.sch (KiCad schematic (older format))
At the start: 22 parts, among them P3 COLS0, P31 PIN20, P32 PIN8, P33 SIO2, P34 ~HOLD~/SIO3, P35 PIN37, P36 PIN29, P37 PIN31, P4 COLS1, U3 Teensy_3.2, U32 SPI_MEMORY_SOIC8, U6 SF-MicroSD-12term, U7 SF-74HC595, U8 SF-74HC595

Commit message: moar layout
Parts:
- removed P31: PIN20, SparkFun-Footprints:Single_PTH, symbol CONN_01X01
- removed P36: PIN29, SparkFun-Footprints:Single_PTH, symbol CONN_01X01
Connections:
- net D: now reaches U3.20 (20,PWM,CS,A6)
- net C: now reaches U3.29 (29,SCL1,A18)
- net KA renamed A
- net KB renamed B

Commit message: layout
Parts:
- added P100: SPI_MOSI, SparkFun-Footprints:TestHole, symbol CONN_01X01
- added P101: SPI_MISO, SparkFun-Footprints:TestHole, symbol CONN_01X01
- added P102: SPI_SCK, SparkFun-Footprints:TestHole, symbol CONN_01X01
- P32, P33, P34, P35, P37: footprint SparkFun-Footprints:Single_PTH -> SparkFun-Footprints:TestHole
Connections:
- net SPI_MISO: now also P101.1 (P1)
- net SPI_MOSI: now also P100.1 (P1)
- net SPI_SCK: now also P102.1 (P1)
Changed lines of the file:
@@
 LIBS:SparkFun-Mounting
 LIBS:SparkFun-Opto
+LIBS:SparkFun-Connectors
 LIBS:Teensy_test_layout-cache
 EELAYER 25 0
@@
 SPI_MOSI
 $Comp
-L +3V3 #PWR019
+L +3V3 #PWR020
 U 1 1 568C434E
 P 8350 1550
-F 0 "#PWR019" H 8350 1400 50  0001 C CNN
+F 0 "#PWR020" H 8350 1400 50  0001 C CNN
 F 1 "+3V3" H 8350 1690 50  0000 C CNN
 F 2 "" H 8350 1550 50  0000 C CNN
@@
 $EndComp
 $Comp
-L +3V3 #PWR020
+L +3V3 #PWR021
 U 1 1 568C4354
 P 8150 1550
-F 0 "#PWR020" H 8150 1400 50  0001 C CNN
+F 0 "#PWR021" H 8150 1400 50  0001 C CNN
 F 1 "+3V3" H 8150 1690 50  0000 C CNN
 F 2 "" H 8150 1550 50  0000 C CNN
@@
 F 0 "P32" H 5850 2650 50  0000 C CNN
 F 1 "PIN8" H 5650 2650 50  0000 C CNN
-F 2 "SparkFun-Footprints:Single_PTH" H 5500 2650 50  0001 C CNN
+F 2 "SparkFun-Footprints:TestHole" H 5500 2650 50  0001 C CNN
 F 3 "" H 5500 2650 50  0000 C CNN
 	1    5500 2650
@@
 F 0 "P35" H 9200 3150 50  0000 C CNN
 F 1 "PIN37" H 9000 3150 50  0000 C CNN
-F 2 "SparkFun-Footprints:Single_PTH" H 8800 3150 50  0001 C CNN
+F 2 "SparkFun-Footprints:TestHole" H 8800 3150 50  0001 C CNN
 F 3 "" H 8800 3150 50  0000 C CNN
 	1    8800 3150
@@
 $EndComp
 $Comp
-L GND #PWR021
+L GND #PWR022
 U 1 1 56A0F405
 P 3750 1950
-F 0 "#PWR021" H 3750 1700 50  0001 C CNN
+F 0 "#PWR022" H 3750 1700 50  0001 C CNN
 F 1 "GND" H 3750 1800 50  0000 C CNN
 F 2 "" H 3750 1950 50  0000 C CNN
@@
 $EndComp
 $Comp
-L GND #PWR022
+L GND #PWR023
 U 1 1 56A0F6ED
 P 3500 3750
-F 0 "#PWR022" H 3500 3500 50  0001 C CNN
+F 0 "#PWR023" H 3500 3500 50  0001 C CNN
 F 1 "GND" H 3500 3600 50  0000 C CNN
 F 2 "" H 3500 3750 50  0000 C CNN
@@
 $EndComp
 $Comp
-L GND #PWR023
+L GND #PWR024
 U 1 1 56A0FB18
 P 2700 7400
-F 0 "#PWR023" H 2700 7150 50  0001 C CNN
+F 0 "#PWR024" H 2700 7150 50  0001 C CNN
 F 1 "GND" H 2700 7250 50  0000 C CNN
 F 2 "" H 2700 7400 50  0000 C CNN
@@
 $EndComp
 $Comp
-L GND #PWR024
+L GND #PWR025
 U 1 1 56A0FBC8
 P 5200 7400
-F 0 "#PWR024" H 5200 7150 50  0001 C CNN
+F 0 "#PWR025" H 5200 7150 50  0001 C CNN
 F 1 "GND" H 5200 7250 50  0000 C CNN
 F 2 "" H 5200 7400 50  0000 C CNN
@@
 $EndComp
 $Comp
-L +3V3 #PWR025
+L +3V3 #PWR026
 U 1 1 56A0FE25
 P 3500 1400
-F 0 "#PWR025" H 3500 1250 50  0001 C CNN
+F 0 "#PWR026" H 3500 1250 50  0001 C CNN
 F 1 "+3V3" H 3500 1540 50  0000 C CNN
 F 2 "" H 3500 1400 50  0000 C CNN
@@
 $EndComp
 $Comp
-L +3V3 #PWR026
+L +3V3 #PWR027
 U 1 1 56A104A5
 P 2700 6300
-F 0 "#PWR026" H 2700 6150 50  0001 C CNN
+F 0 "#PWR027" H 2700 6150 50  0001 C CNN
 F 1 "+3V3" H 2700 6440 50  0000 C CNN
 F 2 "" H 2700 6300 50  0000 C CNN
@@
 $EndComp
 $Comp
-L +3V3 #PWR027
+L +3V3 #PWR028
 U 1 1 56A105FA
 P 5200 6300
-F 0 "#PWR027" H 5200 6150 50  0001 C CNN
+F 0 "#PWR028" H 5200 6150 50  0001 C CNN
 F 1 "+3V3" H 5200 6440 50  0000 C CNN
 F 2 "" H 5200 6300 50  0000 C CNN
@@
 Connection ~ 5200 6350
 Connection ~ 5200 7350
-Text GLabel 2700 2850 0    50   Input ~ 0
+Text GLabel 2500 2850 0    50   Input ~ 0
 RAM_CS
 Wire Wire Line
-	2800 2850 2700 2850
-Text GLabel 2700 2550 0    50   Input ~ 0
+	2800 2850 2500 2850
+Text GLabel 1700 2550 0    50   Input ~ 0
 SPI_MOSI
-Text GLabel 2700 3150 0    50   Input ~ 0
+Text GLabel 2500 3150 0    50   Input ~ 0
 SPI_SCK
-Text GLabel 2700 2650 0    50   Input ~ 0
+Text GLabel 1700 2650 0    50   Input ~ 0
 SPI_MISO
 $Comp
-L +3V3 #PWR028
+L +3V3 #PWR029
 U 1 1 56A12235
 P 2150 2000
-F 0 "#PWR028" H 2150 1850 50  0001 C CNN
+F 0 "#PWR029" H 2150 1850 50  0001 C CNN
 F 1 "+3V3" H 2150 2140 50  0000 C CNN
 F 2 "" H 2150 2000 50  0000 C CNN
@@
 $EndComp
 $Comp
-L +3V3 #PWR029
+L +3V3 #PWR030
 U 1 1 56A12282
 P 1950 2000
-F 0 "#PWR029" H 1950 1850 50  0001 C CNN
+F 0 "#PWR030" H 1950 1850 50  0001 C CNN
 F 1 "+3V3" H 1950 2140 50  0000 C CNN
 F 2 "" H 1950 2000 50  0000 C CNN
@@
 F 0 "P33" H 2100 2750 50  0000 C CNN
 F 1 "SIO2" H 1850 2750 50  0000 C CNN
-F 2 "SparkFun-Footprints:Single_PTH" H 1650 2750 50  0001 C CNN
+F 2 "SparkFun-Footprints:TestHole" H 1650 2750 50  0001 C CNN
 F 3 "" H 1650 2750 50  0000 C CNN
 	1    1650 2750
@@
 F 0 "P34" H 2500 2950 50  0000 C CNN
 F 1 "~HOLD~/SIO3" H 2150 2950 50  0000 C CNN
-F 2 "SparkFun-Footprints:Single_PTH" H 1850 2950 50  0001 C CNN
+F 2 "SparkFun-Footprints:TestHole" H 1850 2950 50  0001 C CNN
 F 3 "" H 1850 2950 50  0000 C CNN
 	1    1850 2950
@@
 Connection ~ 2150 2950
 Wire Wire Line
-	2700 3150 2800 3150
-Wire Wire Line
-	2700 2650 2800 2650
-Wire Wire Line
-	2700 2550 2800 2550
-$Comp
-L +3V3 #PWR030
+	2500 3150 2800 3150
+Wire Wire Line
+	1700 2650 2800 2650
+Wire Wire Line
+	1700 2550 2800 2550
+$Comp
+L +3V3 #PWR031
 U 1 1 56A16EA5
 P 1200 5150
-F 0 "#PWR030" H 1200 5000 50  0001 C CNN
+F 0 "#PWR031" H 1200 5000 50  0001 C CNN
 F 1 "+3V3" H 1200 5290 50  0000 C CNN
 F 2 "" H 1200 5150 50  0000 C CNN
@@
 $EndComp
 $Comp
-L +3V3 #PWR031
+L +3V3 #PWR032
 U 1 1 56A16EFE
 P 3750 5100
-F 0 "#PWR031" H 3750 4950 50  0001 C CNN
+F 0 "#PWR032" H 3750 4950 50  0001 C CNN
 F 1 "+3V3" H 3750 5240 50  0000 C CNN
 F 2 "" H 3750 5100 50  0000 C CNN
@@
 F 0 "P37" H 9200 3850 50  0000 C CNN
 F 1 "PIN31" H 9000 3850 50  0000 C CNN
-F 2 "SparkFun-Footprints:Single_PTH" H 8800 3850 50  0001 C CNN
+F 2 "SparkFun-Footprints:TestHole" H 8800 3850 50  0001 C CNN
 F 3 "" H 8800 3850 50  0000 C CNN
 	1    8800 3850
@@
 Text GLabel 9000 2150 0    50   Input ~ 0
 D
+$Comp
+L CONN_01X01 P100
+U 1 1 56AFECCB
+P 2400 2100
+F 0 "P100" H 2850 2100 50  0000 C CNN
+F 1 "SPI_MOSI" H 2600 2100 50  0000 C CNN
+F 2 "SparkFun-Footprints:TestHole" H 2400 2100 50  0001 C CNN
+F 3 "" H 2400 2100 50  0000 C CNN
+	1    2400 2100
+	0    1    -1   0
+$EndComp
+$Comp
+L CONN_01X01 P101
+U 1 1 56AFED56
+P 2550 2100
+F 0 "P101" H 3000 2100 50  0000 C CNN
+F 1 "SPI_MISO" H 2750 2100 50  0000 C CNN
+F 2 "SparkFun-Footprints:TestHole" H 2550 2100 50  0001 C CNN
+F 3 "" H 2550 2100 50  0000 C CNN
+	1    2550 2100
+	0    1    -1   0
+$EndComp
+$Comp
+L CONN_01X01 P102
+U 1 1 56AFEDB8
+P 2700 2100
+F 0 "P102" H 3150 2100 50  0000 C CNN
+F 1 "SPI_SCK" H 2900 2100 50  0000 C CNN
+F 2 "SparkFun-Footprints:TestHole" H 2700 2100 50  0001 C CNN
+F 3 "" H 2700 2100 50  0000 C CNN
+	1    2700 2100
+	0    1    -1   0
+$EndComp
+Wire Wire Line
+	2400 2300 2400 2550
+Connection ~ 2400 2550
+Wire Wire Line
+	2550 2300 2550 2650
+Connection ~ 2550 2650
+Wire Wire Line
+	2700 2300 2700 3150
+Connection ~ 2700 3150
 $EndSCHEMATC

Commit message: layout
Parts:
- added C69, C70, C71: 22p, Capacitors_SMD:C_0603, symbol C
- added R100, R98, R99: 50, Resistors_SMD:R_0603, symbol R
Connections:
- net GND: now also C69.2, C70.2, C71.2
- net SPI_MISO: now also C69.1, R100.2; no longer P101.1 (P1), U32.2 (SO/SIO1)
- net SPI_MOSI: now also C70.1, R99.2; no longer U3.7 (7,DOUT,RX3)
- net SPI_SCK: now also C71.1, R98.2; no longer U3.14 (14,SCK,A0)
- new net: R99.1, U3.7 (7,DOUT,RX3)
- new net: R98.1, U3.14 (14,SCK,A0)
- new net: P101.1 (P1), R100.1, U32.2 (SO/SIO1)
Other:
- moved on the sheet: P33, P34
Changed lines of the file:
@@
 Text GLabel 5700 2850 0    50   Input ~ 0
 SD_CS
-Text GLabel 5700 3050 0    50   Input ~ 0
+Text GLabel 4750 3050 0    50   Input ~ 0
 SPI_MISO
 $Comp
@@
 Text GLabel 8050 2050 0    50   Input ~ 0
 SCL0
-Text GLabel 9000 1550 0    50   Input ~ 0
+Text GLabel 8250 1250 0    50   Input ~ 0
 SPI_SCK
 Text GLabel 9000 2650 0    50   Input ~ 0
@@
 Text Notes 6500 1350 0    75   ~ 0
 I2C Assignment-\n  I2C0 codec config, misc devices (expansion)\nSPI\n  SD card\n  RAM/ROM\n  LEDs\n
-Text GLabel 5700 2550 0    50   Input ~ 0
+Text GLabel 4450 2550 0    50   Input ~ 0
 SPI_MOSI
 $Comp
-L +3V3 #PWR020
+L +3V3 #PWR024
 U 1 1 568C434E
 P 8350 1550
-F 0 "#PWR020" H 8350 1400 50  0001 C CNN
+F 0 "#PWR024" H 8350 1400 50  0001 C CNN
 F 1 "+3V3" H 8350 1690 50  0000 C CNN
 F 2 "" H 8350 1550 50  0000 C CNN
@@
 $EndComp
 $Comp
-L +3V3 #PWR021
+L +3V3 #PWR025
 U 1 1 568C4354
 P 8150 1550
-F 0 "#PWR021" H 8150 1400 50  0001 C CNN
+F 0 "#PWR025" H 8150 1400 50  0001 C CNN
 F 1 "+3V3" H 8150 1690 50  0000 C CNN
 F 2 "" H 8150 1550 50  0000 C CNN
@@
 $EndComp
 $Comp
-L GND #PWR022
+L GND #PWR026
 U 1 1 56A0F405
 P 3750 1950
-F 0 "#PWR022" H 3750 1700 50  0001 C CNN
+F 0 "#PWR026" H 3750 1700 50  0001 C CNN
 F 1 "GND" H 3750 1800 50  0000 C CNN
 F 2 "" H 3750 1950 50  0000 C CNN
@@
 $EndComp
 $Comp
-L GND #PWR023
+L GND #PWR027
 U 1 1 56A0F6ED
 P 3500 3750
-F 0 "#PWR023" H 3500 3500 50  0001 C CNN
+F 0 "#PWR027" H 3500 3500 50  0001 C CNN
 F 1 "GND" H 3500 3600 50  0000 C CNN
 F 2 "" H 3500 3750 50  0000 C CNN
@@
 $EndComp
 $Comp
-L GND #PWR024
+L GND #PWR028
 U 1 1 56A0FB18
 P 2700 7400
-F 0 "#PWR024" H 2700 7150 50  0001 C CNN
+F 0 "#PWR028" H 2700 7150 50  0001 C CNN
 F 1 "GND" H 2700 7250 50  0000 C CNN
 F 2 "" H 2700 7400 50  0000 C CNN
@@
 $EndComp
 $Comp
-L GND #PWR025
+L GND #PWR029
 U 1 1 56A0FBC8
 P 5200 7400
-F 0 "#PWR025" H 5200 7150 50  0001 C CNN
+F 0 "#PWR029" H 5200 7150 50  0001 C CNN
 F 1 "GND" H 5200 7250 50  0000 C CNN
 F 2 "" H 5200 7400 50  0000 C CNN
@@
 $EndComp
 $Comp
-L +3V3 #PWR026
+L +3V3 #PWR030
 U 1 1 56A0FE25
 P 3500 1400
-F 0 "#PWR026" H 3500 1250 50  0001 C CNN
+F 0 "#PWR030" H 3500 1250 50  0001 C CNN
 F 1 "+3V3" H 3500 1540 50  0000 C CNN
 F 2 "" H 3500 1400 50  0000 C CNN
@@
 $EndComp
 $Comp
-L +3V3 #PWR027
+L +3V3 #PWR031
 U 1 1 56A104A5
 P 2700 6300
-F 0 "#PWR027" H 2700 6150 50  0001 C CNN
+F 0 "#PWR031" H 2700 6150 50  0001 C CNN
 F 1 "+3V3" H 2700 6440 50  0000 C CNN
 F 2 "" H 2700 6300 50  0000 C CNN
@@
 $EndComp
 $Comp
-L +3V3 #PWR028
+L +3V3 #PWR032
 U 1 1 56A105FA
 P 5200 6300
-F 0 "#PWR028" H 5200 6150 50  0001 C CNN
+F 0 "#PWR032" H 5200 6150 50  0001 C CNN
 F 1 "+3V3" H 5200 6440 50  0000 C CNN
 F 2 "" H 5200 6300 50  0000 C CNN
@@
 	9100 2250 9000 2250
 Wire Wire Line
-	5800 3050 5700 3050
+	4750 3050 5800 3050
 Wire Wire Line
 	9000 1750 9100 1750
@@
 	5800 2350 5700 2350
 Wire Wire Line
-	9100 1550 9000 1550
-Wire Wire Line
-	5800 2550 5700 2550
+	8250 1250 8600 1250
+Wire Wire Line
+	4750 2550 4450 2550
 Wire Wire Line
 	9000 3750 9100 3750
@@
 Connection ~ 5200 6350
 Connection ~ 5200 7350
-Text GLabel 2500 2850 0    50   Input ~ 0
+Text GLabel 1050 2850 0    50   Input ~ 0
 RAM_CS
 Wire Wire Line
-	2800 2850 2500 2850
-Text GLabel 1700 2550 0    50   Input ~ 0
+	2800 2850 1050 2850
+Text GLabel 1050 2550 0    50   Input ~ 0
 SPI_MOSI
-Text GLabel 2500 3150 0    50   Input ~ 0
+Text GLabel 1050 3150 0    50   Input ~ 0
 SPI_SCK
-Text GLabel 1700 2650 0    50   Input ~ 0
+Text GLabel 1050 2650 0    50   Input ~ 0
 SPI_MISO
 $Comp
-L +3V3 #PWR029
+L +3V3 #PWR033
 U 1 1 56A12235
 P 2150 2000
-F 0 "#PWR029" H 2150 1850 50  0001 C CNN
+F 0 "#PWR033" H 2150 1850 50  0001 C CNN
 F 1 "+3V3" H 2150 2140 50  0000 C CNN
 F 2 "" H 2150 2000 50  0000 C CNN
@@
 $EndComp
 $Comp
-L +3V3 #PWR030
+L +3V3 #PWR034
 U 1 1 56A12282
 P 1950 2000
-F 0 "#PWR030" H 1950 1850 50  0001 C CNN
+F 0 "#PWR034" H 1950 1850 50  0001 C CNN
 F 1 "+3V3" H 1950 2140 50  0000 C CNN
 F 2 "" H 1950 2000 50  0000 C CNN
@@
 L CONN_01X01 P33
 U 1 1 56A12B3B
-P 1650 2750
-F 0 "P33" H 2100 2750 50  0000 C CNN
-F 1 "SIO2" H 1850 2750 50  0000 C CNN
-F 2 "SparkFun-Footprints:TestHole" H 1650 2750 50  0001 C CNN
-F 3 "" H 1650 2750 50  0000 C CNN
-	1    1650 2750
+P 850 2750
+F 0 "P33" H 1300 2750 50  0000 C CNN
+F 1 "SIO2" H 1050 2750 50  0000 C CNN
+F 2 "SparkFun-Footprints:TestHole" H 850 2750 50  0001 C CNN
+F 3 "" H 850 2750 50  0000 C CNN
+	1    850  2750
 	-1   0    0    -1
 $EndComp
@@
 L CONN_01X01 P34
 U 1 1 56A12E0B
-P 1850 2950
-F 0 "P34" H 2500 2950 50  0000 C CNN
-F 1 "~HOLD~/SIO3" H 2150 2950 50  0000 C CNN
-F 2 "SparkFun-Footprints:TestHole" H 1850 2950 50  0001 C CNN
-F 3 "" H 1850 2950 50  0000 C CNN
-	1    1850 2950
+P 850 2950
+F 0 "P34" H 1500 2950 50  0000 C CNN
+F 1 "~HOLD~/SIO3" H 1150 2950 50  0000 C CNN
+F 2 "SparkFun-Footprints:TestHole" H 850 2950 50  0001 C CNN
+F 3 "" H 850 2950 50  0000 C CNN
+	1    850  2950
 	-1   0    0    -1
 $EndComp
@@
 	2150 2000 2150 2100
 Wire Wire Line
-	1850 2750 2800 2750
-Wire Wire Line
-	2050 2950 2800 2950
+	1050 2750 2800 2750
+Wire Wire Line
+	1050 2950 2800 2950
 Wire Wire Line
 	1950 2500 1950 2750
@@
 Connection ~ 2150 2950
 Wire Wire Line
-	2500 3150 2800 3150
-Wire Wire Line
-	1700 2650 2800 2650
-Wire Wire Line
-	1700 2550 2800 2550
-$Comp
-L +3V3 #PWR031
+	1050 3150 2800 3150
+Wire Wire Line
+	1050 2650 1300 2650
+Wire Wire Line
+	1050 2550 2800 2550
+$Comp
+L +3V3 #PWR035
 U 1 1 56A16EA5
 P 1200 5150
-F 0 "#PWR031" H 1200 5000 50  0001 C CNN
+F 0 "#PWR035" H 1200 5000 50  0001 C CNN
 F 1 "+3V3" H 1200 5290 50  0000 C CNN
 F 2 "" H 1200 5150 50  0000 C CNN
@@
 $EndComp
 $Comp
-L +3V3 #PWR032
+L +3V3 #PWR036
 U 1 1 56A16EFE
 P 3750 5100
-F 0 "#PWR032" H 3750 4950 50  0001 C CNN
+F 0 "#PWR036" H 3750 4950 50  0001 C CNN
 F 1 "+3V3" H 3750 5240 50  0000 C CNN
 F 2 "" H 3750 5100 50  0000 C CNN
@@
 	2700 2300 2700 3150
 Connection ~ 2700 3150
+$Comp
+L C C69
+U 1 1 56B26147
+P 4900 3500
+F 0 "C69" H 4925 3600 50  0000 L CNN
+F 1 "22p" H 4925 3400 50  0000 L CNN
+F 2 "Capacitors_SMD:C_0603" H 4938 3350 50  0001 C CNN
+F 3 "" H 4900 3500 50  0000 C CNN
+	1    4900 3500
+	1    0    0    -1
+$EndComp
+$Comp
+L C C70
+U 1 1 56B2614E
+P 2300 3800
+F 0 "C70" H 2325 3900 50  0000 L CNN
+F 1 "22p" H 2325 3700 50  0000 L CNN
+F 2 "Capacitors_SMD:C_0603" H 2338 3650 50  0001 C CNN
+F 3 "" H 2300 3800 50  0000 C CNN
+	1    2300 3800
+	1    0    0    -1
+$EndComp
+$Comp
+L C C71
+U 1 1 56B26155
+P 2650 3800
+F 0 "C71" H 2675 3900 50  0000 L CNN
+F 1 "22p" H 2675 3700 50  0000 L CNN
+F 2 "Capacitors_SMD:C_0603" H 2688 3650 50  0001 C CNN
+F 3 "" H 2650 3800 50  0000 C CNN
+	1    2650 3800
+	1    0    0    -1
+$EndComp
+$Comp
+L GND #PWR037
+U 1 1 56B2615C
+P 4900 3700
+F 0 "#PWR037" H 4900 3450 50  0001 C CNN
+F 1 "GND" H 4900 3550 50  0000 C CNN
+F 2 "" H 4900 3700 50  0000 C CNN
+F 3 "" H 4900 3700 50  0000 C CNN
+	1    4900 3700
+	1    0    0    -1
+$EndComp
+$Comp
+L GND #PWR038
+U 1 1 56B26162
+P 2300 4000
+F 0 "#PWR038" H 2300 3750 50  0001 C CNN
+F 1 "GND" H 2300 3850 50  0000 C CNN
+F 2 "" H 2300 4000 50  0000 C CNN
+F 3 "" H 2300 4000 50  0000 C CNN
+	1    2300 4000
+	1    0    0    -1
+$EndComp
+$Comp
+L GND #PWR039
+U 1 1 56B26168
+P 2650 4000
+F 0 "#PWR039" H 2650 3750 50  0001 C CNN
+F 1 "GND" H 2650 3850 50  0000 C CNN
+F 2 "" H 2650 4000 50  0000 C CNN
+F 3 "" H 2650 4000 50  0000 C CNN
+	1    2650 4000
+	1    0    0    -1
+$EndComp
+Wire Wire Line
+	2650 3950 2650 4000
+Wire Wire Line
+	2300 3950 2300 4000
+Wire Wire Line
+	4900 3650 4900 3700
+Wire Wire Line
+	2650 3650 2650 3150
+Connection ~ 2650 3150
+Wire Wire Line
+	2300 3650 2300 2550
+Connection ~ 2300 2550
+Wire Wire Line
+	4900 3350 4900 3050
+Connection ~ 4900 3050
+$Comp
+L R R98
+U 1 1 56B27256
+P 8750 1250
+F 0 "R98" V 8830 1250 50  0000 C CNN
+F 1 "50" V 8750 1250 50  0000 C CNN
+F 2 "Resistors_SMD:R_0603" V 8680 1250 50  0001 C CNN
+F 3 "" H 8750 1250 50  0000 C CNN
+	1    8750 1250
+	0    1    1    0
+$EndComp
+Wire Wire Line
+	8900 1250 9000 1250
+Wire Wire Line
+	9000 1250 9000 1550
+Wire Wire Line
+	9000 1550 9100 1550
+$Comp
+L R R99
+U 1 1 56B274BB
+P 4900 2550
+F 0 "R99" V 4980 2550 50  0000 C CNN
+F 1 "50" V 4900 2550 50  0000 C CNN
+F 2 "Resistors_SMD:R_0603" V 4830 2550 50  0001 C CNN
+F 3 "" H 4900 2550 50  0000 C CNN
+	1    4900 2550
+	0    1    1    0
+$EndComp
+Wire Wire Line
+	5050 2550 5800 2550
+$Comp
+L R R100
+U 1 1 56B281EA
+P 1450 2650
+F 0 "R100" V 1530 2650 50  0000 C CNN
+F 1 "50" V 1450 2650 50  0000 C CNN
+F 2 "Resistors_SMD:R_0603" V 1380 2650 50  0001 C CNN
+F 3 "" H 1450 2650 50  0000 C CNN
+	1    1450 2650
+	0    1    1    0
+$EndComp
+Wire Wire Line
+	2800 2650 1600 2650
 $EndSCHEMATC

Commit message: Finished artwork
Parts:
- added R101, R102: 4.7k, Resistors_SMD:R_0603, symbol R
Connections:
- net +3V3: now also R101.1, R102.1
- net SPI_MISO: now also P101.1 (P1)
- net at U6.1 (NC): now also R102.2
- net at U6.8 (RSV): now also R101.2
- net SPI_MOSI_SRC: now reaches R99.1, U3.7 (7,DOUT,RX3)
- net SPI_SCK_SRC: now reaches R98.1, U3.14 (14,SCK,A0)
- net SPI_MISO_SRC: now reaches R100.1, U32.2 (SO/SIO1)
- net SPI_MISO_SRC: no longer P101.1 (P1)
Other:
- moved on the sheet: P101, P3, P4, R100, R98, ROWS1, U6A, U6B, U7A, U8A

Commit message: went to production
Parts:
- U3: footprint teensy footprints:Teensy_3.2_Route -> teensy footprints:Teensy_3.2_Grid
Connections:
- net KEN renamed EN
Changed lines of the file:
@@
 F 0 "U3" V 7050 2800 50  0000 C CNN
 F 1 "Teensy_3.2" V 6950 2800 50  0000 C CNN
-F 2 "teensy footprints:Teensy_3.2_Route" H 6300 3100 50  0001 C CNN
+F 2 "teensy footprints:Teensy_3.2_Grid" H 6300 3100 50  0001 C CNN
 F 3 "" H 6300 3100 50  0000 C CNN
 	2    6600 2800
@@
 F 0 "U3" V 10350 2750 50  0000 C CNN
 F 1 "Teensy_3.2" V 10250 2750 50  0000 C CNN
-F 2 "teensy footprints:Teensy_3.2_Route" H 9600 3050 50  0001 C CNN
+F 2 "teensy footprints:Teensy_3.2_Grid" H 9600 3050 50  0001 C CNN
 F 3 "" H 9600 3050 50  0000 C CNN
 	3    9900 2750
@@
 BSER
 Text GLabel 9000 2250 0    50   Input ~ 0
-KEN
+EN
 Text GLabel 5700 2950 0    50   Input ~ 0
 I2S_MCLK
@@
 SPI_MOSI
 $Comp
-L +3V3 #PWR024
+L +3V3 #PWR025
 U 1 1 568C434E
 P 8350 1550
-F 0 "#PWR024" H 8350 1400 50  0001 C CNN
+F 0 "#PWR025" H 8350 1400 50  0001 C CNN
 F 1 "+3V3" H 8350 1690 50  0000 C CNN
 F 2 "" H 8350 1550 50  0000 C CNN
@@
 $EndComp
 $Comp
-L +3V3 #PWR025
+L +3V3 #PWR026
 U 1 1 568C4354
 P 8150 1550
-F 0 "#PWR025" H 8150 1400 50  0001 C CNN
+F 0 "#PWR026" H 8150 1400 50  0001 C CNN
 F 1 "+3V3" H 8150 1690 50  0000 C CNN
 F 2 "" H 8150 1550 50  0000 C CNN
@@
 $EndComp
 $Comp
-L GND #PWR026
+L GND #PWR027
 U 1 1 56A0F405
 P 3750 1950
-F 0 "#PWR026" H 3750 1700 50  0001 C CNN
+F 0 "#PWR027" H 3750 1700 50  0001 C CNN
 F 1 "GND" H 3750 1800 50  0000 C CNN
 F 2 "" H 3750 1950 50  0000 C CNN
@@
 $EndComp
 $Comp
-L GND #PWR027
+L GND #PWR028
 U 1 1 56A0F6ED
 P 3500 3750
-F 0 "#PWR027" H 3500 3500 50  0001 C CNN
+F 0 "#PWR028" H 3500 3500 50  0001 C CNN
 F 1 "GND" H 3500 3600 50  0000 C CNN
 F 2 "" H 3500 3750 50  0000 C CNN
@@
 $EndComp
 $Comp
-L GND #PWR028
+L GND #PWR029
 U 1 1 56A0FB18
 P 2700 7400
-F 0 "#PWR028" H 2700 7150 50  0001 C CNN
+F 0 "#PWR029" H 2700 7150 50  0001 C CNN
 F 1 "GND" H 2700 7250 50  0000 C CNN
 F 2 "" H 2700 7400 50  0000 C CNN
@@
 $EndComp
 $Comp
-L GND #PWR029
+L GND #PWR030
 U 1 1 56A0FBC8
 P 5200 7400
-F 0 "#PWR029" H 5200 7150 50  0001 C CNN
+F 0 "#PWR030" H 5200 7150 50  0001 C CNN
 F 1 "GND" H 5200 7250 50  0000 C CNN
 F 2 "" H 5200 7400 50  0000 C CNN
@@
 $EndComp
 $Comp
-L +3V3 #PWR030
+L +3V3 #PWR031
 U 1 1 56A0FE25
 P 3500 1400
-F 0 "#PWR030" H 3500 1250 50  0001 C CNN
+F 0 "#PWR031" H 3500 1250 50  0001 C CNN
 F 1 "+3V3" H 3500 1540 50  0000 C CNN
 F 2 "" H 3500 1400 50  0000 C CNN
@@
 $EndComp
 $Comp
-L +3V3 #PWR031
+L +3V3 #PWR032
 U 1 1 56A104A5
 P 2700 6300
-F 0 "#PWR031" H 2700 6150 50  0001 C CNN
+F 0 "#PWR032" H 2700 6150 50  0001 C CNN
 F 1 "+3V3" H 2700 6440 50  0000 C CNN
 F 2 "" H 2700 6300 50  0000 C CNN
@@
 $EndComp
 $Comp
-L +3V3 #PWR032
+L +3V3 #PWR033
 U 1 1 56A105FA
 P 5200 6300
-F 0 "#PWR032" H 5200 6150 50  0001 C CNN
+F 0 "#PWR033" H 5200 6150 50  0001 C CNN
 F 1 "+3V3" H 5200 6440 50  0000 C CNN
 F 2 "" H 5200 6300 50  0000 C CNN
@@
 SPI_MISO
 $Comp
-L +3V3 #PWR033
+L +3V3 #PWR034
 U 1 1 56A12235
 P 2150 2000
-F 0 "#PWR033" H 2150 1850 50  0001 C CNN
+F 0 "#PWR034" H 2150 1850 50  0001 C CNN
 F 1 "+3V3" H 2150 2140 50  0000 C CNN
 F 2 "" H 2150 2000 50  0000 C CNN
@@
 $EndComp
 $Comp
-L +3V3 #PWR034
+L +3V3 #PWR035
 U 1 1 56A12282
 P 1950 2000
-F 0 "#PWR034" H 1950 1850 50  0001 C CNN
+F 0 "#PWR035" H 1950 1850 50  0001 C CNN
 F 1 "+3V3" H 1950 2140 50  0000 C CNN
 F 2 "" H 1950 2000 50  0000 C CNN
@@
 $EndComp
 $Comp
-L +3V3 #PWR035
+L +3V3 #PWR036
 U 1 1 56A16EA5
 P 1200 4850
-F 0 "#PWR035" H 1200 4700 50  0001 C CNN
+F 0 "#PWR036" H 1200 4700 50  0001 C CNN
 F 1 "+3V3" H 1200 4990 50  0000 C CNN
 F 2 "" H 1200 4850 50  0000 C CNN
@@
 $EndComp
 $Comp
-L +3V3 #PWR036
+L +3V3 #PWR037
 U 1 1 56A16EFE
 P 3750 4800
-F 0 "#PWR036" H 3750 4650 50  0001 C CNN
+F 0 "#PWR037" H 3750 4650 50  0001 C CNN
 F 1 "+3V3" H 3750 4940 50  0000 C CNN
 F 2 "" H 3750 4800 50  0000 C CNN
@@
 $EndComp
 $Comp
-L GND #PWR037
+L GND #PWR038
 U 1 1 56B2615C
 P 4900 3700
-F 0 "#PWR037" H 4900 3450 50  0001 C CNN
+F 0 "#PWR038" H 4900 3450 50  0001 C CNN
 F 1 "GND" H 4900 3550 50  0000 C CNN
 F 2 "" H 4900 3700 50  0000 C CNN
@@
 $EndComp
 $Comp
-L GND #PWR038
+L GND #PWR039
 U 1 1 56B26162
 P 2300 4000
-F 0 "#PWR038" H 2300 3750 50  0001 C CNN
+F 0 "#PWR039" H 2300 3750 50  0001 C CNN
 F 1 "GND" H 2300 3850 50  0000 C CNN
 F 2 "" H 2300 4000 50  0000 C CNN
@@
 $EndComp
 $Comp
-L GND #PWR039
+L GND #PWR040
 U 1 1 56B26168
 P 2650 4000
-F 0 "#PWR039" H 2650 3750 50  0001 C CNN
+F 0 "#PWR040" H 2650 3750 50  0001 C CNN
 F 1 "GND" H 2650 3850 50  0000 C CNN
 F 2 "" H 2650 4000 50  0000 C CNN
@@
 $EndComp
 $Comp
-L +3V3 #PWR040
+L +3V3 #PWR041
 U 1 1 56B12EEC
 P 7850 4750
-F 0 "#PWR040" H 7850 4600 50  0001 C CNN
+F 0 "#PWR041" H 7850 4600 50  0001 C CNN
 F 1 "+3V3" H 7850 4890 50  0000 C CNN
 F 2 "" H 7850 4750 50  0000 C CNN
@@
 $EndComp
 $Comp
-L +3V3 #PWR041
+L +3V3 #PWR042
 U 1 1 56B12EF2
 P 7650 4750
-F 0 "#PWR041" H 7650 4600 50  0001 C CNN
+F 0 "#PWR042" H 7650 4600 50  0001 C CNN
 F 1 "+3V3" H 7650 4890 50  0000 C CNN
 F 2 "" H 7650 4750 50  0000 C CNN
