File: Test Projects/page4.sch (KiCad schematic (older format))
At the start: 37 parts, among them P10 CONN_01X06, P11 CONN_01X06, P12 CONN_01X06, P5 CONN_01X06, P6 CONN_01X06, P7 CONN_01X06, P73 IN2TTL, P8 CONN_01X06, P9 CONN_01X06, U10 SF-74x125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

Commit message: Finished artwork
Connections:
- net CHASSIS: now reaches JACK3.6
- net CHASSIS: now also JACK1.6, JACK1.7, JACK2.6, JACK2.7, JACK3.7
Changed lines of the file:
@@
 $EndComp
 $Comp
-L +5V #PWR046
+L +5V #PWR048
 U 1 1 568A643D
 P 2600 1800
-F 0 "#PWR046" H 2600 1650 50  0001 C CNN
+F 0 "#PWR048" H 2600 1650 50  0001 C CNN
 F 1 "+5V" H 2600 1940 50  0000 C CNN
 F 2 "" H 2600 1800 50  0000 C CNN
@@
 	2600 1800 2600 2150
 $Comp
-L GND #PWR047
+L GND #PWR049
 U 1 1 568A64CE
 P 2600 2750
-F 0 "#PWR047" H 2600 2500 50  0001 C CNN
+F 0 "#PWR049" H 2600 2500 50  0001 C CNN
 F 1 "GND" H 2600 2600 50  0000 C CNN
 F 2 "" H 2600 2750 50  0000 C CNN
@@
 $EndComp
 $Comp
-L +5V #PWR048
+L +5V #PWR050
 U 1 1 568A6ABC
 P 5050 1150
-F 0 "#PWR048" H 5050 1000 50  0001 C CNN
+F 0 "#PWR050" H 5050 1000 50  0001 C CNN
 F 1 "+5V" H 5050 1290 50  0000 C CNN
 F 2 "" H 5050 1150 50  0000 C CNN
@@
 $EndComp
 $Comp
-L +5V #PWR049
+L +5V #PWR051
 U 1 1 568A6B2D
 P 8650 1100
-F 0 "#PWR049" H 8650 950 50  0001 C CNN
+F 0 "#PWR051" H 8650 950 50  0001 C CNN
 F 1 "+5V" H 8650 1240 50  0000 C CNN
 F 2 "" H 8650 1100 50  0000 C CNN
@@
 	5050 1650 6150 1650
 $Comp
-L GND #PWR050
+L GND #PWR052
 U 1 1 568A7800
 P 3600 2100
-F 0 "#PWR050" H 3600 1850 50  0001 C CNN
+F 0 "#PWR052" H 3600 1850 50  0001 C CNN
 F 1 "GND" H 3600 1950 50  0000 C CNN
 F 2 "" H 3600 2100 50  0000 C CNN
@@
 Connection ~ 3600 2000
 $Comp
-L +5V #PWR051
+L +5V #PWR053
 U 1 1 568A78C5
 P 4800 1750
-F 0 "#PWR051" H 4800 1600 50  0001 C CNN
+F 0 "#PWR053" H 4800 1600 50  0001 C CNN
 F 1 "+5V" H 4800 1890 50  0000 C CNN
 F 2 "" H 4800 1750 50  0000 C CNN
@@
 	4700 1950 4800 1950
 $Comp
-L GND #PWR052
+L GND #PWR054
 U 1 1 568A816B
 P 7700 2350
-F 0 "#PWR052" H 7700 2100 50  0001 C CNN
+F 0 "#PWR054" H 7700 2100 50  0001 C CNN
 F 1 "GND" H 7700 2200 50  0000 C CNN
 F 2 "" H 7700 2350 50  0000 C CNN
@@
 Connection ~ 7700 2250
 $Comp
-L +5V #PWR053
+L +5V #PWR055
 U 1 1 568A8176
 P 8900 2000
-F 0 "#PWR053" H 8900 1850 50  0001 C CNN
+F 0 "#PWR055" H 8900 1850 50  0001 C CNN
 F 1 "+5V" H 8900 2140 50  0000 C CNN
 F 2 "" H 8900 2000 50  0000 C CNN
@@
 $EndComp
 $Comp
-L +5V #PWR054
+L +5V #PWR056
 U 1 1 56A5543F
 P 6750 2300
-F 0 "#PWR054" H 6750 2150 50  0001 C CNN
+F 0 "#PWR056" H 6750 2150 50  0001 C CNN
 F 1 "+5V" H 6750 2440 50  0000 C CNN
 F 2 "" H 6750 2300 50  0000 C CNN
@@
 	6750 2300 6750 2650
 $Comp
-L GND #PWR055
+L GND #PWR057
 U 1 1 56A55446
 P 6750 3250
-F 0 "#PWR055" H 6750 3000 50  0001 C CNN
+F 0 "#PWR057" H 6750 3000 50  0001 C CNN
 F 1 "GND" H 6750 3100 50  0000 C CNN
 F 2 "" H 6750 3250 50  0000 C CNN
@@
 	1    0    0    -1
 $EndComp
+Wire Wire Line
+	1600 1200 1650 1200
+Wire Wire Line
+	1650 1200 1650 1150
+Wire Wire Line
+	1600 1150 1750 1150
+Text GLabel 1750 1150 2    60   Input ~ 0
+CHASSIS
+Connection ~ 1650 1150
+Wire Wire Line
+	6500 1100 6550 1100
+Wire Wire Line
+	6550 1100 6550 1050
+Wire Wire Line
+	6500 1050 6650 1050
+Text GLabel 6650 1050 2    60   Input ~ 0
+CHASSIS
+Connection ~ 6550 1050
+Wire Wire Line
+	9250 1150 9300 1150
+Wire Wire Line
+	9300 1150 9300 1100
+Wire Wire Line
+	9250 1100 9400 1100
+Text GLabel 9400 1100 2    60   Input ~ 0
+CHASSIS
+Connection ~ 9300 1100
 $EndSCHEMATC
